Commit message: Added tf_prefixes and namespaces

File: wilber_description/urdf/diff_unit.urdf.xacro (robot description, xacro)
@@ -13,5 +13,5 @@
       <xacro:property name="flip" value="-1" />
     </xacro:if>
-    <link name="${side}_diff_unit_link">
+    <link name="${tf_prefix}${side}_diff_unit_link">
       <inertial>
         <origin xyz="0 ${flip*-1*0.05} 0.197" rpy="0 0 0" />
@@ -41,8 +41,8 @@
       </visual>
     </link>
-    <joint name="${side}_diff_unit_joint" type="fixed">
+    <joint name="${tf_prefix}${side}_diff_unit_joint" type="fixed">
       <limit upper="0.4" lower="-0.4" effort="100" velocity="1" />
-      <parent link="chassis_link" />
-      <child link="${side}_diff_unit_link" />
+      <parent link="${tf_prefix}chassis_link" />
+      <child link="${tf_prefix}${side}_diff_unit_link" />
       <origin xyz="${diff_unit_offset_x} ${diff_unit_offset_y*flip} ${diff_unit_offset_z}"
         rpy="0 0 0" />
@@ -50,5 +50,5 @@
       <dynamics damping="100" friction="0.5" />
     </joint>
-    <link name="${side}_diff_unit_headlight_link">
+    <link name="${tf_prefix}${side}_diff_unit_headlight_link">
       <visual>
         <origin xyz="0 ${flip*-0.0244} 0" rpy="0 0 0" />
@@ -59,7 +59,7 @@
       </visual>
     </link>
-    <joint name="${side}_diff_unit_headlight_joint" type="fixed">
-      <parent link="${side}_diff_unit_link" />
-      <child link="${side}_diff_unit_headlight_link" />
+    <joint name="${tf_prefix}${side}_diff_unit_headlight_joint" type="fixed">
+      <parent link="${tf_prefix}${side}_diff_unit_link" />
+      <child link="${tf_prefix}${side}_diff_unit_headlight_link" />
       <origin xyz="0 0 0" rpy="0 0 0" />
     </joint>
@@ -74,5 +74,5 @@
       </visual>
     </gazebo>
-    <link name="${side}_diff_unit_taillight_link">
+    <link name="${tf_prefix}${side}_diff_unit_taillight_link">
       <visual>
         <origin xyz="0 ${flip*-0.0244} 0" rpy="0 0 ${flip*PI}" />
@@ -83,10 +83,10 @@
       </visual>
     </link>
-    <joint name="${side}_diff_unit_taillight_joint" type="fixed">
-      <parent link="${side}_diff_unit_link" />
-      <child link="${side}_diff_unit_taillight_link" />
+    <joint name="${tf_prefix}${side}_diff_unit_taillight_joint" type="fixed">
+      <parent link="${tf_prefix}${side}_diff_unit_link" />
+      <child link="${tf_prefix}${side}_diff_unit_taillight_link" />
       <origin xyz="0 0 0" rpy="0 0 0" />
     </joint>
-    <gazebo reference="${side}_diff_unit_taillight_link">
+    <gazebo reference="${tf_prefix}${side}_diff_unit_taillight_link">
       <visual>
         <material>
@@ -98,5 +98,5 @@
       </visual>
     </gazebo>
-    <gazebo reference="${side}_diff_unit_link">
+    <gazebo reference="${tf_prefix}${side}_diff_unit_link">
       <selfCollide>false</selfCollide>
       <visual>

File: wilber_description/urdf/w200.urdf.xacro (robot description, xacro)
@@ -8,5 +8,6 @@
                 color:='yellow'
                 ns">
-    <xacro:arg name="gazebo_controllers" default="$(find wilber_deploy)/config/control.yaml" />
+    <xacro:arg name="gazebo_controllers"
+      default="$(find wilber_deploy)/config/${tf_prefix}control.yaml" />
     <xacro:arg name="use_platform_controllers" default="true" />
     <!-- Include URDF/XACRO Files -->
@@ -51,11 +52,11 @@
     <xacro:property name="dummy_inertia" value="1e-09" />
     <!-- Chassis -->
-    <link name="base_link"></link>
-    <joint name="base_link_joint" type="fixed">
+    <link name="${tf_prefix}base_link"></link>
+    <joint name="${tf_prefix}base_link_joint" type="fixed">
       <origin xyz="0 0 0.025" rpy="0 0 0" />
-      <parent link="base_link" />
-      <child link="chassis_link" />
-    </joint>
-    <link name="chassis_link">
+      <parent link="${tf_prefix}base_link" />
+      <child link="${tf_prefix}chassis_link" />
+    </joint>
+    <link name="${tf_prefix}chassis_link">
       <inertial>
         <origin xyz="0 0 0" rpy="0 0 0" />
@@ -92,5 +93,5 @@
     <xacro:w200_diff_unit side="left" />
     <xacro:w200_diff_unit side="right" />
-    <link name="diff_link">
+    <link name="${tf_prefix}diff_link">
       <visual>
         <origin xyz="0 0 0" rpy="0 0 0" />
@@ -115,7 +116,7 @@
       </visual>
     </link>
-    <joint name="diff_link_joint" type="fixed">
-      <parent link="chassis_link" />
-      <child link="diff_link" />
+    <joint name="${tf_prefix}diff_link_joint" type="fixed">
+      <parent link="${tf_prefix}chassis_link" />
+      <child link="${tf_prefix}diff_link" />
       <origin xyz="-0.5826 0 0.24979" rpy="0 0 0" />
     </joint>
@@ -160,5 +161,5 @@
 -->
     <!-- Internal IMU -->
-    <link name="imu_0_link">
+    <link name="${tf_prefix}imu_0_link">
       <inertial>
         <mass value="0.001" />
@@ -169,13 +170,13 @@
     </link>
     <joint name="imu_joint" type="fixed">
-      <parent link="chassis_link" />
-      <child link="imu_0_link" />
-    </joint>
-    <gazebo reference="imu_0_link">
+      <parent link="${tf_prefix}chassis_link" />
+      <child link="${tf_prefix}imu_0_link" />
+    </joint>
+    <gazebo reference="${tf_prefix}imu_0_link">
       <sensor type="imu" name="imu_0">
         <always_on>true</always_on>
         <update_rate>50</update_rate>
         <visualize>true</visualize>
-        <ignition_frame_id>imu_0_link</ignition_frame_id>
+        <ignition_frame_id>${tf_prefix}imu_0_link</ignition_frame_id>
         <topic>$(arg ns)/sensors/imu_0/data_raw</topic>
       </sensor>
@@ -196,29 +197,29 @@
           </xacro:unless>
         </hardware>
-        <joint name="front_left_wheel_joint">
-          <command_interface name="velocity">
-            <param name="min">-25</param>
-            <param name="max">25</param>
-          </command_interface>
-          <state_interface name="position" />
-          <state_interface name="velocity" />
-        </joint>
-        <joint name="rear_left_wheel_joint">
-          <command_interface name="velocity">
-            <param name="min">-25</param>
-            <param name="max">25</param>
-          </command_interface>
-          <state_interface name="position" />
-          <state_interface name="velocity" />
-        </joint>
-        <joint name="front_right_wheel_joint">
-          <command_interface name="velocity">
-            <param name="min">-25</param>
-            <param name="max">25</param>
-          </command_interface>
-          <state_interface name="position" />
-          <state_interface name="velocity" />
-        </joint>
-        <joint name="rear_right_wheel_joint">
+        <joint name="${tf_prefix}front_left_wheel_joint">
+          <command_interface name="velocity">
+            <param name="min">-25</param>
+            <param name="max">25</param>
+          </command_interface>
+          <state_interface name="position" />
+          <state_interface name="velocity" />
+        </joint>
+        <joint name="${tf_prefix}rear_left_wheel_joint">
+          <command_interface name="velocity">
+            <param name="min">-25</param>
+            <param name="max">25</param>
+          </command_interface>
+          <state_interface name="position" />
+          <state_interface name="velocity" />
+        </joint>
+        <joint name="${tf_prefix}front_right_wheel_joint">
+          <command_interface name="velocity">
+            <param name="min">-25</param>
+            <param name="max">25</param>
+          </command_interface>
+          <state_interface name="position" />
+          <state_interface name="velocity" />
+        </joint>
+        <joint name="${tf_prefix}rear_right_wheel_joint">
           <command_interface name="velocity">
             <param name="min">-25</param>
@@ -234,23 +235,23 @@
         <plugin filename="libignition-gazebo-wheel-slip-system.so"
           name="ignition::gazebo::systems::WheelSlip">
-          <wheel link_name="front_left_wheel_link">
-            <slip_compliance_lateral>1.0</slip_compliance_lateral>
-            <slip_compliance_longitudinal>1.0</slip_compliance_longitudinal>
-            <wheel_normal_force>686</wheel_normal_force>
-            <wheel_radius>${wheel_radius}</wheel_radius>
-          </wheel>
-          <wheel link_name="front_right_wheel_link">
-            <slip_compliance_lateral>1.0</slip_compliance_lateral>
-            <slip_compliance_longitudinal>1.0</slip_compliance_longitudinal>
-            <wheel_normal_force>686</wheel_normal_force>
-            <wheel_radius>${wheel_radius}</wheel_radius>
-          </wheel>
-          <wheel link_name="rear_left_wheel_link">
-            <slip_compliance_lateral>1.0</slip_compliance_lateral>
-            <slip_compliance_longitudinal>1.0</slip_compliance_longitudinal>
-            <wheel_normal_force>686</wheel_normal_force>
-            <wheel_radius>${wheel_radius}</wheel_radius>
-          </wheel>
-          <wheel link_name="rear_right_wheel_link">
+          <wheel link_name="${tf_prefix}front_left_wheel_link">
+            <slip_compliance_lateral>1.0</slip_compliance_lateral>
+            <slip_compliance_longitudinal>1.0</slip_compliance_longitudinal>
+            <wheel_normal_force>686</wheel_normal_force>
+            <wheel_radius>${wheel_radius}</wheel_radius>
+          </wheel>
+          <wheel link_name="${tf_prefix}front_right_wheel_link">
+            <slip_compliance_lateral>1.0</slip_compliance_lateral>
+            <slip_compliance_longitudinal>1.0</slip_compliance_longitudinal>
+            <wheel_normal_force>686</wheel_normal_force>
+            <wheel_radius>${wheel_radius}</wheel_radius>
+          </wheel>
+          <wheel link_name="${tf_prefix}rear_left_wheel_link">
+            <slip_compliance_lateral>1.0</slip_compliance_lateral>
+            <slip_compliance_longitudinal>1.0</slip_compliance_longitudinal>
+            <wheel_normal_force>686</wheel_normal_force>
+            <wheel_radius>${wheel_radius}</wheel_radius>
+          </wheel>
+          <wheel link_name="${tf_prefix}rear_right_wheel_link">
             <slip_compliance_lateral>1.0</slip_compliance_lateral>
             <slip_compliance_longitudinal>1.0</slip_compliance_longitudinal>

File: wilber_description/urdf/wheels/track.urdf.xacro (robot description, xacro)
@@ -3,5 +3,5 @@
   <xacro:macro name="w200_track" params="prefix side *joint_pose">
     <xacro:property name="rotate" value="${(prefix=='rear')*math.pi}" />
-    <link name="${prefix}_${side}_track_link">
+    <link name="${tf_prefix}${prefix}_${side}_track_link">
       <visual>
         <origin xyz="0 0 0" rpy="0 0 0" />
@@ -24,12 +24,12 @@
       </collision>
     </link>
-    <joint name="${prefix}_${side}_track_joint" type="fixed">
-      <parent link="${side}_diff_unit_link" />
-      <child link="${prefix}_${side}_track_link" />
+    <joint name="${tf_prefix}${prefix}_${side}_track_joint" type="fixed">
+      <parent link="${tf_prefix}${side}_diff_unit_link" />
+      <child link="${tf_prefix}${prefix}_${side}_track_link" />
       <xacro:insert_block name="joint_pose" />
       <axis xyz="0 1 0" />
     </joint>
     <!-- This adds wheels that rotate instead of tracks. -->
-    <link name="${prefix}_${side}_wheel_link">
+    <link name="${tf_prefix}${prefix}_${side}_wheel_link">
       <inertial>
         <origin xyz="0 0 0" rpy="0 0 0" />
@@ -44,11 +44,11 @@
       </collision>
     </link>
-    <joint name="${prefix}_${side}_wheel_joint" type="continuous">
-      <parent link="${prefix}_${side}_track_link" />
-      <child link="${prefix}_${side}_wheel_link" />
+    <joint name="${tf_prefix}${prefix}_${side}_wheel_joint" type="continuous">
+      <parent link="${tf_prefix}${prefix}_${side}_track_link" />
+      <child link="${tf_prefix}${prefix}_${side}_wheel_link" />
       <origin xyz="0.12 0. -0.18" rpy="0 0 ${rotate}" />
       <axis xyz="0 1 0" />
     </joint>
-    <gazebo reference="${prefix}_${side}_wheel_link">
+    <gazebo reference="${tf_prefix}${prefix}_${side}_wheel_link">
       <selfCollide>false</selfCollide>
       <mu1>0.5</mu1>

File: wilber_description/urdf/wheels/wheel.urdf.xacro (robot description, xacro)
@@ -7,5 +7,5 @@
   </xacro:macro>
   <xacro:macro name="w200_wheel" params="prefix side *joint_pose">
-    <link name="${prefix}_${side}_wheel_link">
+    <link name="${tf_prefix}${prefix}_${side}_wheel_link">
       <inertial>
         <origin xyz="0 0 0" rpy="0 0 0" />
@@ -27,14 +27,18 @@
       </collision>
     </link>
-    <joint name="${prefix}_${side}_wheel_joint" type="continuous">
-      <parent link="${side}_diff_unit_link" />
-      <child link="${prefix}_${side}_wheel_link" />
+    <joint name="${tf_prefix}${prefix}_${side}_wheel_joint" type="continuous">
+      <parent link="${tf_prefix}${side}_diff_unit_link" />
+      <child link="${tf_prefix}${prefix}_${side}_wheel_link" />
       <xacro:insert_block name="joint_pose" />
       <axis xyz="0 1 0" />
     </joint>
-    <gazebo reference="${prefix}_${side}_wheel_link">
+    <gazebo reference="${tf_prefix}${prefix}_${side}_wheel_link">
       <selfCollide>false</selfCollide>
-      <mu1>0.5</mu1>
-      <mu2>0.5</mu2>
+      <!-- values from
+      https://github.com/unmannedlab/cartographer/blob/main/src/platform_description/urdf/warthog.urdf.xacro-->
+      <mu1>1.0</mu1>
+      <mu2>1.0</mu2>
+      <kp value="10000000.0" />
+      <kd value="1.0" />
       <fdir1 value="1 0 0" />
       <material>Gazebo/DarkGrey</material>
