Commit message: Added bulkhead

File: wilber_description/urdf/w200.urdf.xacro (robot description, xacro)
@@ -152,12 +152,10 @@
     </xacro:if>
     <!-- Virtual Mounting Point -->
-    <!--
-    <link name="default_mount"></link>
-    <joint name="default_mount_joint" type="fixed">
+    <link name="${tf_prefix}default_mount"></link>
+    <joint name="${tf_prefix}default_mount_joint" type="fixed">
       <origin xyz="0 0 0.27218" rpy="0 0 0" />
-      <parent link="chassis_link" />
-      <child link="default_mount" />
-    </joint>
--->
+      <parent link="${tf_prefix}chassis_link" />
+      <child link="${tf_prefix}default_mount" />
+    </joint>
     <!-- Internal IMU -->
     <link name="${tf_prefix}imu_0_link">

File: wilber_description/urdf/wilber.urdf.xacro (robot description, xacro)
@@ -8,4 +8,12 @@
     <xacro:include filename="$(find clearpath_platform_description)/urdf/common.urdf.xacro" />
     <xacro:include filename="$(find wilber_description)/urdf/w200.urdf.xacro" />
+    <!-- Attachments -->
+    <xacro:include
+        filename="$(find wilber_description)/urdf/attachments/bulkhead.urdf.xacro" />
+    <xacro:bulkhead name="bulkhead" model="$(arg tf_prefix)arm_plate"
+        parent_link="$(arg tf_prefix)default_mount"
+        tf_prefix="$(arg tf_prefix)">
+        <origin xyz="0.0 0.0 0.0" rpy="0.0 0.0 0.0" />
+    </xacro:bulkhead>
     <xacro:w200
         tf_prefix="$(arg tf_prefix)"

Commit message: added GPS

File: wilber_description/urdf/w200.urdf.xacro (robot description, xacro)
@@ -186,4 +186,30 @@
       </gazebo>
     </xacro:if>
+    <!-- GPS -->
+    <link name="${tf_prefix}gps_0_link">
+      <inertial>
+        <mass value="0.001" />
+        <origin xyz="0 0.05 0" rpy="0 0 0" />
+        <inertia ixx="${dummy_inertia}" ixy="0.0" ixz="0.0" iyy="${dummy_inertia}" iyz="0.0"
+          izz="${dummy_inertia}" />
+      </inertial>
+    </link>
+    <joint name="gps_joint" type="fixed">
+      <parent link="${tf_prefix}chassis_link" />
+      <child link="${tf_prefix}gps_0_link" />
+    </joint>
+    <xacro:if value="$(arg is_sim)">
+      <gazebo reference="${tf_prefix}gps_0_link">
+        <sensor type="navsat" name="gps_0">
+          <plugin filename="libignition-gazebo-navsat-system.so" name="ignition::gazebo::systems::NavSat">
+          </plugin>
+          <always_on>true</always_on>
+          <update_rate>50</update_rate>
+          <visualize>true</visualize>
+          <ignition_frame_id>${tf_prefix}gps_0_link</ignition_frame_id>
+          <topic>$(arg ns)/sensors/gps_0/data_raw</topic>
+        </sensor>
+      </gazebo>
+    </xacro:if>
     <!-- Gazebo Controller -->
     <xacro:include filename="$(find wilber_description)/urdf/gazebo.urdf.xacro" />
