Commit message: Add mock hardware plugins and options to description, update is_sim param name to sim_ignition

File: wilbur_description/urdf/gazebo.urdf.xacro (robot description, xacro)
@@ -1,5 +1,5 @@
 <?xml version="1.0"?>
 <robot xmlns:xacro="http://ros.org/wiki/xacro">
-  <xacro:if value="$(arg is_sim)">
+  <xacro:if value="$(arg sim_ignition)">
     <gazebo>
       <plugin filename="libign_ros2_control-system.so"

File: wilbur_description/urdf/w200.urdf.xacro (robot description, xacro)
@@ -5,5 +5,6 @@
     params="wheel:='default'
                 tf_prefix
-                is_sim:=true
+                sim_ignition:=true
+                use_fake_hardware:=false
                 color:='yellow'
                 ns">
@@ -172,5 +173,5 @@
       <child link="${tf_prefix}imu_0_link" />
     </joint>
-    <xacro:if value="$(arg is_sim)">
+    <xacro:if value="${sim_ignition}">
       <gazebo reference="${tf_prefix}imu_0_link">
         <sensor type="imu" name="imu_0">
@@ -198,5 +199,5 @@
       <child link="${tf_prefix}gps_0_link" />
     </joint>
-    <xacro:if value="$(arg is_sim)">
+    <xacro:if value="${sim_ignition}">
       <gazebo reference="${tf_prefix}gps_0_link">
         <sensor type="navsat" name="gps_0">
@@ -218,8 +219,11 @@
         name="w200_hardware" type="system">
         <hardware>
-          <xacro:if value="$(arg is_sim)">
+          <xacro:if value="${sim_ignition}">
             <plugin>ign_ros2_control/IgnitionSystem</plugin>
           </xacro:if>
-          <xacro:unless value="$(arg is_sim)">
+          <xacro:if value="${use_fake_hardware}">
+            <plugin>mock_components/GenericSystem</plugin>
+          </xacro:if>
+          <xacro:unless value="${sim_ignition or use_fake_hardware}">
             <plugin>clearpath_hardware_interfaces/W200Hardware</plugin>
             <param name="wheel_diameter">0.6</param>
@@ -260,5 +264,5 @@
       </ros2_control>
     </xacro:if>
-    <xacro:if value="$(arg is_sim)">
+    <xacro:if value="${sim_ignition}">
       <gazebo>
         <plugin filename="libignition-gazebo-wheel-slip-system.so"

File: wilbur_description/urdf/wilbur.urdf.xacro (robot description, xacro)
@@ -3,9 +3,8 @@
     <xacro:arg name="tf_prefix" default="" />
     <xacro:arg name="ns" default="" />
-    <xacro:arg
-        name="is_sim" default="true" />
+    <xacro:arg name="sim_ignition" default="false" />
+    <xacro:arg name="use_fake_hardware" default="true" />
     <xacro:arg name="parent" default="world" />
-    <xacro:arg
-        name="ur_type" default="ur10e" />
+    <xacro:arg name="ur_type" default="ur10e" />
     <!-- Includes -->
     <xacro:include filename="$(find clearpath_platform_description)/urdf/common.urdf.xacro" />
@@ -40,9 +39,11 @@
     </xacro:frame>
     <!-- Manipulators -->
+    <xacro:property name="initial_positions_file" default="$(find wilbur_deploy)/config/ur_initial_positions.yaml" />
     <xacro:ur_robot
         name="arm_0_"
         tf_prefix="$(arg tf_prefix)arm_0_"
         parent="arm_plate_mount"
-        sim_ignition="true"
+        use_fake_hardware="$(arg use_fake_hardware)"
+        initial_positions="${xacro.load_yaml(initial_positions_file)}"
         joint_limits_parameters_file="$(find ur_description)/config/$(arg ur_type)/joint_limits.yaml"
         kinematics_parameters_file="$(find ur_description)/config/$(arg ur_type)/default_kinematics.yaml"
@@ -58,5 +59,6 @@
     <xacro:w200
         tf_prefix="$(arg tf_prefix)"
-        is_sim="$(arg is_sim)"
+        sim_ignition="$(arg sim_ignition)"
+        use_fake_hardware="$(arg use_fake_hardware)"
         ns="$(arg ns)"
     />
