Commit message: Add default poses, make it possible to skip ros2 control configs on per robot basis

File: wilbur_description/urdf/w200.urdf.xacro (robot description, xacro)
@@ -11,5 +11,5 @@
     <xacro:arg name="gazebo_controllers"
       default="$(find wilbur_deploy)/config/${tf_prefix}control.yaml" />
-    <xacro:arg name="use_platform_controllers" default="true" />
+    <xacro:arg name="use_w200_controllers" default="true" />
     <!-- Include URDF/XACRO Files -->
     <xacro:include filename="$(find wilbur_description)/urdf/wheels/track.urdf.xacro" />
@@ -215,7 +215,6 @@
     <xacro:include filename="$(find wilbur_description)/urdf/gazebo.urdf.xacro" />
     <!-- ROS2 controls -->
-    <xacro:if value="$(arg use_platform_controllers)">
-      <ros2_control
-        name="w200_hardware" type="system">
+    <xacro:if value="$(arg use_w200_controllers)">
+      <ros2_control name="w200_hardware" type="system">
         <hardware>
           <xacro:if value="${sim_ignition}">
@@ -235,6 +234,10 @@
             <param name="max">25</param>
           </command_interface>
-          <state_interface name="position" />
-          <state_interface name="velocity" />
+          <state_interface name="position" >
+            <param name="initial_value">0.0</param>
+          </state_interface>
+          <state_interface name="velocity" >
+            <param name="initial_value">0.0</param>
+          </state_interface>
         </joint>
         <joint name="${tf_prefix}rear_left_wheel_joint">
@@ -243,6 +246,10 @@
             <param name="max">25</param>
           </command_interface>
-          <state_interface name="position" />
-          <state_interface name="velocity" />
+          <state_interface name="position" >
+            <param name="initial_value">0.0</param>
+          </state_interface>
+          <state_interface name="velocity" >
+            <param name="initial_value">0.0</param>
+          </state_interface>
         </joint>
         <joint name="${tf_prefix}front_right_wheel_joint">
@@ -251,6 +258,10 @@
             <param name="max">25</param>
           </command_interface>
-          <state_interface name="position" />
-          <state_interface name="velocity" />
+          <state_interface name="position" >
+            <param name="initial_value">0.0</param>
+          </state_interface>
+          <state_interface name="velocity" >
+            <param name="initial_value">0.0</param>
+          </state_interface>
         </joint>
         <joint name="${tf_prefix}rear_right_wheel_joint">
@@ -259,6 +270,10 @@
             <param name="max">25</param>
           </command_interface>
-          <state_interface name="position" />
-          <state_interface name="velocity" />
+          <state_interface name="position" >
+            <param name="initial_value">0.0</param>
+          </state_interface>
+          <state_interface name="velocity" >
+            <param name="initial_value">0.0</param>
+          </state_interface>
         </joint>
       </ros2_control>

File: wilbur_description/urdf/wilbur.urdf.xacro (robot description, xacro)
@@ -7,4 +7,6 @@
     <xacro:arg name="parent" default="world" />
     <xacro:arg name="ur_type" default="ur10e" />
+    <xacro:arg name="generate_ros2_control_tag" default="false" />
+    <xacro:arg name="use_w200_controllers" value="false" />
     <!-- Includes -->
     <xacro:include filename="$(find clearpath_platform_description)/urdf/common.urdf.xacro" />
@@ -49,6 +51,8 @@
         kinematics_parameters_file="$(find ur_description)/config/$(arg ur_type)/default_kinematics.yaml"
         physical_parameters_file="$(find ur_description)/config/$(arg ur_type)/physical_parameters.yaml"
-        visual_parameters_file="$(find ur_description)/config/$(arg ur_type)/visual_parameters.yaml">
-        <origin xyz="0.0 0.0 0.0" rpy="0.0 0.0 0.0" />
+        visual_parameters_file="$(find ur_description)/config/$(arg ur_type)/visual_parameters.yaml"
+        generate_ros2_control_tag="$(arg generate_ros2_control_tag)"
+      >
+      <origin xyz="0.0 0.0 0.0" rpy="0.0 0.0 0.0" />
     </xacro:ur_robot>
     <!-- arm_0_gripper -->

Commit message: created wilbur_gz package - urdf compiles at this point. nothing else

File: wilbur_description/urdf/w200.urdf.xacro (robot description, xacro)
@@ -1,5 +1,5 @@
 <?xml version='1.0'?>
 <robot xmlns:xacro="http://www.ros.org/wiki/xacro">
-  <!-- W@00 Platform Macro-->
+  <!-- W200 Platform Macro-->
   <xacro:macro name="w200"
     params="wheel:='default'
@@ -9,7 +9,4 @@
                 color:='yellow'
                 ns">
-    <xacro:arg name="gazebo_controllers"
-      default="$(find wilbur_deploy)/config/gazebo_controllers.yaml" />
-    <xacro:arg name="use_w200_controllers" default="true" />
     <!-- Include URDF/XACRO Files -->
     <xacro:include filename="$(find wilbur_description)/urdf/wheels/track.urdf.xacro" />
@@ -173,17 +170,4 @@
       <child link="${tf_prefix}imu_0_link" />
     </joint>
-    <xacro:if value="${sim_ignition}">
-      <gazebo reference="${tf_prefix}imu_0_link">
-        <sensor type="imu" name="imu_0">
-          <plugin filename="libignition-gazebo-imu-system.so" name="ignition::gazebo::systems::Imu">
-          </plugin>
-          <always_on>true</always_on>
-          <update_rate>50</update_rate>
-          <visualize>true</visualize>
-          <ignition_frame_id>${tf_prefix}imu_0_link</ignition_frame_id>
-          <topic>$(arg ns)/sensors/imu_0/data_raw</topic>
-        </sensor>
-      </gazebo>
-    </xacro:if>
     <!-- GPS -->
     <link name="${tf_prefix}gps_0_link">
@@ -199,114 +183,22 @@
       <child link="${tf_prefix}gps_0_link" />
     </joint>
+    <!-- ROS2 controls -->
+    <xacro:include filename="$(find wilbur_description)/urdf/w200.ros2_control.xacro" />
+    <!-- todo do we need a ns/name paradigm for ros2 control system plugins for multiple/namespacing-->
+    <xacro:w200_ros2_control
+      name="w200_ros2_control"
+      use_fake_hardware="${use_fake_hardware}"
+      sim_ignition="${sim_ignition}"
+    />
+    <!-- w200_gz - plugins specific for the w200 for gazebo -->
     <xacro:if value="${sim_ignition}">
-      <gazebo reference="${tf_prefix}gps_0_link">
-        <sensor type="navsat" name="gps_0">
-          <plugin filename="libignition-gazebo-navsat-system.so" name="ignition::gazebo::systems::NavSat">
-          </plugin>
-          <always_on>true</always_on>
-          <update_rate>50</update_rate>
-          <visualize>true</visualize>
-          <ignition_frame_id>${tf_prefix}gps_0_link</ignition_frame_id>
-          <topic>$(arg ns)/sensors/gps_0/data_raw</topic>
-        </sensor>
-      </gazebo>
-    </xacro:if>
-    <!-- Gazebo Controller -->
-    <xacro:include filename="$(find wilbur_description)/urdf/gazebo.urdf.xacro" />
-    <!-- ROS2 controls -->
-    <xacro:if value="$(arg use_w200_controllers)">
-      <ros2_control name="w200_hardware" type="system">
-        <hardware>
-          <xacro:if value="${sim_ignition}">
-            <plugin>ign_ros2_control/IgnitionSystem</plugin>
-          </xacro:if>
-          <xacro:if value="${use_fake_hardware}">
-            <plugin>mock_components/GenericSystem</plugin>
-          </xacro:if>
-          <xacro:unless value="${sim_ignition or use_fake_hardware}">
-            <plugin>clearpath_hardware_interfaces/W200Hardware</plugin>
-            <param name="wheel_diameter">0.6</param>
-          </xacro:unless>
-        </hardware>
-        <joint name="${tf_prefix}front_left_wheel_joint">
-          <command_interface name="velocity">
-            <param name="min">-25</param>
-            <param name="max">25</param>
-          </command_interface>
-          <state_interface name="position" >
-            <param name="initial_value">0.0</param>
-          </state_interface>
-          <state_interface name="velocity" >
-            <param name="initial_value">0.0</param>
-          </state_interface>
-        </joint>
-        <joint name="${tf_prefix}rear_left_wheel_joint">
-          <command_interface name="velocity">
-            <param name="min">-25</param>
-            <param name="max">25</param>
-          </command_interface>
-          <state_interface name="position" >
-            <param name="initial_value">0.0</param>
-          </state_interface>
-          <state_interface name="velocity" >
-            <param name="initial_value">0.0</param>
-          </state_interface>
-        </joint>
-        <joint name="${tf_prefix}front_right_wheel_joint">
-          <command_interface name="velocity">
-            <param name="min">-25</param>
-            <param name="max">25</param>
-          </command_interface>
-          <state_interface name="position" >
-            <param name="initial_value">0.0</param>
-          </state_interface>
-          <state_interface name="velocity" >
-            <param name="initial_value">0.0</param>
-          </state_interface>
-        </joint>
-        <joint name="${tf_prefix}rear_right_wheel_joint">
-          <command_interface name="velocity">
-            <param name="min">-25</param>
-            <param name="max">25</param>
-          </command_interface>
-          <state_interface name="position" >
-            <param name="initial_value">0.0</param>
-          </state_interface>
-          <state_interface name="velocity" >
-            <param name="initial_value">0.0</param>
-          </state_interface>
-        </joint>
-      </ros2_control>
-    </xacro:if>
-    <xacro:if value="${sim_ignition}">
-      <gazebo>
-        <plugin filename="libignition-gazebo-wheel-slip-system.so"
-          name="ignition::gazebo::systems::WheelSlip">
-          <wheel link_name="${tf_prefix}front_left_wheel_link">
-            <slip_compliance_lateral>1.0</slip_compliance_lateral>
-            <slip_compliance_longitudinal>1.0</slip_compliance_longitudinal>
-            <wheel_normal_force>686</wheel_normal_force>
-            <wheel_radius>${wheel_radius}</wheel_radius>
-          </wheel>
-          <wheel link_name="${tf_prefix}front_right_wheel_link">
-            <slip_compliance_lateral>1.0</slip_compliance_lateral>
-            <slip_compliance_longitudinal>1.0</slip_compliance_longitudinal>
-            <wheel_normal_force>686</wheel_normal_force>
-            <wheel_radius>${wheel_radius}</wheel_radius>
-          </wheel>
-          <wheel link_name="${tf_prefix}rear_left_wheel_link">
-            <slip_compliance_lateral>1.0</slip_compliance_lateral>
-            <slip_compliance_longitudinal>1.0</slip_compliance_longitudinal>
-            <wheel_normal_force>686</wheel_normal_force>
-            <wheel_radius>${wheel_radius}</wheel_radius>
-          </wheel>
-          <wheel link_name="${tf_prefix}rear_right_wheel_link">
-            <slip_compliance_lateral>1.0</slip_compliance_lateral>
-            <slip_compliance_longitudinal>1.0</slip_compliance_longitudinal>
-            <wheel_normal_force>686</wheel_normal_force>
-            <wheel_radius>${wheel_radius}</wheel_radius>
-          </wheel>
-        </plugin>
-      </gazebo>
+      <xacro:include filename="$(find wilbur_gz)/urdf/w200_gz.xacro" />
+      <xacro:w200_gz
+        tf_prefix="${tf_prefix}"
+        wheel_radius="${wheel_radius}"
+        imu_link_name="imu_0_link"
+        gps_link_name="gps_0_link"
+        ns="${ns}">
+      </xacro:w200_gz>
     </xacro:if>
   </xacro:macro>

File: wilbur_description/urdf/wilbur.urdf.xacro (robot description, xacro)
@@ -2,11 +2,12 @@
 <robot name="wilbur" xmlns:xacro="http://ros.org/wiki/xacro">
     <xacro:arg name="tf_prefix" default="" />
+    <!-- todo convert file to 2 spaces -->
     <xacro:arg name="ns" default="" />
     <xacro:arg name="sim_ignition" default="false" />
-    <xacro:arg name="use_fake_hardware" default="true" />
+    <xacro:arg name="use_fake_hardware" default="true" /> <!-- todo look into calling this use_mock_hardware to be forward leaning-->
     <xacro:arg name="parent" default="world" />
-    <xacro:arg name="ur_type" default="ur10e" />
-    <xacro:arg name="generate_ros2_control_tag" default="false" />
-    <xacro:arg name="use_w200_controllers" default="false" />
+    <xacro:arg name="ur_type" default="ur10e" /> <!-- todo set to value-->
+    <xacro:arg name="generate_ros2_control_tag" default="false" /> <!-- would we ever have this false-->
+    <xacro:arg name="use_w200_controllers" default="false" /> <!-- appears unused-->
     <!-- Includes -->
     <xacro:include filename="$(find clearpath_platform_description)/urdf/common.urdf.xacro" />
@@ -18,8 +19,5 @@
     <!--xacro:include
         filename="$(find clearpath_manipulators_description)/urdf/arm/universal_robots.urdf.xacro" /-->
-    <xacro:include
-        filename="$(find ur_description)/urdf/ur_macro.xacro" />
-    <!--xacro:include
-        filename="$(find ur_description)/urdf/gripper/robotiq_2f_85.urdf.xacro" /-->
+    <xacro:include filename="$(find ur_description)/urdf/ur_macro.xacro" />
     <!-- Attachments -->
     <xacro:bulkhead
@@ -31,4 +29,5 @@
     </xacro:bulkhead>
     <!-- Links -->
+    <!-- todo - reduce dependency on clearpath palatform description buildin macros -->
     <xacro:mesh
         name="control_frame"
@@ -37,4 +36,5 @@
         <origin xyz="0.0 0.0 0.0" rpy="0.0 0.0 0.0" />
     </xacro:mesh>
+    <!-- todo - reduce dependency on clearpath palatform description buildin macros -->
     <xacro:frame name="arm_0_end_effector" parent_link="arm_0_tool0">
         <origin xyz="0.0 0.0 0.0" rpy="0.0 0.0 0.0" />
@@ -42,4 +42,5 @@
     <!-- Manipulators -->
     <xacro:property name="initial_positions_file" default="$(find wilbur_deploy)/config/ur_initial_positions.yaml" />
+    <!-- todo expose out args for hardware-->
     <xacro:ur_robot
         name="arm_0_"
@@ -63,4 +64,5 @@
     </xacro:robotiq_2f_85-->
     <xacro:w200
+        wheel="default"
         tf_prefix="$(arg tf_prefix)"
         sim_ignition="$(arg sim_ignition)"
@@ -68,3 +70,12 @@
         ns="$(arg ns)"
     />
+    <xacro:if value="$(arg sim_ignition)">
+      <xacro:include filename="$(find wilbur_gz)/urdf/wilbur_gz.ros2_control.xacro" />
+      <xacro:wilbur_gz_ros2_control
+        gazebo_controllers_config_file="$(find wilbur_gz)/config/gazebo_controllers.yaml"
+        ns="$(arg ns)"
+      />
+      <xacro:include filename="$(find wilbur_gz)/urdf/wilbur_gz.xacro" />
+      <xacro:wilbur_gz/>
+    </xacro:if>
 </robot>

File: wilbur_gz/urdf/wilbur_gz.ros2_control.xacro (robot description, xacro)
@@ -1,9 +1,13 @@
 <?xml version="1.0"?>
 <robot xmlns:xacro="http://ros.org/wiki/xacro">
-  <xacro:if value="$(arg sim_ignition)">
+  <xacro:macro name="wilbur_gz_ros2_control" params="
+    gazebo_controllers_config_file:=$(find wilbur_gz)/config/gazebo_controllers.yaml
+    ns
+  ">
     <gazebo>
+      <!-- gazebo plugin to enable ros2 control for the system -->
       <plugin filename="libign_ros2_control-system.so"
         name="ign_ros2_control::IgnitionROS2ControlPlugin">
-        <parameters>$(arg gazebo_controllers)</parameters>
+        <parameters>$(arg gazebo_controllers_config_file)</parameters>
         <controller_manager_name>controller_manager</controller_manager_name>
         <ros>
@@ -21,13 +25,4 @@
       </plugin>
     </gazebo>
-    <gazebo>
-      <plugin filename="libignition-gazebo-pose-publisher-system.so"
-        name="ignition::gazebo::systems::PosePublisher">
-        <publish_link_pose>true</publish_link_pose>
-        <publish_nested_model_pose>true</publish_nested_model_pose>
-        <use_pose_vector_msg>true</use_pose_vector_msg>
-        <update_frequency>50</update_frequency>
-      </plugin>
-    </gazebo>
-  </xacro:if>
+  </xacro:macro>
 </robot>
