Commit message: Remove gazebo references from wilbur_descriptions and got the gz sim working

File: wilbur_description/urdf/w200.urdf.xacro (robot description, xacro)
@@ -13,5 +13,4 @@
     use_fake_hardware="$(arg use_fake_hardware)"
     ns="$(arg ns)"
-    generate_ros2_control_tag="$(arg generate_ros2_control_tag)"
   />
 </robot>

File: wilbur_description/urdf/wilbur.urdf.xacro (robot description, xacro)
@@ -11,4 +11,5 @@
   <xacro:arg name="wilbur_ur10e_initial_positions"
     default="$(find wilbur_deploy)/config/ur_initial_positions.yaml" />
+  <xacro:arg name="generate_ros2_control_tag" default="false" />
   <!-- Force absolute mesh paths, necessary for Gazebo. -->
   <xacro:property name="force_abs_paths" value="$(arg abs_mesh_paths)" scope="global" />
@@ -23,4 +24,5 @@
     gripper_com_port="$(arg gripper_com_port)"
     wilbur_ur10e_initial_positions="$(arg wilbur_ur10e_initial_positions)"
+    generate_ros2_control_tag="$(arg generate_ros2_control_tag)"
   />
 </robot>

File: wilbur_description/urdf/wilbur.xacro (robot description, xacro)
@@ -60,4 +60,5 @@
         parent="${tf_prefix}arm_plate_mount"
         initial_positions="${xacro.load_yaml(initial_positions_file)}"
+        generate_ros2_control_tag="${generate_ros2_control_tag}"
       >
         <origin xyz="0.0 0.0 0.0" rpy="0.0 0.0 0.0" />
@@ -68,4 +69,5 @@
       <xacro:dextivr_hande
         name="dextivr_hande"
+        generate_ros2_control_tag="$(arg generate_ros2_control_tag)"
         tf_prefix="${tf_prefix}arm_0_"
         parent="${tf_prefix}arm_0_end_effector_link"

File: wilbur_description/urdf/wilbur_ur10e_macro.urdf.xacro (robot description, xacro)
@@ -8,4 +8,5 @@
             parent:='world'
             initial_positions='$(find wilbur_deploy)/config/ur_initial_positions.yaml'
+            generate_ros2_control_tag:=false
             ">
     <xacro:include filename="$(find ur_description)/urdf/ur_macro.xacro" />

File: wilbur_gz/urdf/wilbur_gz.ros2_control.xacro (robot description, xacro)
@@ -3,4 +3,7 @@
   <xacro:macro name="wilbur_gz_ros2_control" params="
     gazebo_controllers_config_file
+    include_ur=true
+    tf_prefix=''
+    name='wilbur'
     ns
   ">
@@ -25,4 +28,107 @@
       </plugin>
     </gazebo>
+    <ros2_control name="${name}" type="system">
+      <hardware>
+          <plugin>gz_ros2_control/GazeboSimSystem</plugin>
+      </hardware>
+      <xacro:if value="$(arg include_ur)">
+        <joint name="${tf_prefix}arm_0_shoulder_pan_joint">
+          <command_interface name="position" />
+          <command_interface name="velocity" />
+          <command_interface name="effort" />
+          <state_interface name="position" />
+          <state_interface name="velocity" />
+          <state_interface name="effort" />
+        </joint>
+        <joint name="${tf_prefix}arm_0_shoulder_lift_joint">
+          <command_interface name="position" />
+          <command_interface name="velocity" />
+          <command_interface name="effort" />
+          <state_interface name="position" />
+          <state_interface name="velocity" />
+          <state_interface name="effort" />
+        </joint>
+        <joint name="${tf_prefix}arm_0_elbow_joint">
+          <command_interface name="position" />
+          <command_interface name="velocity" />
+          <command_interface name="effort" />
+          <state_interface name="position" />
+          <state_interface name="velocity" />
+          <state_interface name="effort" />
+        </joint>
+        <joint name="${tf_prefix}arm_0_wrist_1_joint">
+          <command_interface name="position" />
+          <command_interface name="velocity" />
+          <command_interface name="effort" />
+          <state_interface name="position" />
+          <state_interface name="velocity" />
+          <state_interface name="effort" />
+        </joint>
+        <joint name="${tf_prefix}arm_0_wrist_2_joint">
+          <command_interface name="position" />
+          <command_interface name="velocity" />
+          <command_interface name="effort" />
+          <state_interface name="position" />
+          <state_interface name="velocity" />
+          <state_interface name="effort" />
+        </joint>
+        <joint name="${tf_prefix}arm_0_wrist_3_joint">
+          <command_interface name="position" />
+          <command_interface name="velocity" />
+          <command_interface name="effort" />
+          <state_interface name="position" />
+          <state_interface name="velocity" />
+          <state_interface name="effort" />
+        </joint>
+      </xacro:if>
+      <joint name="${tf_prefix}front_left_wheel_joint">
+        <command_interface name="velocity">
+          <param name="min">-25</param>
+          <param name="max">25</param>
+        </command_interface>
+        <state_interface name="position">
+          <param name="initial_value">0.0</param>
+        </state_interface>
+        <state_interface name="velocity">
+          <param name="initial_value">0.0</param>
+        </state_interface>
+      </joint>
+      <joint name="${tf_prefix}rear_left_wheel_joint">
+        <command_interface name="velocity">
+          <param name="min">-25</param>
+          <param name="max">25</param>
+        </command_interface>
+        <state_interface name="position">
+          <param name="initial_value">0.0</param>
+        </state_interface>
+        <state_interface name="velocity">
+          <param name="initial_value">0.0</param>
+        </state_interface>
+      </joint>
+      <joint name="${tf_prefix}front_right_wheel_joint">
+        <command_interface name="velocity">
+          <param name="min">-25</param>
+          <param name="max">25</param>
+        </command_interface>
+        <state_interface name="position">
+          <param name="initial_value">0.0</param>
+        </state_interface>
+        <state_interface name="velocity">
+          <param name="initial_value">0.0</param>
+        </state_interface>
+      </joint>
+      <joint name="${tf_prefix}rear_right_wheel_joint">
+        <command_interface name="velocity">
+          <param name="min">-25</param>
+          <param name="max">25</param>
+        </command_interface>
+        <state_interface name="position">
+          <param name="initial_value">0.0</param>
+        </state_interface>
+        <state_interface name="velocity">
+          <param name="initial_value">0.0</param>
+        </state_interface>
+      </joint>
+    </ros2_control>
   </xacro:macro>
 </robot>

File: wilbur_gz/urdf/wilbur_gz.urdf.xacro (robot description, xacro)
@@ -12,6 +12,10 @@
     <xacro:arg name="wilbur_ur10e_initial_positions"
         default="$(find wilbur_deploy)/config/ur_initial_positions.yaml" />
+        "
     <xacro:include filename="$(find wilbur_description)/urdf/wilbur.xacro" />
+    <xacro:include filename="$(find wilbur_gz)/urdf/wilbur_gz.ros2_control.xacro" />
+    <xacro:include filename="$(find wilbur_gz)/urdf/wilbur_gz.xacro" />
     <xacro:property name="force_abs_paths" value="$(arg abs_mesh_paths)" scope="global" />
+    <xacro:property name="generate_ros2_control_tag" value="false" />
     <xacro:wilbur
         tf_prefix="$(arg tf_prefix)"
@@ -23,12 +27,13 @@
         gripper_com_port="$(arg gripper_com_port)"
         wilbur_ur10e_initial_positions="$(arg wilbur_ur10e_initial_positions)"
+        generate_ros2_control_tag="${generate_ros2_control_tag}"
     />
     <xacro:include filename="$(find wilbur_gz)/urdf/wilbur_gz.ros2_control.xacro" />
     <xacro:include filename="$(find wilbur_gz)/urdf/wilbur_gz.xacro" />
     <xacro:if value="$(arg include_ur)">
-        <xacro:wilbur_gz_ros2_control
-            gazebo_controllers_config_file="$(find wilbur_gz)/config/gazebo_controllers.yaml"
-            ns="$(arg ns)"
-        />
+    <xacro:wilbur_gz_ros2_control
+        gazebo_controllers_config_file="$(find wilbur_gz)/config/gazebo_controllers.yaml"
+        ns="$(arg ns)"
+    />
     </xacro:if>
     <xacro:unless value="$(arg include_ur)">
@@ -39,7 +44,3 @@
     </xacro:unless>
     <xacro:wilbur_gz />
-    <xacro:w200_ros2_control
-        name="wilbur"
-        tf_prefix="$(arg tf_prefix)"
-        include_ur="$(arg include_ur)" />
 </robot>

File: wilbur_gz/urdf/wilbur_gz.xacro (robot description, xacro)
@@ -14,113 +14,3 @@
     </gazebo>
   </xacro:macro>
-  <xacro:macro name="w200_ros2_control"
-    params="
-    name
-    tf_prefix
-    include_ur:=true
-  ">
-    <ros2_control name="${name}" type="system">
-      <hardware>
-        <plugin>gz_ros2_control/GazeboSimSystem</plugin>
-      </hardware>
-      <xacro:if value="$(arg include_ur)">
-        <joint name="${tf_prefix}arm_0_shoulder_pan_joint">
-          <command_interface name="position" />
-          <command_interface name="velocity" />
-          <command_interface name="effort" />
-          <state_interface name="position" />
-          <state_interface name="velocity" />
-          <state_interface name="effort" />
-        </joint>
-        <joint name="${tf_prefix}arm_0_shoulder_lift_joint">
-          <command_interface name="position" />
-          <command_interface name="velocity" />
-          <command_interface name="effort" />
-          <state_interface name="position" />
-          <state_interface name="velocity" />
-          <state_interface name="effort" />
-        </joint>
-        <joint name="${tf_prefix}arm_0_elbow_joint">
-          <command_interface name="position" />
-          <command_interface name="velocity" />
-          <command_interface name="effort" />
-          <state_interface name="position" />
-          <state_interface name="velocity" />
-          <state_interface name="effort" />
-        </joint>
-        <joint name="${tf_prefix}arm_0_wrist_1_joint">
-          <command_interface name="position" />
-          <command_interface name="velocity" />
-          <command_interface name="effort" />
-          <state_interface name="position" />
-          <state_interface name="velocity" />
-          <state_interface name="effort" />
-        </joint>
-        <joint name="${tf_prefix}arm_0_wrist_2_joint">
-          <command_interface name="position" />
-          <command_interface name="velocity" />
-          <command_interface name="effort" />
-          <state_interface name="position" />
-          <state_interface name="velocity" />
-          <state_interface name="effort" />
-        </joint>
-        <joint name="${tf_prefix}arm_0_wrist_3_joint">
-          <command_interface name="position" />
-          <command_interface name="velocity" />
-          <command_interface name="effort" />
-          <state_interface name="position" />
-          <state_interface name="velocity" />
-          <state_interface name="effort" />
-        </joint>
-      </xacro:if>
-      <joint name="${tf_prefix}front_left_wheel_joint">
-        <command_interface name="velocity">
-          <param name="min">-25</param>
-          <param name="max">25</param>
-        </command_interface>
-        <state_interface name="position">
-          <param name="initial_value">0.0</param>
-        </state_interface>
-        <state_interface name="velocity">
-          <param name="initial_value">0.0</param>
-        </state_interface>
-      </joint>
-      <joint name="${tf_prefix}rear_left_wheel_joint">
-        <command_interface name="velocity">
-          <param name="min">-25</param>
-          <param name="max">25</param>
-        </command_interface>
-        <state_interface name="position">
-          <param name="initial_value">0.0</param>
-        </state_interface>
-        <state_interface name="velocity">
-          <param name="initial_value">0.0</param>
-        </state_interface>
-      </joint>
-      <joint name="${tf_prefix}front_right_wheel_joint">
-        <command_interface name="velocity">
-          <param name="min">-25</param>
-          <param name="max">25</param>
-        </command_interface>
-        <state_interface name="position">
-          <param name="initial_value">0.0</param>
-        </state_interface>
-        <state_interface name="velocity">
-          <param name="initial_value">0.0</param>
-        </state_interface>
-      </joint>
-      <joint name="${tf_prefix}rear_right_wheel_joint">
-        <command_interface name="velocity">
-          <param name="min">-25</param>
-          <param name="max">25</param>
-        </command_interface>
-        <state_interface name="position">
-          <param name="initial_value">0.0</param>
-        </state_interface>
-        <state_interface name="velocity">
-          <param name="initial_value">0.0</param>
-        </state_interface>
-      </joint>
-    </ros2_control>
-  </xacro:macro>
 </robot>
