Commit message: separating out functinoality for split controller manager

File: wilbur_description/urdf/gen_mesh.xacro (robot description, xacro)
@@ -6,5 +6,5 @@
     </xacro:if>
     <xacro:unless value="${force_abs_path}">
-      <xacro:property name="mesh" value="package://$(find ${pkg_name})/${file_path}" scope="parent"/>
+      <xacro:property name="mesh" value="package://${pkg_name}/${file_path}" scope="parent"/>
     </xacro:unless>
     <mesh filename="${mesh}" scale="${scale}"/>

File: wilbur_description/urdf/w200.urdf.xacro (robot description, xacro)
@@ -1,209 +1,17 @@
-<?xml version='1.0'?>
-<robot xmlns:xacro="http://www.ros.org/wiki/xacro">
-  <!-- W200 Platform Macro-->
-  <xacro:macro name="w200"
-    params="wheel:='default'
-                tf_prefix
-                sim_ignition:=false
-                use_fake_hardware:=true
-                color:='yellow'
-                ns
-                generate_ros2_control_tag:=true">
-    <!-- Include URDF/XACRO Files -->
-    <xacro:include filename="$(find wilbur_description)/urdf/wheels/track.urdf.xacro" />
-    <xacro:include filename="$(find wilbur_description)/urdf/wheels/wheel.urdf.xacro" />
-    <xacro:property name="PI" value="3.1415926535897931" /> <!--pi is build in - replace with lowercase pi throughout and remove property -->
-    <xacro:include filename="$(find wilbur_description)/urdf/diff_unit.urdf.xacro" />
-    <!-- Colors: yellow, orange, olive, sand -->
-    <xacro:property name="warthog_color" value="${'warthog_'+color}" />
-    <material name="warthog_yellow">
-      <color rgba="0.95 0.816 0.082 1.0" />
-    </material>
-    <material name="warthog_orange">
-      <color rgba="1.0 0.48 0.0 1.0" />
-    </material>
-    <material name="warthog_olive">
-      <color rgba="0.333 0.419 0.184 1.0" />
-    </material>
-    <material name="warthog_sand">
-      <color rgba="0.86 0.75 0.54 1.0" />
-    </material>
-    <!-- Variables -->
-    <xacro:property name="wheel_radius" value="0.3" />
-    <xacro:property name="wheel_width" value="0.25" />
-    <xacro:property name="wheel_mass" value="15" />
-    <xacro:property name="wheel_to_track_ratio" value="0.5962" />
-    <xacro:property name="axle_x_offset" value="0.457367" />
-    <xacro:property name="axle_y_offset" value="0.0" />
-    <xacro:property name="axle_z_offset" value="-0.012977" />
-    <xacro:property name="track_z_offset" value="-0.2" />
-    <xacro:property name="diff_unit_length" value="1.34" />
-    <xacro:property name="diff_unit_width" value="0.28" />
-    <xacro:property name="diff_unit_height" value="0.63" />
-    <xacro:property name="diff_unit_mass" value="50" />
-    <xacro:property name="diff_unit_offset_x" value="0.00" />
-    <xacro:property name="diff_unit_offset_y" value="0.56821" />
-    <xacro:property name="diff_unit_offset_z" value="0.0" />
-    <xacro:property name="chassis_length" value="1.35" />
-    <xacro:property name="chassis_width" value="0.70" />
-    <xacro:property name="chassis_height" value="0.30" />
-    <xacro:property name="chassis_mass" value="100" />
-    <xacro:property name="dummy_inertia" value="1e-09" />
-    <!-- Chassis -->
-    <link name="${tf_prefix}base_link"></link>
-    <joint name="${tf_prefix}base_link_joint" type="fixed">
-      <origin xyz="0 0 0.025" rpy="0 0 0" />
-      <parent link="${tf_prefix}base_link" />
-      <child link="${tf_prefix}chassis_link" />
-    </joint>
-    <link name="${tf_prefix}chassis_link">
-      <inertial>
-        <origin xyz="0 0 0" rpy="0 0 0" />
-        <mass value="${chassis_mass}" />
-        <xacro:box_inertia m="${chassis_mass}" x="${chassis_length}"
-          y="${chassis_width}" z="${chassis_height}" />
-      </inertial>
-      <visual>
-        <origin xyz="0 0 0" rpy="0 0 0" />
-        <geometry>
-          <mesh filename="package://clearpath_platform_description/meshes/w200/chassis.stl" />
-        </geometry>
-        <material name="clearpath_black">
-          <color rgba="0.15 0.15 0.15 1.0" />
-        </material>
-      </visual>
-      <visual>
-        <origin xyz="0 0 0" rpy="0 0 0" />
-        <geometry>
-          <mesh filename="package://clearpath_platform_description/meshes/w200/e-stop.stl" />
-        </geometry>
-        <material name="clearpath_red">
-          <color rgba="0.9 0.0 0.0 1.0" />
-        </material>
-      </visual>
-      <collision>
-        <origin xyz="0 0 0" rpy="0 0 0" />
-        <geometry>
-          <mesh
-            filename="package://clearpath_platform_description/meshes/w200/chassis-collision.stl" />
-        </geometry>
-      </collision>
-    </link>
-    <!-- Diff. Unit -->
-    <xacro:w200_diff_unit side="left" />
-    <xacro:w200_diff_unit side="right" />
-    <link name="${tf_prefix}diff_link">
-      <visual>
-        <origin xyz="0 0 0" rpy="0 0 0" />
-        <geometry>
-          <mesh filename="package://clearpath_platform_description/meshes/w200/diff-link.stl" />
-        </geometry>
-        <material name="clearpath_light_grey" />
-      </visual>
-      <visual>
-        <origin xyz="0 0 0" rpy="0 0 0" />
-        <geometry>
-          <mesh filename="package://clearpath_platform_description/meshes/w200/susp-link.stl" />
-        </geometry>
-        <material name="clearpath_light_grey" />
-      </visual>
-      <visual>
-        <origin xyz="0 0 0" rpy="0 0 0" />
-        <geometry>
-          <mesh filename="package://clearpath_platform_description/meshes/w200/susp-link.stl" />
-        </geometry>
-        <material name="clearpath_light_grey" />
-      </visual>
-    </link>
-    <joint name="${tf_prefix}diff_link_joint" type="fixed">
-      <parent link="${tf_prefix}chassis_link" />
-      <child link="${tf_prefix}diff_link" />
-      <origin xyz="-0.5826 0 0.24979" rpy="0 0 0" />
-    </joint>
-    <!-- Wheels -->
-    <xacro:if value="${wheel == 'default'}">
-      <xacro:w200_wheel prefix="front" side="left">
-        <origin xyz="${axle_x_offset*1} ${axle_y_offset*1} ${axle_z_offset}" rpy="0 0 0" />
-      </xacro:w200_wheel>
-      <xacro:w200_wheel prefix="front" side="right">
-        <origin xyz="${axle_x_offset*1} ${axle_y_offset*-1} ${axle_z_offset}" rpy="0 0 0" />
-      </xacro:w200_wheel>
-      <xacro:w200_wheel prefix="rear" side="left">
-        <origin xyz="${axle_x_offset*-1} ${axle_y_offset*1} ${axle_z_offset}" rpy="0 0 0" />
-      </xacro:w200_wheel>
-      <xacro:w200_wheel prefix="rear" side="right">
-        <origin xyz="${axle_x_offset*-1} ${axle_y_offset*-1} ${axle_z_offset}" rpy="0 0 0" />
-      </xacro:w200_wheel>
-    </xacro:if>
-    <!-- Tracks -->
-    <xacro:if value="${wheel == 'track'}">
-      <xacro:w200_track prefix="front" side="left">
-        <origin xyz="${axle_x_offset*1} ${axle_y_offset*1} ${axle_z_offset}" rpy="0 0 0" />
-      </xacro:w200_track>
-      <xacro:w200_track prefix="front" side="right">
-        <origin xyz="${axle_x_offset*1} ${axle_y_offset*-1} ${axle_z_offset}" rpy="0 0 0" />
-      </xacro:w200_track>
-      <xacro:w200_track prefix="rear" side="left">
-        <origin xyz="${axle_x_offset*-1} ${axle_y_offset*1} ${axle_z_offset}" rpy="0 0 ${PI}" />
-      </xacro:w200_track>
-      <xacro:w200_track prefix="rear" side="right">
-        <origin xyz="${axle_x_offset*-1} ${axle_y_offset*-1} ${axle_z_offset}" rpy="0 0 ${PI}" />
-      </xacro:w200_track>
-    </xacro:if>
-    <!-- Virtual Mounting Point -->
-    <link name="${tf_prefix}default_mount"></link>
-    <joint name="${tf_prefix}default_mount_joint" type="fixed">
-      <origin xyz="0 0 0.27218" rpy="0 0 0" />
-      <parent link="${tf_prefix}chassis_link" />
-      <child link="${tf_prefix}default_mount" />
-    </joint>
-    <!-- Internal IMU -->
-    <link name="${tf_prefix}imu_0_link">
-      <inertial>
-        <mass value="0.001" />
-        <origin xyz="0 0 0" rpy="0 0 0" />
-        <inertia ixx="${dummy_inertia}" ixy="0.0" ixz="0.0" iyy="${dummy_inertia}" iyz="0.0"
-          izz="${dummy_inertia}" />
-      </inertial>
-    </link>
-    <joint name="imu_joint" type="fixed">
-      <parent link="${tf_prefix}chassis_link" />
-      <child link="${tf_prefix}imu_0_link" />
-    </joint>
-    <!-- GPS -->
-    <link name="${tf_prefix}gps_0_link">
-      <inertial>
-        <mass value="0.001" />
-        <origin xyz="0 0.05 0" rpy="0 0 0" />
-        <inertia ixx="${dummy_inertia}" ixy="0.0" ixz="0.0" iyy="${dummy_inertia}" iyz="0.0"
-          izz="${dummy_inertia}" />
-      </inertial>
-    </link>
-    <joint name="gps_joint" type="fixed">
-      <parent link="${tf_prefix}chassis_link" />
-      <child link="${tf_prefix}gps_0_link" />
-    </joint>
-    <!-- ROS2 controls -->
-    <xacro:include filename="$(find wilbur_description)/urdf/w200.ros2_control.xacro" />
-    <!-- todo do we need a ns/name paradigm for ros2 control system plugins for multiple/namespacing-->
-    <xacro:if value="${generate_ros2_control_tag}">
-      <xacro:w200_ros2_control
-        name="w200_ros2_control"
-        use_fake_hardware="${use_fake_hardware}"
-        sim_ignition="${sim_ignition}"
-        tf_prefix="${tf_prefix}"
-      />
-    </xacro:if>
-    <!-- w200_gz - plugins specific for the w200 for gazebo -->
-    <xacro:if value="${sim_ignition}">
-      <xacro:include filename="$(find wilbur_gz)/urdf/w200_gz.xacro" />
-      <xacro:w200_gz
-        tf_prefix="${tf_prefix}"
-        wheel_radius="${wheel_radius}"
-        imu_link_name="imu_0_link"
-        gps_link_name="gps_0_link"
-        ns="${ns}">
-      </xacro:w200_gz>
-    </xacro:if>
-  </xacro:macro>
+<?xml version="1.0"?>
+<robot name="w200" xmlns:xacro="http://ros.org/wiki/xacro">
+  <xacro:arg name="tf_prefix" default="" />
+  <xacro:arg name="ns" default="" />
+  <xacro:arg name="sim_ignition" default="false" />
+  <xacro:arg name="use_fake_hardware" default="true" /> <!-- todo look into calling this use_mock_hardware to be forward leaning-->
+  <xacro:arg name="generate_ros2_control_tag" default="true" /> <!-- for mujoco cannot have this -->
+  <xacro:include filename="$(find wilbur_description)/urdf/w200_macro.urdf.xacro" />
+  <xacro:w200
+    wheel="default"
+    tf_prefix="$(arg tf_prefix)"
+    sim_ignition="$(arg sim_ignition)"
+    use_fake_hardware="$(arg use_fake_hardware)"
+    ns="$(arg ns)"
+    generate_ros2_control_tag="$(arg generate_ros2_control_tag)"
+  />
 </robot>

File: wilbur_description/urdf/wilbur.urdf.xacro (robot description, xacro)
@@ -11,5 +11,5 @@
     <!-- todo - reduce the dependency on clear_path_description-->
     <xacro:include filename="$(find clearpath_platform_description)/urdf/common.urdf.xacro" />
-    <xacro:include filename="$(find wilbur_description)/urdf/w200.urdf.xacro" />
+    <xacro:include filename="$(find wilbur_description)/urdf/w200_macro.urdf.xacro" />
     <xacro:include
         filename="$(find wilbur_description)/urdf/attachments/bulkhead.urdf.xacro" />
@@ -17,5 +17,5 @@
     <xacro:include filename="$(find clearpath_platform_description)/urdf/links/mesh.urdf.xacro" />
     <xacro:include filename="$(find wilbur_description)/urdf/gen_mesh.xacro"/>
-    <xacro:include filename="$(find ur_description)/urdf/ur_macro.xacro" />
+    <xacro:include filename="$(find wilbur_description)/urdf/wilbur_ur10e_macro.urdf.xacro" />
     <!-- if ignition or gazebo - need to use absolute paths instead of relative-->
     <xacro:property name="force_abs_paths" value="$(arg sim_ignition)" scope="global"/>
@@ -48,13 +48,8 @@
       <origin xyz="0 0 0" rpy="0 0 0" />
     </joint>
-    <!-- todo - reduce dependency on clearpath platform description building macros -->
-    <!-- todo - add tf prefix-->
-    <xacro:frame name="arm_0_end_effector" parent_link="arm_0_tool0">
-        <origin xyz="0.0 0.0 0.0" rpy="0.0 0.0 0.0" />
-    </xacro:frame>
-    <!-- Manipulators -->
+        <!-- Manipulators -->
     <xacro:property name="initial_positions_file"  value="$(arg wilbur_ur10e_initial_positions)"  />
     <!-- todo expose out args for hardware-->
-    <xacro:ur_robot
+    <xacro:wilbur_ur10e
         name="arm_0_"
         tf_prefix="$(arg tf_prefix)arm_0_"
@@ -63,12 +58,8 @@
         sim_ignition="$(arg sim_ignition)"
         initial_positions="${xacro.load_yaml(initial_positions_file)}"
-        joint_limits_parameters_file="$(find ur_description)/config/ur10e/joint_limits.yaml"
-        kinematics_parameters_file="$(find ur_description)/config/ur10e/default_kinematics.yaml"
-        physical_parameters_file="$(find ur_description)/config/ur10e/physical_parameters.yaml"
-        visual_parameters_file="$(find ur_description)/config/ur10e/visual_parameters.yaml"
         generate_ros2_control_tag="$(arg generate_ros2_control_tag)"
       >
       <origin xyz="0.0 0.0 0.0" rpy="0.0 0.0 0.0" />
-    </xacro:ur_robot>
+    </xacro:wilbur_ur10e>
     <!-- arm_0_gripper -->
     <!--xacro:robotiq_2f_85
