Commit message: Corrected the spelling of Wilbur

File: wilbur_description/urdf/diff_unit.urdf.xacro (robot description, xacro)
@@ -23,5 +23,5 @@
         <origin xyz="0 0 0" rpy="0 0 ${flip*PI/2}" />
         <geometry>
-          <mesh filename="package://wilber_description/meshes/fenders.stl" />
+          <mesh filename="package://wilbur_description/meshes/fenders.stl" />
         </geometry>
         <material name="${warthog_color}" />
@@ -30,5 +30,5 @@
         <origin xyz="0 0 0" rpy="0 0 ${flip*PI/2}" />
         <geometry>
-          <mesh filename="package://wilber_description/meshes/fenders.stl" />
+          <mesh filename="package://wilbur_description/meshes/fenders.stl" />
         </geometry>
       </collision>
@@ -36,5 +36,5 @@
         <origin xyz="0 0 0" rpy="0 0 ${flip*PI/2}" />
         <geometry>
-          <mesh filename="package://wilber_description/meshes/rocker.stl" />
+          <mesh filename="package://wilbur_description/meshes/rocker.stl" />
         </geometry>
         <material name="clearpath_black" />
@@ -54,5 +54,5 @@
         <origin xyz="0 ${flip*-0.0244} 0" rpy="0 0 0" />
         <geometry>
-          <mesh filename="package://wilber_description/meshes/light.stl" />
+          <mesh filename="package://wilbur_description/meshes/light.stl" />
         </geometry>
         <material name="clearpath_white" />
@@ -78,5 +78,5 @@
         <origin xyz="0 ${flip*-0.0244} 0" rpy="0 0 ${flip*PI}" />
         <geometry>
-          <mesh filename="package://wilber_description/meshes/light.stl" />
+          <mesh filename="package://wilbur_description/meshes/light.stl" />
         </geometry>
         <material name="clearpath_red" />

File: wilbur_description/urdf/w200.urdf.xacro (robot description, xacro)
@@ -9,11 +9,11 @@
                 ns">
     <xacro:arg name="gazebo_controllers"
-      default="$(find wilber_deploy)/config/${tf_prefix}control.yaml" />
+      default="$(find wilbur_deploy)/config/${tf_prefix}control.yaml" />
     <xacro:arg name="use_platform_controllers" default="true" />
     <!-- Include URDF/XACRO Files -->
-    <xacro:include filename="$(find wilber_description)/urdf/wheels/track.urdf.xacro" />
-    <xacro:include filename="$(find wilber_description)/urdf/wheels/wheel.urdf.xacro" />
+    <xacro:include filename="$(find wilbur_description)/urdf/wheels/track.urdf.xacro" />
+    <xacro:include filename="$(find wilbur_description)/urdf/wheels/wheel.urdf.xacro" />
     <xacro:property name="PI" value="3.1415926535897931" />
-    <xacro:include filename="$(find wilber_description)/urdf/diff_unit.urdf.xacro" />
+    <xacro:include filename="$(find wilbur_description)/urdf/diff_unit.urdf.xacro" />
     <!-- Colors: yellow, orange, olive, sand -->
     <xacro:property name="warthog_color" value="${'warthog_'+color}" />
@@ -68,5 +68,5 @@
         <origin xyz="0 0 0" rpy="0 0 0" />
         <geometry>
-          <mesh filename="package://wilber_description/meshes/chassis.stl" />
+          <mesh filename="package://wilbur_description/meshes/chassis.stl" />
         </geometry>
         <material name="clearpath_black">
@@ -77,5 +77,5 @@
         <origin xyz="0 0 0" rpy="0 0 0" />
         <geometry>
-          <mesh filename="package://wilber_description/meshes/e-stop.stl" />
+          <mesh filename="package://wilbur_description/meshes/e-stop.stl" />
         </geometry>
         <material name="clearpath_red">
@@ -86,5 +86,5 @@
         <origin xyz="0 0 0" rpy="0 0 0" />
         <geometry>
-          <mesh filename="package://wilber_description/meshes/chassis-collision.stl" />
+          <mesh filename="package://wilbur_description/meshes/chassis-collision.stl" />
         </geometry>
       </collision>
@@ -97,5 +97,5 @@
         <origin xyz="0 0 0" rpy="0 0 0" />
         <geometry>
-          <mesh filename="package://wilber_description/meshes/diff-link.stl" />
+          <mesh filename="package://wilbur_description/meshes/diff-link.stl" />
         </geometry>
         <material name="clearpath_light_grey" />
@@ -104,5 +104,5 @@
         <origin xyz="0 0 0" rpy="0 0 0" />
         <geometry>
-          <mesh filename="package://wilber_description/meshes/susp-link.stl" />
+          <mesh filename="package://wilbur_description/meshes/susp-link.stl" />
         </geometry>
         <material name="clearpath_light_grey" />
@@ -111,5 +111,5 @@
         <origin xyz="0 0 0" rpy="0 0 0" />
         <geometry>
-          <mesh filename="package://wilber_description/meshes/susp-link.stl" />
+          <mesh filename="package://wilbur_description/meshes/susp-link.stl" />
         </geometry>
         <material name="clearpath_light_grey" />
@@ -185,5 +185,5 @@
     </xacro:if>
     <!-- Gazebo Controller -->
-    <xacro:include filename="$(find wilber_description)/urdf/gazebo.urdf.xacro" />
+    <xacro:include filename="$(find wilbur_description)/urdf/gazebo.urdf.xacro" />
     <!-- ROS2 controls -->
     <xacro:if value="$(arg use_platform_controllers)">

File: wilbur_description/urdf/wheels/track.urdf.xacro (robot description, xacro)
@@ -7,5 +7,5 @@
         <origin xyz="0 0 0" rpy="0 0 0" />
         <geometry>
-          <mesh filename="package://wilber_description/meshes/tracks.dae" />
+          <mesh filename="package://wilbur_description/meshes/tracks.dae" />
         </geometry>
         <material name="clearpath_dark_grey" />

File: wilbur_description/urdf/wheels/wheel.urdf.xacro (robot description, xacro)
@@ -16,5 +16,5 @@
         <origin xyz="0 0 0" rpy="0 0 ${PI/2}" />
         <geometry>
-          <mesh filename="package://wilber_description/meshes/wheel.stl" />
+          <mesh filename="package://wilbur_description/meshes/wheel.stl" />
         </geometry>
         <material name="clearpath_dark_grey" />

File: wilbur_description/urdf/wilbur.urdf.xacro (robot description, xacro)
@@ -1,4 +1,4 @@
 <?xml version="1.0"?>
-<robot name="wilber" xmlns:xacro="http://ros.org/wiki/xacro">
+<robot name="wilbur" xmlns:xacro="http://ros.org/wiki/xacro">
     <xacro:arg name="tf_prefix" default="" />
     <xacro:arg name="ns" default="" />
@@ -7,8 +7,8 @@
     <!-- Includes -->
     <xacro:include filename="$(find clearpath_platform_description)/urdf/common.urdf.xacro" />
-    <xacro:include filename="$(find wilber_description)/urdf/w200.urdf.xacro" />
+    <xacro:include filename="$(find wilbur_description)/urdf/w200.urdf.xacro" />
     <!-- Attachments -->
     <xacro:include
-        filename="$(find wilber_description)/urdf/attachments/bulkhead.urdf.xacro" />
+        filename="$(find wilbur_description)/urdf/attachments/bulkhead.urdf.xacro" />
     <xacro:bulkhead name="bulkhead" model="$(arg tf_prefix)arm_plate"
         parent_link="$(arg tf_prefix)default_mount"

Commit message: Added dependency on clearpath_platform_description and using that package for meshes, rather than keeping copies here

File: wilbur_description/urdf/diff_unit.urdf.xacro (robot description, xacro)
@@ -23,5 +23,5 @@
         <origin xyz="0 0 0" rpy="0 0 ${flip*PI/2}" />
         <geometry>
-          <mesh filename="package://wilbur_description/meshes/fenders.stl" />
+          <mesh filename="package://clearpath_platform_description/meshes/w200/fenders.stl" />
         </geometry>
         <material name="${warthog_color}" />
@@ -30,5 +30,5 @@
         <origin xyz="0 0 0" rpy="0 0 ${flip*PI/2}" />
         <geometry>
-          <mesh filename="package://wilbur_description/meshes/fenders.stl" />
+          <mesh filename="package://clearpath_platform_description/meshes/w200/fenders.stl" />
         </geometry>
       </collision>
@@ -36,5 +36,5 @@
         <origin xyz="0 0 0" rpy="0 0 ${flip*PI/2}" />
         <geometry>
-          <mesh filename="package://wilbur_description/meshes/rocker.stl" />
+          <mesh filename="package://clearpath_platform_description/meshes/w200/rocker.stl" />
         </geometry>
         <material name="clearpath_black" />
@@ -54,5 +54,5 @@
         <origin xyz="0 ${flip*-0.0244} 0" rpy="0 0 0" />
         <geometry>
-          <mesh filename="package://wilbur_description/meshes/light.stl" />
+          <mesh filename="package://clearpath_platform_description/meshes/w200/light.stl" />
         </geometry>
         <material name="clearpath_white" />
@@ -78,5 +78,5 @@
         <origin xyz="0 ${flip*-0.0244} 0" rpy="0 0 ${flip*PI}" />
         <geometry>
-          <mesh filename="package://wilbur_description/meshes/light.stl" />
+          <mesh filename="package://clearpath_platform_description/meshes/w200/light.stl" />
         </geometry>
         <material name="clearpath_red" />

File: wilbur_description/urdf/w200.urdf.xacro (robot description, xacro)
@@ -68,5 +68,5 @@
         <origin xyz="0 0 0" rpy="0 0 0" />
         <geometry>
-          <mesh filename="package://wilbur_description/meshes/chassis.stl" />
+          <mesh filename="package://clearpath_platform_description/meshes/w200/chassis.stl" />
         </geometry>
         <material name="clearpath_black">
@@ -77,5 +77,5 @@
         <origin xyz="0 0 0" rpy="0 0 0" />
         <geometry>
-          <mesh filename="package://wilbur_description/meshes/e-stop.stl" />
+          <mesh filename="package://clearpath_platform_description/meshes/w200/e-stop.stl" />
         </geometry>
         <material name="clearpath_red">
@@ -86,5 +86,6 @@
         <origin xyz="0 0 0" rpy="0 0 0" />
         <geometry>
-          <mesh filename="package://wilbur_description/meshes/chassis-collision.stl" />
+          <mesh
+            filename="package://clearpath_platform_description/meshes/w200/chassis-collision.stl" />
         </geometry>
       </collision>
@@ -97,5 +98,5 @@
         <origin xyz="0 0 0" rpy="0 0 0" />
         <geometry>
-          <mesh filename="package://wilbur_description/meshes/diff-link.stl" />
+          <mesh filename="package://clearpath_platform_description/meshes/w200/diff-link.stl" />
         </geometry>
         <material name="clearpath_light_grey" />
@@ -104,5 +105,5 @@
         <origin xyz="0 0 0" rpy="0 0 0" />
         <geometry>
-          <mesh filename="package://wilbur_description/meshes/susp-link.stl" />
+          <mesh filename="package://clearpath_platform_description/meshes/w200/susp-link.stl" />
         </geometry>
         <material name="clearpath_light_grey" />
@@ -111,5 +112,5 @@
         <origin xyz="0 0 0" rpy="0 0 0" />
         <geometry>
-          <mesh filename="package://wilbur_description/meshes/susp-link.stl" />
+          <mesh filename="package://clearpath_platform_description/meshes/w200/susp-link.stl" />
         </geometry>
         <material name="clearpath_light_grey" />

File: wilbur_description/urdf/wheels/wheel.urdf.xacro (robot description, xacro)
@@ -16,5 +16,5 @@
         <origin xyz="0 0 0" rpy="0 0 ${PI/2}" />
         <geometry>
-          <mesh filename="package://wilbur_description/meshes/wheel.stl" />
+          <mesh filename="package://clearpath_platform_description/meshes/w200/wheel.stl" />
         </geometry>
         <material name="clearpath_dark_grey" />

Commit message: moved the last missing gazebo stuff to wilbur_gz

File: wilbur_description/urdf/diff_unit.urdf.xacro (robot description, xacro)
@@ -64,14 +64,4 @@
       <origin xyz="0 0 0" rpy="0 0 0" />
     </joint>
-    <gazebo reference="${side}_diff_unit_headlight_link">
-      <visual>
-        <material>
-          <ambient>0.9 0.9 0.9 1</ambient>
-          <diffuse>0.9 0.9 0.9 1</diffuse>
-          <specular>0.9 0.9 0.9 1</specular>
-          <emissive>0.9 0.9 0.9 1</emissive>
-        </material>
-      </visual>
-    </gazebo>
     <link name="${tf_prefix}${side}_diff_unit_taillight_link">
       <visual>
@@ -88,23 +78,4 @@
       <origin xyz="0 0 0" rpy="0 0 0" />
     </joint>
-    <gazebo reference="${tf_prefix}${side}_diff_unit_taillight_link">
-      <visual>
-        <material>
-          <ambient>0.9 0 0 1</ambient>
-          <diffuse>0.9 0 0 1</diffuse>
-          <specular>0.9 0 0 1</specular>
-          <emissive>0.9 0 0 1</emissive>
-        </material>
-      </visual>
-    </gazebo>
-    <gazebo reference="${tf_prefix}${side}_diff_unit_link">
-      <selfCollide>false</selfCollide>
-      <visual>
-        <material>
-          <specular>0.1 0.1 0.1 1</specular>
-          <emissive>0 0 0 0</emissive>
-        </material>
-      </visual>
-    </gazebo>
   </xacro:macro>
 </robot>

File: wilbur_description/urdf/wheels/track.urdf.xacro (robot description, xacro)
@@ -50,11 +50,4 @@
       <axis xyz="0 1 0" />
     </joint>
-    <gazebo reference="${tf_prefix}${prefix}_${side}_wheel_link">
-      <selfCollide>false</selfCollide>
-      <mu1>0.5</mu1>
-      <mu2>0.5</mu2>
-      <fdir1 value="1 0 0" />
-      <material>Gazebo/DarkGrey</material>
-    </gazebo>
   </xacro:macro>
 </robot>

File: wilbur_description/urdf/wheels/wheel.urdf.xacro (robot description, xacro)
@@ -33,15 +33,4 @@
       <axis xyz="0 1 0" />
     </joint>
-    <gazebo reference="${tf_prefix}${prefix}_${side}_wheel_link">
-      <selfCollide>false</selfCollide>
-      <!-- values from
-      https://github.com/unmannedlab/cartographer/blob/main/src/platform_description/urdf/warthog.urdf.xacro-->
-      <mu1>1.0</mu1>
-      <mu2>1.0</mu2>
-      <kp value="10000000.0" />
-      <kd value="1.0" />
-      <fdir1 value="1 0 0" />
-      <material>Gazebo/DarkGrey</material>
-    </gazebo>
   </xacro:macro>
 </robot>

File: wilbur_gz/urdf/w200_gz.xacro (robot description, xacro)
@@ -1,4 +1,57 @@
 <?xml version="1.0"?>
 <robot xmlns:xacro="http://ros.org/wiki/xacro">
+  <xacro:macro name="wheel_gz" params="prefix side tf_prefix">
+    <gazebo reference="${tf_prefix}${prefix}_${side}_wheel_link">
+      <selfCollide>false</selfCollide>
+      <!-- values from
+      https://github.com/unmannedlab/cartographer/blob/main/src/platform_description/urdf/warthog.urdf.xacro-->
+      <mu1>1.0</mu1>
+      <mu2>1.0</mu2>
+      <kp value="10000000.0" />
+      <kd value="1.0" />
+      <fdir1 value="1 0 0" />
+      <material>Gazebo/DarkGrey</material>
+    </gazebo>
+  </xacro:macro>
+  <xacro:macro name="track_gz" params="prefix side tf_prefix">
+      <gazebo reference="${tf_prefix}${prefix}_${side}_wheel_link">
+      <selfCollide>false</selfCollide>
+      <mu1>0.5</mu1>
+      <mu2>0.5</mu2>
+      <fdir1 value="1 0 0" />
+      <material>Gazebo/DarkGrey</material>
+    </gazebo>
+  </xacro:macro>
+  <xacro:macro name="diff_unit_gz" params="side tf_prefix">
+    <gazebo reference="${tf_prefix}${side}_diff_unit_taillight_link">
+      <visual>
+        <material>
+          <ambient>0.9 0 0 1</ambient>
+          <diffuse>0.9 0 0 1</diffuse>
+          <specular>0.9 0 0 1</specular>
+          <emissive>0.9 0 0 1</emissive>
+        </material>
+      </visual>
+    </gazebo>
+    <gazebo reference="${tf_prefix}${side}_diff_unit_headlight_link">
+      <visual>
+        <material>
+          <ambient>0.9 0.9 0.9 1</ambient>
+          <diffuse>0.9 0.9 0.9 1</diffuse>
+          <specular>0.9 0.9 0.9 1</specular>
+          <emissive>0.9 0.9 0.9 1</emissive>
+        </material>
+      </visual>
+    </gazebo>
+    <gazebo reference="${tf_prefix}${side}_diff_unit_link">
+      <selfCollide>false</selfCollide>
+      <visual>
+        <material>
+          <specular>0.1 0.1 0.1 1</specular>
+          <emissive>0 0 0 0</emissive>
+        </material>
+      </visual>
+    </gazebo>
+  </xacro:macro>
   <!-- macro for gazebo plugins specific for the w200-->
   <xacro:macro name="w200_gz"
@@ -31,4 +84,8 @@
       </sensor>
     </gazebo>
+    <xacro:wheel_gz prefix="front" side="left" tf_prefix="${tf_prefix}"/>
+    <xacro:wheel_gz prefix="front" side="right" tf_prefix="${tf_prefix}"/>
+    <xacro:wheel_gz prefix="rear" side="left" tf_prefix="${tf_prefix}"/>
+    <xacro:wheel_gz prefix="rear" side="right" tf_prefix="${tf_prefix}"/>
     <gazebo>
       <plugin filename="libignition-gazebo-wheel-slip-system.so"
@@ -60,4 +117,6 @@
       </plugin>
     </gazebo>
+    <xacro:diff_unit_gz side="right" tf_prefix="${tf_prefix}"/>
+    <xacro:diff_unit_gz side="left" tf_prefix="${tf_prefix}"/>
   </xacro:macro>
 </robot>
