Commit message: deleting the controller manager because they are not used anywhere and also because they redeclare robot_description

File: wilbur_description/urdf/w200_macro.urdf.xacro (robot description, xacro)
@@ -13,5 +13,6 @@
     <xacro:include filename="$(find wilbur_description)/urdf/wheels/track.urdf.xacro" />
     <xacro:include filename="$(find wilbur_description)/urdf/wheels/wheel.urdf.xacro" />
-    <xacro:property name="PI" value="3.1415926535897931" /> <!--pi is build in - replace with lowercase pi throughout and remove property -->
+    <xacro:property name="PI" value="3.1415926535897931" /> <!--pi
+    is build in - replace with lowercase pi throughout and remove property -->
     <xacro:include filename="$(find wilbur_description)/urdf/diff_unit.urdf.xacro" />
     <!-- Colors: yellow, orange, olive, sand -->
@@ -67,5 +68,6 @@
         <origin xyz="0 0 0" rpy="0 0 0" />
         <geometry>
-          <xacro:gen_mesh force_abs_path="${force_abs_paths}" pkg_name="wilbur_description" file_path="meshes/w200/chassis.stl" />
+          <xacro:gen_mesh force_abs_path="${force_abs_paths}" pkg_name="wilbur_description"
+            file_path="meshes/w200/chassis.stl" />
         </geometry>
         <material name="clearpath_black">
@@ -76,5 +78,6 @@
         <origin xyz="0 0 0" rpy="0 0 0" />
         <geometry>
-          <xacro:gen_mesh force_abs_path="${force_abs_paths}" pkg_name="wilbur_description" file_path="meshes/w200/e-stop.stl" />
+          <xacro:gen_mesh force_abs_path="${force_abs_paths}" pkg_name="wilbur_description"
+            file_path="meshes/w200/e-stop.stl" />
         </geometry>
         <material name="clearpath_red">
@@ -85,5 +88,6 @@
         <origin xyz="0 0 0" rpy="0 0 0" />
         <geometry>
-          <xacro:gen_mesh force_abs_path="${force_abs_paths}" pkg_name="wilbur_description" file_path="meshes/w200/chassis-collision.stl" />
+          <xacro:gen_mesh force_abs_path="${force_abs_paths}" pkg_name="wilbur_description"
+            file_path="meshes/w200/chassis-collision.stl" />
         </geometry>
       </collision>
@@ -96,5 +100,6 @@
         <origin xyz="0 0 0" rpy="0 0 0" />
         <geometry>
-          <xacro:gen_mesh force_abs_path="${force_abs_paths}" pkg_name="wilbur_description" file_path="meshes/w200/diff-link.stl" />
+          <xacro:gen_mesh force_abs_path="${force_abs_paths}" pkg_name="wilbur_description"
+            file_path="meshes/w200/diff-link.stl" />
         </geometry>
         <material name="clearpath_light_grey" />
@@ -103,5 +108,6 @@
         <origin xyz="0 0 0" rpy="0 0 0" />
         <geometry>
-          <xacro:gen_mesh force_abs_path="${force_abs_paths}" pkg_name="wilbur_description" file_path="meshes/w200/susp-link.stl" />
+          <xacro:gen_mesh force_abs_path="${force_abs_paths}" pkg_name="wilbur_description"
+            file_path="meshes/w200/susp-link.stl" />
         </geometry>
         <material name="clearpath_light_grey" />
@@ -110,5 +116,6 @@
         <origin xyz="0 0 0" rpy="0 0 0" />
         <geometry>
-          <xacro:gen_mesh force_abs_path="${force_abs_paths}" pkg_name="wilbur_description" file_path="meshes/w200/susp-link.stl" />
+          <xacro:gen_mesh force_abs_path="${force_abs_paths}" pkg_name="wilbur_description"
+            file_path="meshes/w200/susp-link.stl" />
         </geometry>
         <material name="clearpath_light_grey" />
@@ -185,5 +192,6 @@
     <!-- ROS2 controls -->
     <xacro:include filename="$(find wilbur_description)/urdf/w200.ros2_control.xacro" />
-    <!-- todo do we need a ns/name paradigm for ros2 control system plugins for multiple/namespacing-->
+    <!-- todo do we need a ns/name paradigm for ros2 control system plugins for
+    multiple/namespacing-->
     <xacro:if value="${generate_ros2_control_tag}">
       <xacro:w200_ros2_control
