Commit message: Add stub hande to description and moveit config

File: wilbur_description/urdf/wilbur_ur10e_macro.urdf.xacro (robot description, xacro)
@@ -13,6 +13,6 @@
     <xacro:include filename="$(find ur_description)/urdf/ur_macro.xacro" />
     <xacro:include filename="$(find clearpath_platform_description)/urdf/links/frame.urdf.xacro" />
-    <!-- todo - add tf prefix -->
-    <!-- todo - remove clearpath frame -->
+    <xacro:include filename="$(find dextivr_hande_description)/urdf/dextivr_hande.xacro" />
+    <!-- todo - add tf prefix-->
     <xacro:frame name="arm_0_end_effector" parent_link="arm_0_tool0">
         <origin xyz="0.0 0.0 0.0" rpy="0.0 0.0 0.0" />
@@ -36,7 +36,15 @@
       <xacro:insert_block name="origin" />
     </xacro:ur_robot>
-    <!-- todo - add gripper-->
-    <!-- todo add grasp link in the moveit pro orientation
-    https://docs.picknik.ai/how_to/configuration_tutorials/configure_custom_robot/#configuring-grasp-preview -->
+    <!-- Hand-e -->
+    <!-- TODO: Actually attach it using mounting hardware -->
+    <xacro:dextivr_hande
+      name="dextivr_hande"
+      tf_prefix="${tf_prefix}"
+      parent="${tf_prefix}end_effector_link"
+      use_fake_hardware="${use_fake_hardware}"
+      marker_opacity="0.5"
+      finger_xacro="fngr_v6">
+      <origin xyz="0 0 0" rpy="0 0 ${radians(-90)}"/>
+    </xacro:dextivr_hande>
   </xacro:macro>
 </robot>

Commit message: removed the hande addition

File: wilbur_description/urdf/wilbur_ur10e_macro.urdf.xacro (robot description, xacro)
@@ -7,49 +7,21 @@
             *origin
             parent:='world'
-            use_fake_hardware:=false
-            sim_ignition:=false
             initial_positions='$(find wilbur_deploy)/config/ur_initial_positions.yaml'
-            gripper_com_port:=/dev/ttyUSB0
-            generate_ros2_control_tag:=true">
+            ">
     <xacro:include filename="$(find ur_description)/urdf/ur_macro.xacro" />
     <xacro:include filename="$(find wilbur_description)/urdf/links/frame.urdf.xacro" />
-    <xacro:include filename="$(find dextivr_hande_description)/urdf/dextivr_hande.xacro" />
-    <!-- todo - add tf prefix-->
-    <xacro:frame name="arm_0_end_effector" parent_link="arm_0_tool0">
-        <origin xyz="0.0 0.0 0.0" rpy="0.0 0.0 0.0" />
-    </xacro:frame>
     <!-- Manipulators -->
-    <!-- TODO ur_robot macro changed and we lost a bunch of important args (use_fake_hardware, initial_positions, generate_ros2_control_tag, etc.)
-         this seems super important and we need to figure out what the implications are and/or how to get those back -->
-    <xacro:property name="initial_positions_file"  value="$(arg wilbur_ur10e_initial_positions)"  />
-    <!-- todo expose out args for hardware-->
+    <xacro:property name="initial_positions_file" value="$(arg wilbur_ur10e_initial_positions)" />
     <xacro:ur_robot
-        name="${name}"
-        tf_prefix="${tf_prefix}"
-        parent="${parent}"
-        joint_limits_parameters_file="$(find ur_description)/config/ur10e/joint_limits.yaml"
-        kinematics_parameters_file="$(find ur_description)/config/ur10e/default_kinematics.yaml"
-        physical_parameters_file="$(find ur_description)/config/ur10e/physical_parameters.yaml"
-        visual_parameters_file="$(find ur_description)/config/ur10e/visual_parameters.yaml"
-      >
+      name="${name}"
+      tf_prefix="${tf_prefix}"
+      parent="${parent}"
+      joint_limits_parameters_file="$(find ur_description)/config/ur10e/joint_limits.yaml"
+      kinematics_parameters_file="$(find ur_description)/config/ur10e/default_kinematics.yaml"
+      physical_parameters_file="$(find ur_description)/config/ur10e/physical_parameters.yaml"
+      visual_parameters_file="$(find ur_description)/config/ur10e/visual_parameters.yaml"
+    >
       <xacro:insert_block name="origin" />
     </xacro:ur_robot>
-    <!-- Hand-e -->
-    <!-- TODO: Update EE stack to match the physical hardware -->
-    <!-- https://js-er-code.jsc.nasa.gov/imetro/robots/wilbur/wilbur/-/issues/34 -->
-    <!--       There is not place or actual end effector stack, this is just here as a -->
-    <!--       placeholder for the control stack. -->
-    <xacro:dextivr_hande
-      name="dextivr_hande"
-      tf_prefix="${tf_prefix}"
-      parent="${tf_prefix}end_effector_link"
-      sim_ignition="${sim_ignition}"
-      use_fake_hardware="${use_fake_hardware}"
-      fake_sensor_commands="false"
-      com_port="${gripper_com_port}"
-      marker_opacity="0.5"
-      finger_xacro="fngr_v6">
-      <origin xyz="0 0 0" rpy="0 0 ${radians(-90)}"/>
-    </xacro:dextivr_hande>
   </xacro:macro>
 </robot>
