Commit message: added control_frame

File: wilbur_description/urdf/wilbur.urdf.xacro (robot description, xacro)
@@ -8,7 +8,14 @@
     <xacro:include filename="$(find clearpath_platform_description)/urdf/common.urdf.xacro" />
     <xacro:include filename="$(find wilbur_description)/urdf/w200.urdf.xacro" />
-    <!-- Attachments -->
     <xacro:include
         filename="$(find wilbur_description)/urdf/attachments/bulkhead.urdf.xacro" />
+    <xacro:include filename="$(find clearpath_platform_description)/urdf/links/frame.urdf.xacro" />
+    <xacro:include filename="$(find clearpath_platform_description)/urdf/links/mesh.urdf.xacro" />
+    <!-- Attachments -->
+    <!-- Links -->
+    <xacro:mesh name="control_frame" parent_link="default_mount"
+        visual="package://wilbur_description/meshes/control_frame.stl">
+        <origin xyz="0.0 0.0 0.0" rpy="0.0 0.0 0.0" />
+    </xacro:mesh>
     <xacro:bulkhead name="bulkhead" model="$(arg tf_prefix)arm_plate"
         parent_link="$(arg tf_prefix)default_mount"
@@ -16,4 +23,7 @@
         <origin xyz="0.0 0.0 0.0" rpy="0.0 0.0 0.0" />
     </xacro:bulkhead>
+    <!--xacro:frame name="arm_0_end_effector" parent_link="arm_0_tool0">
+        <origin xyz="0.0 0.0 0.0" rpy="0.0 0.0 0.0" />
+    </xacro:frame-->
     <xacro:w200
         tf_prefix="$(arg tf_prefix)"

Commit message: Added Ur10e model -- still need to verify controls work

File: wilbur_description/urdf/wilbur.urdf.xacro (robot description, xacro)
@@ -3,6 +3,9 @@
     <xacro:arg name="tf_prefix" default="" />
     <xacro:arg name="ns" default="" />
-    <xacro:arg name="is_sim" default="true" />
+    <xacro:arg
+        name="is_sim" default="true" />
     <xacro:arg name="parent" default="world" />
+    <xacro:arg
+        name="ur_type" default="ur10e" />
     <!-- Includes -->
     <xacro:include filename="$(find clearpath_platform_description)/urdf/common.urdf.xacro" />
@@ -12,18 +15,55 @@
     <xacro:include filename="$(find clearpath_platform_description)/urdf/links/frame.urdf.xacro" />
     <xacro:include filename="$(find clearpath_platform_description)/urdf/links/mesh.urdf.xacro" />
+    <!--xacro:include
+        filename="$(find clearpath_manipulators_description)/urdf/arm/universal_robots.urdf.xacro" /-->
+    <xacro:include
+        filename="$(find ur_description)/urdf/ur_macro.xacro" />
+    <!--xacro:include
+        filename="$(find ur_description)/urdf/gripper/robotiq_2f_85.urdf.xacro" /-->
     <!-- Attachments -->
-    <!-- Links -->
-    <xacro:mesh name="control_frame" parent_link="default_mount"
-        visual="package://wilbur_description/meshes/control_frame.stl">
-        <origin xyz="0.0 0.0 0.0" rpy="0.0 0.0 0.0" />
-    </xacro:mesh>
-    <xacro:bulkhead name="bulkhead" model="$(arg tf_prefix)arm_plate"
+    <xacro:bulkhead
+        name="bulkhead"
+        model="$(arg tf_prefix)arm_plate"
         parent_link="$(arg tf_prefix)default_mount"
         tf_prefix="$(arg tf_prefix)">
         <origin xyz="0.0 0.0 0.0" rpy="0.0 0.0 0.0" />
     </xacro:bulkhead>
+    <!-- Links -->
+    <xacro:mesh
+        name="control_frame"
+        parent_link="default_mount"
+        visual="package://wilbur_description/meshes/control_frame.stl">
+        <origin xyz="0.0 0.0 0.0" rpy="0.0 0.0 0.0" />
+    </xacro:mesh>
     <!--xacro:frame name="arm_0_end_effector" parent_link="arm_0_tool0">
         <origin xyz="0.0 0.0 0.0" rpy="0.0 0.0 0.0" />
     </xacro:frame-->
+    <!-- Manipulators -->
+    <!-- arm_0 -->
+    <!--xacro:universal_robots name="arm_0"
+        parent_link="arm_plate_mount"
+        robot_ip="192.168.131.40"
+        ur_type="ur10e"
+        initial_positions_file="$(find wilbur_description)/config/arm0_initial_positions.yaml"
+        sim_ignition="true"
+        use_fake_hardware="true">
+        <origin xyz="0.0 0.0 0.0" rpy="0.0 0.0 0.0" />
+    </xacro:universal_robots-->
+    <xacro:ur_robot
+        name="arm_0_"
+        tf_prefix="$(arg tf_prefix)arm_0_"
+        parent="arm_plate_mount"
+        sim_ignition="true"
+        joint_limits_parameters_file="$(find ur_description)/config/$(arg ur_type)/joint_limits.yaml"
+        kinematics_parameters_file="$(find ur_description)/config/$(arg ur_type)/default_kinematics.yaml"
+        physical_parameters_file="$(find ur_description)/config/$(arg ur_type)/physical_parameters.yaml"
+        visual_parameters_file="$(find ur_description)/config/$(arg ur_type)/visual_parameters.yaml">
+        <origin xyz="0.0 0.0 0.0" rpy="0.0 0.0 0.0" />
+    </xacro:ur_robot>
+    <!-- arm_0_gripper -->
+    <!--xacro:robotiq_2f_85
+    name="arm_0_gripper" parent_link="arm_0_end_effector_link">
+        <origin xyz="0.0 0.0 0.0" rpy="0.0 0.0 0.0" />
+    </xacro:robotiq_2f_85-->
     <xacro:w200
         tf_prefix="$(arg tf_prefix)"

Commit message: Arm moveable with moveit

File: wilbur_description/urdf/wilbur.urdf.xacro (robot description, xacro)
@@ -36,18 +36,8 @@
         <origin xyz="0.0 0.0 0.0" rpy="0.0 0.0 0.0" />
     </xacro:mesh>
-    <!--xacro:frame name="arm_0_end_effector" parent_link="arm_0_tool0">
+    <xacro:frame name="arm_0_end_effector" parent_link="arm_0_tool0">
         <origin xyz="0.0 0.0 0.0" rpy="0.0 0.0 0.0" />
-    </xacro:frame-->
+    </xacro:frame>
     <!-- Manipulators -->
-    <!-- arm_0 -->
-    <!--xacro:universal_robots name="arm_0"
-        parent_link="arm_plate_mount"
-        robot_ip="192.168.131.40"
-        ur_type="ur10e"
-        initial_positions_file="$(find wilbur_description)/config/arm0_initial_positions.yaml"
-        sim_ignition="true"
-        use_fake_hardware="true">
-        <origin xyz="0.0 0.0 0.0" rpy="0.0 0.0 0.0" />
-    </xacro:universal_robots-->
     <xacro:ur_robot
         name="arm_0_"

Commit message: added absolute vs relative path on mesh

File: wilbur_description/urdf/wilbur.urdf.xacro (robot description, xacro)
@@ -13,7 +13,10 @@
     <xacro:include filename="$(find clearpath_platform_description)/urdf/links/frame.urdf.xacro" />
     <xacro:include filename="$(find clearpath_platform_description)/urdf/links/mesh.urdf.xacro" />
+    <xacro:include filename="$(find wilbur_description)/urdf/gen_mesh.xacro"/>
     <!--xacro:include
         filename="$(find clearpath_manipulators_description)/urdf/arm/universal_robots.urdf.xacro" /-->
     <xacro:include filename="$(find ur_description)/urdf/ur_macro.xacro" />
+    <!-- if ignition or gazebo - need to use absolute paths instead of relative-->
+    <xacro:property name="force_abs_paths" value="$(arg sim_ignition)" scope="global"/>
     <!-- Attachments -->
     <xacro:bulkhead
@@ -25,11 +28,23 @@
     </xacro:bulkhead>
     <!-- Links -->
-    <!-- todo - reduce dependency on clearpath platform description buildin macros -->
-    <xacro:mesh
-        name="control_frame"
-        parent_link="default_mount"
-        visual="file://$(find wilbur_description)/meshes/control_frame.stl">
-        <origin xyz="0.0 0.0 0.0" rpy="0.0 0.0 0.0" />
-    </xacro:mesh>
+    <link name="control_frame_link">
+      <visual>
+        <geometry>
+          <xacro:gen_mesh force_abs_path="${force_abs_paths}" pkg_name="wilbur_description" file_path="meshes/control_frame.stl"/>
+        </geometry>
+        <material name="clearpath_dark_grey"/>
+      </visual>
+      <collision>
+        <geometry>
+          <xacro:gen_mesh force_abs_path="${force_abs_paths}" pkg_name="wilbur_description" file_path="meshes/control_frame.stl"/>
+        </geometry>
+        <material name="clearpath_dark_grey"/>
+      </collision>
+    </link>
+    <joint name="control_frame_joint" type="fixed">
+      <parent link="default_mount" />
+      <child link="control_frame_link" />
+      <origin xyz="0 0 0" rpy="0 0 0" />
+    </joint>
     <!-- todo - reduce dependency on clearpath platform description buildin macros -->
     <xacro:frame name="arm_0_end_effector" parent_link="arm_0_tool0">

Commit message: add option to remove UR and fix UR URDF parameters

File: wilbur_description/urdf/wilbur.urdf.xacro (robot description, xacro)
@@ -6,4 +6,5 @@
     <xacro:arg name="use_fake_hardware" default="true" /> <!-- todo look into calling this use_mock_hardware to be forward leaning-->
     <xacro:arg name="parent" default="world" />
+    <xacro:arg name="include_ur" default="true"/>
     <xacro:arg name="generate_ros2_control_tag" default="true" /> <!-- for mujoco cannot have this -->
     <xacro:arg name="wilbur_ur10e_initial_positions" default="$(find wilbur_deploy)/config/ur_initial_positions.yaml" />
@@ -49,17 +50,19 @@
     </joint>
         <!-- Manipulators -->
-    <xacro:property name="initial_positions_file"  value="$(arg wilbur_ur10e_initial_positions)"  />
-    <!-- todo expose out args for hardware-->
-    <xacro:wilbur_ur10e
-        name="arm_0_"
-        tf_prefix="$(arg tf_prefix)arm_0_"
-        parent="$(arg tf_prefix)arm_plate_mount"
-        use_fake_hardware="$(arg use_fake_hardware)"
-        sim_ignition="$(arg sim_ignition)"
-        initial_positions="${xacro.load_yaml(initial_positions_file)}"
-        generate_ros2_control_tag="$(arg generate_ros2_control_tag)"
-      >
-      <origin xyz="0.0 0.0 0.0" rpy="0.0 0.0 0.0" />
-    </xacro:wilbur_ur10e>
+    <xacro:if value="$(arg include_ur)">
+      <xacro:property name="initial_positions_file"  value="$(arg wilbur_ur10e_initial_positions)"  />
+      <!-- todo expose out args for hardware-->
+      <xacro:wilbur_ur10e
+          name="arm_0_"
+          tf_prefix="$(arg tf_prefix)arm_0_"
+          parent="$(arg tf_prefix)arm_plate_mount"
+          use_fake_hardware="$(arg use_fake_hardware)"
+          sim_ignition="$(arg sim_ignition)"
+          initial_positions="${xacro.load_yaml(initial_positions_file)}"
+          generate_ros2_control_tag="$(arg generate_ros2_control_tag)"
+        >
+        <origin xyz="0.0 0.0 0.0" rpy="0.0 0.0 0.0" />
+      </xacro:wilbur_ur10e>
+    </xacro:if>
     <xacro:w200
         wheel="default"

File: wilbur_description/urdf/wilbur_ur10e_macro.urdf.xacro (robot description, xacro)
@@ -26,12 +26,8 @@
         tf_prefix="${tf_prefix}"
         parent="${parent}"
-        use_fake_hardware="${use_fake_hardware}"
-        sim_ignition="${sim_ignition}"
-        initial_positions="${xacro.load_yaml(initial_positions_file)}"
         joint_limits_parameters_file="$(find ur_description)/config/ur10e/joint_limits.yaml"
         kinematics_parameters_file="$(find ur_description)/config/ur10e/default_kinematics.yaml"
         physical_parameters_file="$(find ur_description)/config/ur10e/physical_parameters.yaml"
         visual_parameters_file="$(find ur_description)/config/ur10e/visual_parameters.yaml"
-        generate_ros2_control_tag="${generate_ros2_control_tag}"
       >
       <xacro:insert_block name="origin" />

Commit message: changed the parameter that sets absolute paths

File: wilbur_description/urdf/wilbur.urdf.xacro (robot description, xacro)
@@ -3,4 +3,5 @@
     <xacro:arg name="tf_prefix" default="" />
     <xacro:arg name="ns" default="" />
+    <xacro:arg name="abs_mesh_paths" default="false" />
     <xacro:arg name="sim_ignition" default="false" />
     <xacro:arg name="use_fake_hardware" default="true" /> <!-- todo look into calling this use_mock_hardware to be forward leaning-->
@@ -17,6 +18,6 @@
     <xacro:include filename="$(find wilbur_description)/urdf/gen_mesh.xacro"/>
     <xacro:include filename="$(find wilbur_description)/urdf/wilbur_ur10e_macro.urdf.xacro" />
-    <!-- if ignition or gazebo - need to use absolute paths instead of relative-->
-    <xacro:property name="force_abs_paths" value="$(arg sim_ignition)" scope="global"/>
+    <!-- Force absolute mesh paths, necessary for Gazebo. -->
+    <xacro:property name="force_abs_paths" value="$(arg abs_mesh_paths)" scope="global"/>
     <!-- Attachments -->
     <xacro:bulkhead

Commit message: layer of abstraction for wilbur

File: wilbur_description/urdf/wilbur.urdf.xacro (robot description, xacro)
@@ -1,83 +1,26 @@
 <?xml version="1.0"?>
 <robot name="wilbur" xmlns:xacro="http://ros.org/wiki/xacro">
-    <xacro:arg name="tf_prefix" default="" />
-    <xacro:arg name="ns" default="" />
-    <xacro:arg name="abs_mesh_paths" default="false" />
-    <xacro:arg name="sim_ignition" default="false" />
-    <xacro:arg name="use_fake_hardware" default="true" /> <!-- todo look into calling this use_mock_hardware to be forward leaning-->
-    <xacro:arg name="parent" default="world" />
-    <xacro:arg name="include_ur" default="true"/>
-    <xacro:arg name="generate_ros2_control_tag" default="true" /> <!-- for mujoco cannot have this -->
-    <xacro:arg name="wilbur_ur10e_initial_positions" default="$(find wilbur_deploy)/config/ur_initial_positions.yaml" />
-    <!-- Includes -->
-    <xacro:include filename="$(find wilbur_description)/urdf/common.urdf.xacro" />
-    <xacro:include filename="$(find wilbur_description)/urdf/w200_macro.urdf.xacro" />
-    <xacro:include filename="$(find wilbur_description)/urdf/attachments/bulkhead.urdf.xacro" />
-    <xacro:include filename="$(find wilbur_description)/urdf/links/frame.urdf.xacro" />
-    <xacro:include filename="$(find wilbur_description)/urdf/links/mesh.urdf.xacro" />
-    <xacro:include filename="$(find wilbur_description)/urdf/gen_mesh.xacro"/>
-    <xacro:include filename="$(find wilbur_description)/urdf/wilbur_ur10e_macro.urdf.xacro" />
-    <!-- Force absolute mesh paths, necessary for Gazebo. -->
-    <xacro:property name="force_abs_paths" value="$(arg abs_mesh_paths)" scope="global"/>
-    <!-- Attachments -->
-    <xacro:bulkhead
-        name="bulkhead"
-        model="$(arg tf_prefix)arm_plate"
-        parent_link="$(arg tf_prefix)default_mount"
-        tf_prefix="$(arg tf_prefix)">
-        <origin xyz="0.0 0.0 0.0" rpy="0.0 0.0 0.0" />
-    </xacro:bulkhead>
-    <!-- Links -->
-    <link name="$(arg tf_prefix)control_frame_link">
-      <visual>
-        <geometry>
-          <xacro:gen_mesh force_abs_path="${force_abs_paths}" pkg_name="wilbur_description" file_path="meshes/control_frame.stl"/>
-        </geometry>
-        <material name="clearpath_dark_grey"/>
-      </visual>
-      <collision>
-        <geometry>
-          <xacro:gen_mesh force_abs_path="${force_abs_paths}" pkg_name="wilbur_description" file_path="meshes/control_frame.stl"/>
-        </geometry>
-        <material name="clearpath_dark_grey"/>
-      </collision>
-    </link>
-    <joint name="$(arg tf_prefix)control_frame_joint" type="fixed">
-      <parent link="$(arg tf_prefix)default_mount" />
-      <child link="$(arg tf_prefix)control_frame_link" />
-      <origin xyz="0 0 0" rpy="0 0 0" />
-    </joint>
-    <!-- Manipulators -->
-    <xacro:if value="$(arg include_ur)">
-      <xacro:property name="initial_positions_file"  value="$(arg wilbur_ur10e_initial_positions)"  />
-      <!-- todo expose out args for hardware-->
-      <xacro:wilbur_ur10e
-          name="arm_0_"
-          tf_prefix="$(arg tf_prefix)arm_0_"
-          parent="$(arg tf_prefix)arm_plate_mount"
-          use_fake_hardware="$(arg use_fake_hardware)"
-          sim_ignition="$(arg sim_ignition)"
-          initial_positions="${xacro.load_yaml(initial_positions_file)}"
-          generate_ros2_control_tag="$(arg generate_ros2_control_tag)"
-        >
-        <origin xyz="0.0 0.0 0.0" rpy="0.0 0.0 0.0" />
-      </xacro:wilbur_ur10e>
-    </xacro:if>
-    <xacro:w200
-        wheel="default"
-        tf_prefix="$(arg tf_prefix)"
-        sim_ignition="$(arg sim_ignition)"
-        use_fake_hardware="$(arg use_fake_hardware)"
-        ns="$(arg ns)"
-        generate_ros2_control_tag="$(arg generate_ros2_control_tag)"
-    />
-    <xacro:if value="$(arg sim_ignition)">
-      <xacro:include filename="$(find wilbur_gz)/urdf/wilbur_gz.ros2_control.xacro" />
-      <xacro:wilbur_gz_ros2_control
-        gazebo_controllers_config_file="$(find wilbur_gz)/config/gazebo_controllers.yaml"
-        ns="$(arg ns)"
-      />
-      <xacro:include filename="$(find wilbur_gz)/urdf/wilbur_gz.xacro" />
-      <xacro:wilbur_gz/>
-    </xacro:if>
+  <xacro:arg name="tf_prefix" default="" />
+  <xacro:arg name="ns" default="" />
+  <xacro:arg name="abs_mesh_paths" default="false" />
+  <xacro:arg name="sim_ignition" default="false" />
+  <xacro:arg name="use_mock_hardware" default="true" />
+  <xacro:arg name="parent" default="world" />
+  <xacro:arg name="include_ur" default="true" />
+  <xacro:arg name="gripper_com_port" default="/dev/ttyUSB0" />
+  <xacro:arg name="wilbur_ur10e_initial_positions"
+    default="$(find wilbur_deploy)/config/ur_initial_positions.yaml" />
+  <!-- Force absolute mesh paths, necessary for Gazebo. -->
+  <xacro:property name="force_abs_paths" value="$(arg abs_mesh_paths)" scope="global" />
+  <xacro:include filename="$(find wilbur_description)/urdf/wilbur.xacro" />
+  <xacro:wilbur
+    tf_prefix="$(arg tf_prefix)"
+    ns="$(arg ns)"
+    parent="$(arg parent)"
+    sim_ignition="$(arg sim_ignition)"
+    use_mock_hardware="$(arg use_mock_hardware)"
+    include_ur="$(arg include_ur)"
+    gripper_com_port="$(arg gripper_com_port)"
+    wilbur_ur10e_initial_positions="$(arg wilbur_ur10e_initial_positions)"
+  />
 </robot>
