Commit message: added comments and tf_prefixes

File: wilbur_description/urdf/w200.ros2_control.xacro (robot description, xacro)
@@ -5,4 +5,5 @@
     use_fake_hardware:=false
     sim_ignition:=false
+    tf_prefix
   ">
     <ros2_control name="${name}" type="system">

File: wilbur_description/urdf/w200.urdf.xacro (robot description, xacro)
@@ -13,5 +13,5 @@
     <xacro:include filename="$(find wilbur_description)/urdf/wheels/track.urdf.xacro" />
     <xacro:include filename="$(find wilbur_description)/urdf/wheels/wheel.urdf.xacro" />
-    <xacro:property name="PI" value="3.1415926535897931" />
+    <xacro:property name="PI" value="3.1415926535897931" /> <!--pi is build in - replace with lowercase pi throughout and remove property -->
     <xacro:include filename="$(find wilbur_description)/urdf/diff_unit.urdf.xacro" />
     <!-- Colors: yellow, orange, olive, sand -->
@@ -192,4 +192,5 @@
         use_fake_hardware="${use_fake_hardware}"
         sim_ignition="${sim_ignition}"
+        tf_prefix="${tf_prefix}"
       />
     </xacro:if>

File: wilbur_description/urdf/wilbur.urdf.xacro (robot description, xacro)
@@ -7,5 +7,7 @@
     <xacro:arg name="parent" default="world" />
     <xacro:arg name="generate_ros2_control_tag" default="true" /> <!-- for mujoco cannot have this -->
+    <xacro:arg name="wilbur_ur10e_initial_positions" default="$(find wilbur_deploy)/config/ur_initial_positions.yaml" />
     <!-- Includes -->
+    <!-- todo - reduce the dependency on clear_path_description-->
     <xacro:include filename="$(find clearpath_platform_description)/urdf/common.urdf.xacro" />
     <xacro:include filename="$(find wilbur_description)/urdf/w200.urdf.xacro" />
@@ -15,6 +17,4 @@
     <xacro:include filename="$(find clearpath_platform_description)/urdf/links/mesh.urdf.xacro" />
     <xacro:include filename="$(find wilbur_description)/urdf/gen_mesh.xacro"/>
-    <!--xacro:include
-        filename="$(find clearpath_manipulators_description)/urdf/arm/universal_robots.urdf.xacro" /-->
     <xacro:include filename="$(find ur_description)/urdf/ur_macro.xacro" />
     <!-- if ignition or gazebo - need to use absolute paths instead of relative-->
@@ -29,5 +29,5 @@
     </xacro:bulkhead>
     <!-- Links -->
-    <link name="control_frame_link">
+    <link name="$(arg tf_prefix)control_frame_link">
       <visual>
         <geometry>
@@ -43,20 +43,21 @@
       </collision>
     </link>
-    <joint name="control_frame_joint" type="fixed">
-      <parent link="default_mount" />
-      <child link="control_frame_link" />
+    <joint name="$(arg tf_prefix)control_frame_joint" type="fixed">
+      <parent link="$(arg tf_prefix)default_mount" />
+      <child link="$(arg tf_prefix)control_frame_link" />
       <origin xyz="0 0 0" rpy="0 0 0" />
     </joint>
     <!-- todo - reduce dependency on clearpath platform description buildin macros -->
+    <!-- todo - add tf prefix-->
     <xacro:frame name="arm_0_end_effector" parent_link="arm_0_tool0">
         <origin xyz="0.0 0.0 0.0" rpy="0.0 0.0 0.0" />
     </xacro:frame>
     <!-- Manipulators -->
-    <xacro:property name="initial_positions_file" default="$(find wilbur_deploy)/config/ur_initial_positions.yaml" />
+    <xacro:property name="initial_positions_file"  value="$(arg wilbur_ur10e_initial_positions)"  />
     <!-- todo expose out args for hardware-->
     <xacro:ur_robot
         name="arm_0_"
         tf_prefix="$(arg tf_prefix)arm_0_"
-        parent="arm_plate_mount"
+        parent="$(arg tf_prefix)arm_plate_mount"
         use_fake_hardware="$(arg use_fake_hardware)"
         sim_ignition="$(arg sim_ignition)"

Commit message: added todos

File: wilbur_description/urdf/w200.ros2_control.xacro (robot description, xacro)
@@ -18,5 +18,5 @@
           <!-- HARDWARE -->
           <plugin>clearpath_hardware_interfaces/W200Hardware</plugin>
-          <!-- should compute diameter from wheel radius property-->
+          <!-- todo - should compute diameter from wheel radius property-->
           <param name="wheel_diameter">0.6</param>
         </xacro:unless>

File: wilbur_description/urdf/wilbur.urdf.xacro (robot description, xacro)
@@ -62,9 +62,4 @@
       <origin xyz="0.0 0.0 0.0" rpy="0.0 0.0 0.0" />
     </xacro:wilbur_ur10e>
-    <!-- arm_0_gripper -->
-    <!--xacro:robotiq_2f_85
-    name="arm_0_gripper" parent_link="arm_0_end_effector_link">
-        <origin xyz="0.0 0.0 0.0" rpy="0.0 0.0 0.0" />
-    </xacro:robotiq_2f_85-->
     <xacro:w200
         wheel="default"

File: wilbur_description/urdf/wilbur_ur10e_macro.urdf.xacro (robot description, xacro)
@@ -13,5 +13,6 @@
     <xacro:include filename="$(find ur_description)/urdf/ur_macro.xacro" />
     <xacro:include filename="$(find clearpath_platform_description)/urdf/links/frame.urdf.xacro" />
-    <!-- todo - add tf prefix-->
+    <!-- todo - add tf prefix -->
+    <!-- todo - remove clearpath frame -->
     <xacro:frame name="arm_0_end_effector" parent_link="arm_0_tool0">
         <origin xyz="0.0 0.0 0.0" rpy="0.0 0.0 0.0" />
@@ -35,4 +36,7 @@
       <xacro:insert_block name="origin" />
     </xacro:ur_robot>
+    <!-- todo - add gripper-->
+    <!-- todo add grasp link in the moveit pro orientation
+    https://docs.picknik.ai/how_to/configuration_tutorials/configure_custom_robot/#configuring-grasp-preview -->
   </xacro:macro>
 </robot>

Commit message: added ur joints to the ros2_control

File: wilbur_description/urdf/w200.ros2_control.xacro (robot description, xacro)
@@ -22,4 +22,54 @@
         </xacro:unless>
       </hardware>
+      <xacro:if value="$(arg include_ur)">
+        <joint name="${tf_prefix}arm_0_shoulder_pan_joint">
+          <command_interface name="position" />
+          <command_interface name="velocity" />
+          <command_interface name="effort" />
+          <state_interface name="position" />
+          <state_interface name="velocity" />
+          <state_interface name="effort" />
+        </joint>
+        <joint name="${tf_prefix}arm_0_shoulder_lift_joint">
+          <command_interface name="position" />
+          <command_interface name="velocity" />
+          <command_interface name="effort" />
+          <state_interface name="position" />
+          <state_interface name="velocity" />
+          <state_interface name="effort" />
+        </joint>
+        <joint name="${tf_prefix}arm_0_elbow_joint">
+          <command_interface name="position" />
+          <command_interface name="velocity" />
+          <command_interface name="effort" />
+          <state_interface name="position" />
+          <state_interface name="velocity" />
+          <state_interface name="effort" />
+        </joint>
+        <joint name="${tf_prefix}arm_0_wrist_1_joint">
+          <command_interface name="position" />
+          <command_interface name="velocity" />
+          <command_interface name="effort" />
+          <state_interface name="position" />
+          <state_interface name="velocity" />
+          <state_interface name="effort" />
+        </joint>
+        <joint name="${tf_prefix}arm_0_wrist_2_joint">
+          <command_interface name="position" />
+          <command_interface name="velocity" />
+          <command_interface name="effort" />
+          <state_interface name="position" />
+          <state_interface name="velocity" />
+          <state_interface name="effort" />
+        </joint>
+        <joint name="${tf_prefix}arm_0_wrist_3_joint">
+          <command_interface name="position" />
+          <command_interface name="velocity" />
+          <command_interface name="effort" />
+          <state_interface name="position" />
+          <state_interface name="velocity" />
+          <state_interface name="effort" />
+        </joint>
+      </xacro:if>
       <joint name="${tf_prefix}front_left_wheel_joint">
         <command_interface name="velocity">

Commit message: added joint state broadcaster to the controller manager list

File: wilbur_description/urdf/w200.ros2_control.xacro (robot description, xacro)
@@ -1,5 +1,6 @@
 <?xml version="1.0"?>
 <robot xmlns:xacro="http://ros.org/wiki/xacro">
-  <xacro:macro name="w200_ros2_control" params="
+  <xacro:macro name="w200_ros2_control"
+    params="
     name
     use_fake_hardware:=false
@@ -77,8 +78,8 @@
           <param name="max">25</param>
         </command_interface>
-        <state_interface name="position" >
+        <state_interface name="position">
           <param name="initial_value">0.0</param>
         </state_interface>
-        <state_interface name="velocity" >
+        <state_interface name="velocity">
           <param name="initial_value">0.0</param>
         </state_interface>
@@ -89,8 +90,8 @@
           <param name="max">25</param>
         </command_interface>
-        <state_interface name="position" >
+        <state_interface name="position">
           <param name="initial_value">0.0</param>
         </state_interface>
-        <state_interface name="velocity" >
+        <state_interface name="velocity">
           <param name="initial_value">0.0</param>
         </state_interface>
@@ -101,8 +102,8 @@
           <param name="max">25</param>
         </command_interface>
-        <state_interface name="position" >
+        <state_interface name="position">
           <param name="initial_value">0.0</param>
         </state_interface>
-        <state_interface name="velocity" >
+        <state_interface name="velocity">
           <param name="initial_value">0.0</param>
         </state_interface>
@@ -113,8 +114,8 @@
           <param name="max">25</param>
         </command_interface>
-        <state_interface name="position" >
+        <state_interface name="position">
           <param name="initial_value">0.0</param>
         </state_interface>
-        <state_interface name="velocity" >
+        <state_interface name="velocity">
           <param name="initial_value">0.0</param>
         </state_interface>

Commit message: replaced all instances of sim ignition with sim gazebo

File: wilbur_description/urdf/w200.ros2_control.xacro (robot description, xacro)
@@ -5,10 +5,10 @@
     name
     use_fake_hardware:=false
-    sim_ignition:=false
+    sim_gazebo:=false
     tf_prefix
   ">
     <ros2_control name="${name}" type="system">
       <hardware>
-        <xacro:if value="${sim_ignition}">
+        <xacro:if value="${sim_gazebo}">
           <plugin>gz_ros2_control/GazeboSimSystem</plugin>
         </xacro:if>
@@ -16,5 +16,5 @@
           <plugin>mock_components/GenericSystem</plugin>
         </xacro:if>
-        <xacro:unless value="${sim_ignition or use_fake_hardware}">
+        <xacro:unless value="${sim_gazebo or use_fake_hardware}">
           <!-- HARDWARE -->
           <plugin>clearpath_hardware_interfaces/W200Hardware</plugin>

File: wilbur_description/urdf/w200.urdf.xacro (robot description, xacro)
@@ -3,6 +3,7 @@
   <xacro:arg name="tf_prefix" default="" />
   <xacro:arg name="ns" default="" />
-  <xacro:arg name="sim_ignition" default="false" />
-  <xacro:arg name="use_fake_hardware" default="true" /> <!-- todo look into calling this use_mock_hardware to be forward leaning-->
+  <xacro:arg name="sim_gazebo" default="false" />
+  <xacro:arg name="use_fake_hardware" default="true" /> <!-- todo look into calling this
+  use_mock_hardware to be forward leaning-->
   <xacro:arg name="generate_ros2_control_tag" default="true" /> <!-- for mujoco cannot have this -->
   <xacro:include filename="$(find wilbur_description)/urdf/w200_macro.urdf.xacro" />
@@ -10,5 +11,5 @@
     wheel="default"
     tf_prefix="$(arg tf_prefix)"
-    sim_ignition="$(arg sim_ignition)"
+    sim_gazebo="$(arg sim_gazebo)"
     use_fake_hardware="$(arg use_fake_hardware)"
     ns="$(arg ns)"

File: wilbur_description/urdf/wilbur.urdf.xacro (robot description, xacro)
@@ -4,5 +4,5 @@
   <xacro:arg name="ns" default="" />
   <xacro:arg name="abs_mesh_paths" default="false" />
-  <xacro:arg name="sim_ignition" default="false" />
+  <xacro:arg name="sim_gazebo" default="false" />
   <xacro:arg name="use_mock_hardware" default="true" />
   <xacro:arg name="parent" default="world" />
@@ -18,5 +18,5 @@
     ns="$(arg ns)"
     parent="$(arg parent)"
-    sim_ignition="$(arg sim_ignition)"
+    sim_gazebo="$(arg sim_gazebo)"
     use_mock_hardware="$(arg use_mock_hardware)"
     include_ur="$(arg include_ur)"

File: wilbur_description/urdf/wilbur.xacro (robot description, xacro)
@@ -5,5 +5,5 @@
             ns:=''
             parent:=world
-            sim_ignition:=false
+            sim_gazebo:=false
             use_mock_hardware:=false
             include_ur:=true
@@ -70,5 +70,5 @@
         tf_prefix="${tf_prefix}arm_0_"
         parent="${tf_prefix}arm_0_end_effector_link"
-        sim_ignition="${sim_ignition}"
+        sim_ignition="${sim_gazebo}"
         use_fake_hardware="${use_mock_hardware}"
         fake_sensor_commands="false"

File: wilbur_description/urdf/wilbur_ur10e.urdf.xacro (robot description, xacro)
@@ -2,11 +2,12 @@
 <robot name="w200" xmlns:xacro="http://ros.org/wiki/xacro">
   <xacro:arg name="tf_prefix" default="" />
-  <xacro:arg name="sim_ignition" default="false" />
-  <xacro:arg name="use_fake_hardware" default="true" /> <!-- todo look into calling this use_mock_hardware to be forward leaning-->
+  <xacro:arg name="use_fake_hardware" default="true" /> <!-- todo look into calling this
+  use_mock_hardware to be forward leaning-->
   <xacro:arg name="generate_ros2_control_tag" default="true" /> <!-- for mujoco cannot have this -->
-  <xacro:arg name="wilbur_ur10e_initial_positions" default="$(find wilbur_deploy)/config/ur_initial_positions.yaml" />
+  <xacro:arg name="wilbur_ur10e_initial_positions"
+    default="$(find wilbur_deploy)/config/ur_initial_positions.yaml" />
   <xacro:include filename="$(find wilbur_description)/urdf/wilbur_ur10e_macro.urdf.xacro" />
   <!-- Manipulators -->
-  <xacro:property name="initial_positions_file"  value="$(arg wilbur_ur10e_initial_positions)"  />
+  <xacro:property name="initial_positions_file" value="$(arg wilbur_ur10e_initial_positions)" />
   <link name="world" />
   <!-- todo expose out args for hardware-->
@@ -16,8 +17,7 @@
     parent="world"
     use_fake_hardware="$(arg use_fake_hardware)"
-    sim_ignition="$(arg sim_ignition)"
     initial_positions="${xacro.load_yaml(initial_positions_file)}"
     generate_ros2_control_tag="$(arg generate_ros2_control_tag)"
-    >
+  >
     <origin xyz="0.0 0.0 0.0" rpy="0.0 0.0 0.0" />
   </xacro:wilbur_ur10e>

File: wilbur_gz/urdf/wilbur_gz.urdf.xacro (robot description, xacro)
@@ -3,5 +3,5 @@
     <!-- Even though we do not need this argument, and shouldn't be using it is required by
      dextivr_hande.xacro in dextivr_hande -->
-    <xacro:arg name="sim_ignition" default="true" />
+    <xacro:arg name="sim_gazebo" default="true" />
     <xacro:arg name="tf_prefix" default="" />
     <xacro:arg name="ns" default="" />
@@ -18,5 +18,5 @@
         ns="$(arg ns)"
         parent="$(arg parent)"
-        sim_ignition="true"
+        sim_gazebo="true"
         use_mock_hardware="false"
         include_ur="$(arg include_ur)"
