Commit message: Gazebo sim mostly working
Arm not tested, but controller loads, hande doesn't work yet, some
interaction between the hande description and the rest of the code.

File: wilbur_description/urdf/w200.ros2_control.xacro (robot description, xacro)
@@ -5,16 +5,12 @@
     name
     use_fake_hardware:=false
-    sim_ignition:=false
     tf_prefix
   ">
     <ros2_control name="${name}" type="system">
       <hardware>
-        <xacro:if value="${sim_ignition}">
-          <plugin>gz_ros2_control/GazeboSimSystem</plugin>
-        </xacro:if>
         <xacro:if value="${use_fake_hardware}">
           <plugin>mock_components/GenericSystem</plugin>
         </xacro:if>
-        <xacro:unless value="${sim_ignition or use_fake_hardware}">
+        <xacro:unless value="${use_fake_hardware}">
           <!-- HARDWARE -->
           <plugin>clearpath_hardware_interfaces/W200Hardware</plugin>
@@ -72,4 +68,10 @@
           <state_interface name="effort" />
         </joint>
+      <!-- Left finger joint (usually the active one) -->
+      <joint name="${tf_prefix}hande_left_finger_joint">
+        <command_interface name="position"/>
+        <state_interface name="position"/>
+        <state_interface name="velocity"/>
+      </joint>
       </xacro:if>
       <joint name="${tf_prefix}front_left_wheel_joint">

File: wilbur_description/urdf/wilbur.xacro (robot description, xacro)
@@ -20,6 +20,5 @@
     <!-- Sub-robots -->
     <xacro:include filename="$(find wilbur_description)/urdf/w200_macro.urdf.xacro" />
-    <xacro:include filename="$(find wilbur_description)/urdf/wilbur_ur10e_macro.urdf.xacro" />
-    <xacro:include filename="$(find dextivr_hande_description)/urdf/dextivr_hande.xacro" />
+    <xacro:include filename="$(find wilbur_description)/urdf/w200.ros2_control.xacro" />
     <!-- Attachments -->
     <xacro:bulkhead
@@ -53,4 +52,6 @@
     <!-- Manipulators -->
     <xacro:if value="${include_ur}">
+      <xacro:include filename="$(find wilbur_description)/urdf/wilbur_ur10e_macro.urdf.xacro" />
+      <xacro:include filename="$(find dextivr_hande_description)/urdf/dextivr_hande.xacro" />
       <xacro:property name="initial_positions_file" value="${wilbur_ur10e_initial_positions}" />
       <!-- todo expose out args for hardware-->
@@ -60,5 +61,4 @@
         parent="${tf_prefix}arm_plate_mount"
         initial_positions="${xacro.load_yaml(initial_positions_file)}"
-        generate_ros2_control_tag="${generate_ros2_control_tag}"
       >
         <origin xyz="0.0 0.0 0.0" rpy="0.0 0.0 0.0" />
@@ -67,7 +67,6 @@
         <origin xyz="0.0 0.0 0.0" rpy="0.0 0.0 0.0" />
       </xacro:frame>
-      <xacro:dextivr_hande
+      <!--xacro:dextivr_hande
         name="dextivr_hande"
-        generate_ros2_control_tag="$(arg generate_ros2_control_tag)"
         tf_prefix="${tf_prefix}arm_0_"
         parent="${tf_prefix}arm_0_end_effector_link"
@@ -79,5 +78,5 @@
         finger_xacro="fngr_v6">
         <origin xyz="0 0 0" rpy="0 0 ${radians(-90)}" />
-      </xacro:dextivr_hande>
+      </xacro:dextivr_hande-->
     </xacro:if>
     <xacro:w200
@@ -86,4 +85,11 @@
       ns="${ns}"
     />
+    <xacro:if value="${generate_ros2_control_tag}">
+      <xacro:w200_ros2_control
+        name=''
+        use_fake_hardware="${use_mock_hardware}"
+        tf_prefix="${tf_prefix">
+      </xacro:w200_ros2_control>
+    </xacro:if>
   </xacro:macro>
 </robot>

File: wilbur_description/urdf/wilbur_ur10e.urdf.xacro (robot description, xacro)
@@ -4,5 +4,4 @@
   <xacro:arg name="sim_ignition" default="false" />
   <xacro:arg name="use_fake_hardware" default="true" /> <!-- todo look into calling this use_mock_hardware to be forward leaning-->
-  <xacro:arg name="generate_ros2_control_tag" default="true" /> <!-- for mujoco cannot have this -->
   <xacro:arg name="wilbur_ur10e_initial_positions" default="$(find wilbur_deploy)/config/ur_initial_positions.yaml" />
   <xacro:include filename="$(find wilbur_description)/urdf/wilbur_ur10e_macro.urdf.xacro" />
@@ -18,5 +17,4 @@
     sim_ignition="$(arg sim_ignition)"
     initial_positions="${xacro.load_yaml(initial_positions_file)}"
-    generate_ros2_control_tag="$(arg generate_ros2_control_tag)"
     >
     <origin xyz="0.0 0.0 0.0" rpy="0.0 0.0 0.0" />

File: wilbur_gz/urdf/wilbur_gz.ros2_control.xacro (robot description, xacro)
@@ -4,4 +4,5 @@
     gazebo_controllers_config_file
     include_ur=true
+    include_hande=false
     tf_prefix=''
     name='wilbur'
@@ -14,16 +15,4 @@
         <parameters>${gazebo_controllers_config_file}</parameters>
         <controller_manager_name>controller_manager</controller_manager_name>
-        <ros>
-          <remapping>~/odom:=odom</remapping>
-          <remapping>~/cmd_vel_unstamped:=cmd_vel_unstamped</remapping>
-          <remapping>/tf:=tf</remapping>
-          <remapping>/tf_static:=tf_static</remapping>
-          <remapping>/diagnostics:=diagnostics</remapping>
-          <remapping>/dynamic_joint_states:=dynamic_joint_states</remapping>
-          <remapping>joint_states:=joint_states</remapping>
-          <remapping>~/reference:=cmd_vel</remapping>
-          <remapping>~/odometry:=odom</remapping>
-          <namespace>${ns}</namespace>
-        </ros>
       </plugin>
     </gazebo>
@@ -32,5 +21,14 @@
           <plugin>gz_ros2_control/GazeboSimSystem</plugin>
       </hardware>
-      <xacro:if value="$(arg include_ur)">
+      <xacro:if value="${include_ur}">
+        <!--xacro:if value="${include_hande}">
+          <xacro:include filename="$(find robotiq_hande_description)/urdf/robotiq_hande.ros2_control.xacro" />
+          <xacro:robotiq_hande_ros2_control
+              tf_prefix="${tf_prefix}"
+              sim_ignition="true"
+              use_fake_hardware="false"
+              fake_sensor_commands="true"
+          />
+        </xacro:if-->
         <joint name="${tf_prefix}arm_0_shoulder_pan_joint">
           <command_interface name="position" />

File: wilbur_gz/urdf/wilbur_gz.urdf.xacro (robot description, xacro)
@@ -17,6 +17,6 @@
     <xacro:include filename="$(find wilbur_gz)/urdf/wilbur_gz.xacro" />
     <xacro:property name="force_abs_paths" value="$(arg abs_mesh_paths)" scope="global" />
-    <xacro:property name="generate_ros2_control_tag" value="false" />
     <xacro:wilbur
+        generate_ros2_control_tag="false"
         tf_prefix="$(arg tf_prefix)"
         ns="$(arg ns)"
@@ -27,20 +27,12 @@
         gripper_com_port="$(arg gripper_com_port)"
         wilbur_ur10e_initial_positions="$(arg wilbur_ur10e_initial_positions)"
-        generate_ros2_control_tag="${generate_ros2_control_tag}"
     />
     <xacro:include filename="$(find wilbur_gz)/urdf/wilbur_gz.ros2_control.xacro" />
     <xacro:include filename="$(find wilbur_gz)/urdf/wilbur_gz.xacro" />
-    <xacro:if value="$(arg include_ur)">
     <xacro:wilbur_gz_ros2_control
+        tf_prefix="$(arg tf_prefix)"
         gazebo_controllers_config_file="$(find wilbur_gz)/config/gazebo_controllers.yaml"
         ns="$(arg ns)"
     />
-    </xacro:if>
-    <xacro:unless value="$(arg include_ur)">
-        <xacro:wilbur_gz_ros2_control
-            gazebo_controllers_config_file="$(find wilbur_gz)/config/gazebo_controllers_no_ur.yaml"
-            ns="$(arg ns)"
-        />
-    </xacro:unless>
     <xacro:wilbur_gz />
 </robot>
