Commit message: replaced the ur ros2 control joint with ur_descrption macro

File: wilbur_description/urdf/wilbur.xacro (robot description, xacro)
@@ -56,5 +56,5 @@
       <!-- todo expose out args for hardware-->
       <xacro:wilbur_ur10e
-        name="arm_0_"
+        name="arm_0"
         tf_prefix="${tf_prefix}arm_0_"
         parent="${tf_prefix}arm_plate_mount"

File: wilbur_description/urdf/wilbur_mock.ros2_control.xacro (robot description, xacro)
@@ -1,113 +1,73 @@
 <?xml version="1.0"?>
 <robot xmlns:xacro="http://ros.org/wiki/xacro">
-    <xacro:macro name="w200_ros2_control"
-        params="
+  <xacro:include filename="$(find ur_description)/urdf/inc/ur_joint_control.xacro" />
+  <xacro:include filename="$(find ur_description)/urdf/inc/ur_sensors.xacro" />
+  <xacro:macro name="w200_ros2_control"
+    params="
         name
         tf_prefix
         include_ur:=false
+        wilbur_ur10e_initial_positions:=${dict(shoulder_pan_joint=0.0,shoulder_lift_joint=-1.57,elbow_joint=0.0,wrist_1_joint=-1.57,wrist_2_joint=0.0,wrist_3_joint=0.0)}
     ">
-        <ros2_control name="${name}" type="system">
-            <hardware>
-                <plugin>mock_components/GenericSystem</plugin>
-            </hardware>
-            <xacro:if value="$(arg include_ur)">
-                <joint name="${tf_prefix}arm_0_shoulder_pan_joint">
-                    <command_interface name="position" />
-                    <command_interface name="velocity" />
-                    <command_interface name="effort" />
-                    <state_interface name="position" />
-                    <state_interface name="velocity" />
-                    <state_interface name="effort" />
-                </joint>
-                <joint name="${tf_prefix}arm_0_shoulder_lift_joint">
-                    <command_interface name="position" />
-                    <command_interface name="velocity" />
-                    <command_interface name="effort" />
-                    <state_interface name="position" />
-                    <state_interface name="velocity" />
-                    <state_interface name="effort" />
-                </joint>
-                <joint name="${tf_prefix}arm_0_elbow_joint">
-                    <command_interface name="position" />
-                    <command_interface name="velocity" />
-                    <command_interface name="effort" />
-                    <state_interface name="position" />
-                    <state_interface name="velocity" />
-                    <state_interface name="effort" />
-                </joint>
-                <joint name="${tf_prefix}arm_0_wrist_1_joint">
-                    <command_interface name="position" />
-                    <command_interface name="velocity" />
-                    <command_interface name="effort" />
-                    <state_interface name="position" />
-                    <state_interface name="velocity" />
-                    <state_interface name="effort" />
-                </joint>
-                <joint name="${tf_prefix}arm_0_wrist_2_joint">
-                    <command_interface name="position" />
-                    <command_interface name="velocity" />
-                    <command_interface name="effort" />
-                    <state_interface name="position" />
-                    <state_interface name="velocity" />
-                    <state_interface name="effort" />
-                </joint>
-                <joint name="${tf_prefix}arm_0_wrist_3_joint">
-                    <command_interface name="position" />
-                    <command_interface name="velocity" />
-                    <command_interface name="effort" />
-                    <state_interface name="position" />
-                    <state_interface name="velocity" />
-                    <state_interface name="effort" />
-                </joint>
-            </xacro:if>
-            <joint name="${tf_prefix}front_left_wheel_joint">
-                <command_interface name="velocity">
-                    <param name="min">-25</param>
-                    <param name="max">25</param>
-                </command_interface>
-                <state_interface name="position">
-                    <param name="initial_value">0.0</param>
-                </state_interface>
-                <state_interface name="velocity">
-                    <param name="initial_value">0.0</param>
-                </state_interface>
-            </joint>
-            <joint name="${tf_prefix}rear_left_wheel_joint">
-                <command_interface name="velocity">
-                    <param name="min">-25</param>
-                    <param name="max">25</param>
-                </command_interface>
-                <state_interface name="position">
-                    <param name="initial_value">0.0</param>
-                </state_interface>
-                <state_interface name="velocity">
-                    <param name="initial_value">0.0</param>
-                </state_interface>
-            </joint>
-            <joint name="${tf_prefix}front_right_wheel_joint">
-                <command_interface name="velocity">
-                    <param name="min">-25</param>
-                    <param name="max">25</param>
-                </command_interface>
-                <state_interface name="position">
-                    <param name="initial_value">0.0</param>
-                </state_interface>
-                <state_interface name="velocity">
-                    <param name="initial_value">0.0</param>
-                </state_interface>
-            </joint>
-            <joint name="${tf_prefix}rear_right_wheel_joint">
-                <command_interface name="velocity">
-                    <param name="min">-25</param>
-                    <param name="max">25</param>
-                </command_interface>
-                <state_interface name="position">
-                    <param name="initial_value">0.0</param>
-                </state_interface>
-                <state_interface name="velocity">
-                    <param name="initial_value">0.0</param>
-                </state_interface>
-            </joint>
-        </ros2_control>
-    </xacro:macro>
+    <ros2_control name="${name}" type="system">
+      <hardware>
+        <plugin>mock_components/GenericSystem</plugin>
+      </hardware>
+      <xacro:if value="$(arg include_ur)">
+        <xacro:ur_joint_control_description
+          tf_prefix="${tf_prefix}arm_0_"
+          initial_positions="${wilbur_ur10e_initial_positions}"
+        />
+        <xacro:ur_sensors tf_prefix="${tf_prefix}" />
+      </xacro:if>
+      <joint name="${tf_prefix}front_left_wheel_joint">
+        <command_interface name="velocity">
+          <param name="min">-25</param>
+          <param name="max">25</param>
+        </command_interface>
+        <state_interface name="position">
+          <param name="initial_value">0.0</param>
+        </state_interface>
+        <state_interface name="velocity">
+          <param name="initial_value">0.0</param>
+        </state_interface>
+      </joint>
+      <joint name="${tf_prefix}rear_left_wheel_joint">
+        <command_interface name="velocity">
+          <param name="min">-25</param>
+          <param name="max">25</param>
+        </command_interface>
+        <state_interface name="position">
+          <param name="initial_value">0.0</param>
+        </state_interface>
+        <state_interface name="velocity">
+          <param name="initial_value">0.0</param>
+        </state_interface>
+      </joint>
+      <joint name="${tf_prefix}front_right_wheel_joint">
+        <command_interface name="velocity">
+          <param name="min">-25</param>
+          <param name="max">25</param>
+        </command_interface>
+        <state_interface name="position">
+          <param name="initial_value">0.0</param>
+        </state_interface>
+        <state_interface name="velocity">
+          <param name="initial_value">0.0</param>
+        </state_interface>
+      </joint>
+      <joint name="${tf_prefix}rear_right_wheel_joint">
+        <command_interface name="velocity">
+          <param name="min">-25</param>
+          <param name="max">25</param>
+        </command_interface>
+        <state_interface name="position">
+          <param name="initial_value">0.0</param>
+        </state_interface>
+        <state_interface name="velocity">
+          <param name="initial_value">0.0</param>
+        </state_interface>
+      </joint>
+    </ros2_control>
+  </xacro:macro>
 </robot>

File: wilbur_description/urdf/wilbur_mock.urdf.xacro (robot description, xacro)
@@ -13,4 +13,6 @@
     <xacro:include filename="$(find wilbur_description)/urdf/wilbur.xacro" />
     <xacro:property name="force_abs_paths" value="$(arg abs_mesh_paths)" scope="global" />
+    <!-- convert to property to use substitution in function -->
+    <xacro:property name="initial_positions_file" default="$(arg wilbur_ur10e_initial_positions)"/>
     <xacro:wilbur
         tf_prefix="$(arg tf_prefix)"
@@ -27,4 +29,6 @@
         name="wilbur"
         tf_prefix="$(arg tf_prefix)"
-        include_ur="$(arg include_ur)" />
+        include_ur="$(arg include_ur)"
+        wilbur_ur10e_initial_positions="${xacro.load_yaml(initial_positions_file)}"
+        />
 </robot>

File: wilbur_description/urdf/wilbur_ur10e.urdf.xacro (robot description, xacro)
@@ -14,5 +14,5 @@
   <xacro:wilbur_ur10e
     name="arm_0_"
-    tf_prefix="$(arg tf_prefix)arm_0_"
+    tf_prefix="$(arg tf_prefix)"
     parent="world"
     use_fake_hardware="$(arg use_fake_hardware)"

File: wilbur_gz/urdf/wilbur_gz.xacro (robot description, xacro)
@@ -14,4 +14,6 @@
     </gazebo>
   </xacro:macro>
+  <xacro:include filename="$(find ur_description)/urdf/inc/ur_joint_control.xacro" />
+  <xacro:include filename="$(find ur_description)/urdf/inc/ur_sensors.xacro" />
   <xacro:macro name="w200_ros2_control"
     params="
@@ -19,4 +21,5 @@
     tf_prefix
     include_ur:=false
+    wilbur_ur10e_initial_positions:=${dict(shoulder_pan_joint=0.0,shoulder_lift_joint=-1.57,elbow_joint=0.0,wrist_1_joint=-1.57,wrist_2_joint=0.0,wrist_3_joint=0.0)}
   ">
     <ros2_control name="${name}" type="system">
@@ -25,52 +28,9 @@
       </hardware>
       <xacro:if value="$(arg include_ur)">
-        <joint name="${tf_prefix}arm_0_shoulder_pan_joint">
-          <command_interface name="position" />
-          <command_interface name="velocity" />
-          <command_interface name="effort" />
-          <state_interface name="position" />
-          <state_interface name="velocity" />
-          <state_interface name="effort" />
-        </joint>
-        <joint name="${tf_prefix}arm_0_shoulder_lift_joint">
-          <command_interface name="position" />
-          <command_interface name="velocity" />
-          <command_interface name="effort" />
-          <state_interface name="position" />
-          <state_interface name="velocity" />
-          <state_interface name="effort" />
-        </joint>
-        <joint name="${tf_prefix}arm_0_elbow_joint">
-          <command_interface name="position" />
-          <command_interface name="velocity" />
-          <command_interface name="effort" />
-          <state_interface name="position" />
-          <state_interface name="velocity" />
-          <state_interface name="effort" />
-        </joint>
-        <joint name="${tf_prefix}arm_0_wrist_1_joint">
-          <command_interface name="position" />
-          <command_interface name="velocity" />
-          <command_interface name="effort" />
-          <state_interface name="position" />
-          <state_interface name="velocity" />
-          <state_interface name="effort" />
-        </joint>
-        <joint name="${tf_prefix}arm_0_wrist_2_joint">
-          <command_interface name="position" />
-          <command_interface name="velocity" />
-          <command_interface name="effort" />
-          <state_interface name="position" />
-          <state_interface name="velocity" />
-          <state_interface name="effort" />
-        </joint>
-        <joint name="${tf_prefix}arm_0_wrist_3_joint">
-          <command_interface name="position" />
-          <command_interface name="velocity" />
-          <command_interface name="effort" />
-          <state_interface name="position" />
-          <state_interface name="velocity" />
-          <state_interface name="effort" />
-        </joint>
+        <xacro:ur_joint_control_description
+          tf_prefix="${tf_prefix}arm_0_"
+          initial_positions="${wilbur_ur10e_initial_positions}"
+        />
+        <xacro:ur_sensors tf_prefix="${tf_prefix}" />
       </xacro:if>
       <joint name="${tf_prefix}front_left_wheel_joint">

Commit message: not in working condition

File: wilbur_description/urdf/wilbur.xacro (robot description, xacro)
@@ -1,10 +1,11 @@
 <?xml version="1.0"?>
-<robot name="wilbur" xmlns:xacro="http://ros.org/wiki/xacro">
+<robot xmlns:xacro="http://ros.org/wiki/xacro">
   <xacro:macro name="wilbur"
     params="tf_prefix:=''
             ns:=''
-            parent:=wolrd
+            parent:=world
             sim_ignition:=false
             use_mock_hardware:=false
+            generate_ros2_control_tag:=false
             include_ur:=true
             gripper_com_port:=/dev/ttyUSB0
@@ -43,5 +44,4 @@
             file_path="meshes/control_frame.stl" />
         </geometry>
-        <material name="clearpath_dark_grey" />
       </collision>
     </link>
