Commit message: fix wheel mesh path

File: wilbur_description/urdf/wheels/wheel.urdf.xacro (robot description, xacro)
@@ -16,5 +16,5 @@
         <origin xyz="0 0 0" rpy="0 0 ${PI/2}" />
         <geometry>
-          <mesh filename="package://clearpath_platform_description/meshes/w200/wheel.stl" />
+          <mesh filename="package://clearpath_platform_description/meshes/w200/wheels/outdoor.stl" />
         </geometry>
         <material name="clearpath_dark_grey" />
