Commit message: adding pre-commit

File: wilbur_description/urdf/attachments/bulkhead.urdf.xacro (robot description, xacro)
@@ -1,10 +1,11 @@
 <?xml version="1.0"?>
 <robot xmlns:xacro="http://www.ros.org/wiki/xacro">
-  <xacro:macro name="bulkhead"
-    params="name:=bulkhead
-                                      model:=default
-                                      parent_link:=default_mount
-                                      *origin
-                                      tf_prefix">
+  <xacro:macro name="bulkhead" params="
+    name:=bulkhead
+    model:=default
+    parent_link:=default_mount
+    *origin
+    tf_prefix
+  ">
     <xacro:include
       filename="$(find clearpath_platform_description)/urdf/w200/attachments/arm_plate.urdf.xacro" />

File: wilbur_description/urdf/wilbur.urdf.xacro (robot description, xacro)
@@ -48,5 +48,5 @@
       <origin xyz="0 0 0" rpy="0 0 0" />
     </joint>
-    <!-- todo - reduce dependency on clearpath platform description buildin macros -->
+    <!-- todo - reduce dependency on clearpath platform description building macros -->
     <!-- todo - add tf prefix-->
     <xacro:frame name="arm_0_end_effector" parent_link="arm_0_tool0">

Commit message: pulled in meshes for w200 from clearpath

File: wilbur_description/urdf/attachments/bulkhead.urdf.xacro (robot description, xacro)
@@ -14,5 +14,5 @@
         <origin xyz="0.00705 0 0.24184" rpy="0 0 0" />
         <geometry>
-          <mesh filename="package://clearpath_platform_description/meshes/w200/bulkhead.stl" />
+          <mesh filename="package://wilbur_description/meshes/w200/bulkhead.stl" />
         </geometry>
         <material name="clearpath_black">
@@ -24,5 +24,5 @@
         <geometry>
           <mesh
-            filename="package://clearpath_platform_description/meshes/w200/bulkhead-collision.stl" />
+            filename="package://wilbur_description/meshes/w200/bulkhead-collision.stl" />
         </geometry>
       </collision>

File: wilbur_description/urdf/diff_unit.urdf.xacro (robot description, xacro)
@@ -23,5 +23,5 @@
         <origin xyz="0 0 0" rpy="0 0 ${flip*PI/2}" />
         <geometry>
-          <mesh filename="package://clearpath_platform_description/meshes/w200/fenders.stl" />
+          <mesh filename="package://wilbur_description/meshes/w200/fenders.stl" />
         </geometry>
         <material name="${warthog_color}" />
@@ -30,5 +30,5 @@
         <origin xyz="0 0 0" rpy="0 0 ${flip*PI/2}" />
         <geometry>
-          <mesh filename="package://clearpath_platform_description/meshes/w200/fenders.stl" />
+          <mesh filename="package://wilbur_description/meshes/w200/fenders.stl" />
         </geometry>
       </collision>
@@ -36,5 +36,5 @@
         <origin xyz="0 0 0" rpy="0 0 ${flip*PI/2}" />
         <geometry>
-          <mesh filename="package://clearpath_platform_description/meshes/w200/rocker.stl" />
+          <mesh filename="package://wilbur_description/meshes/w200/rocker.stl" />
         </geometry>
         <material name="clearpath_black" />
@@ -54,5 +54,5 @@
         <origin xyz="0 ${flip*-0.0244} 0" rpy="0 0 0" />
         <geometry>
-          <mesh filename="package://clearpath_platform_description/meshes/w200/light.stl" />
+          <mesh filename="package://wilbur_description/meshes/w200/light.stl" />
         </geometry>
         <material name="clearpath_white" />
@@ -68,5 +68,5 @@
         <origin xyz="0 ${flip*-0.0244} 0" rpy="0 0 ${flip*PI}" />
         <geometry>
-          <mesh filename="package://clearpath_platform_description/meshes/w200/light.stl" />
+          <mesh filename="package://wilbur_description/meshes/w200/light.stl" />
         </geometry>
         <material name="clearpath_red" />

File: wilbur_description/urdf/w200_macro.urdf.xacro (robot description, xacro)
@@ -67,5 +67,5 @@
         <origin xyz="0 0 0" rpy="0 0 0" />
         <geometry>
-          <mesh filename="package://clearpath_platform_description/meshes/w200/chassis.stl" />
+          <mesh filename="package://wilbur_description/meshes/w200/chassis.stl" />
         </geometry>
         <material name="clearpath_black">
@@ -76,5 +76,5 @@
         <origin xyz="0 0 0" rpy="0 0 0" />
         <geometry>
-          <mesh filename="package://clearpath_platform_description/meshes/w200/e-stop.stl" />
+          <mesh filename="package://wilbur_description/meshes/w200/e-stop.stl" />
         </geometry>
         <material name="clearpath_red">
@@ -86,5 +86,5 @@
         <geometry>
           <mesh
-            filename="package://clearpath_platform_description/meshes/w200/chassis-collision.stl" />
+            filename="package://wilbur_description/meshes/w200/chassis-collision.stl" />
         </geometry>
       </collision>
@@ -97,5 +97,5 @@
         <origin xyz="0 0 0" rpy="0 0 0" />
         <geometry>
-          <mesh filename="package://clearpath_platform_description/meshes/w200/diff-link.stl" />
+          <mesh filename="package://wilbur_description/meshes/w200/diff-link.stl" />
         </geometry>
         <material name="clearpath_light_grey" />
@@ -104,5 +104,5 @@
         <origin xyz="0 0 0" rpy="0 0 0" />
         <geometry>
-          <mesh filename="package://clearpath_platform_description/meshes/w200/susp-link.stl" />
+          <mesh filename="package://wilbur_description/meshes/w200/susp-link.stl" />
         </geometry>
         <material name="clearpath_light_grey" />
@@ -111,5 +111,5 @@
         <origin xyz="0 0 0" rpy="0 0 0" />
         <geometry>
-          <mesh filename="package://clearpath_platform_description/meshes/w200/susp-link.stl" />
+          <mesh filename="package://wilbur_description/meshes/w200/susp-link.stl" />
         </geometry>
         <material name="clearpath_light_grey" />

File: wilbur_description/urdf/wheels/wheel.urdf.xacro (robot description, xacro)
@@ -16,5 +16,5 @@
         <origin xyz="0 0 0" rpy="0 0 ${PI/2}" />
         <geometry>
-          <mesh filename="package://clearpath_platform_description/meshes/w200/wheels/outdoor.stl" />
+          <mesh filename="package://wilbur_description/meshes/w200/wheels/outdoor.stl" />
         </geometry>
         <material name="clearpath_dark_grey" />

Commit message: replaced all mesh imports with custom xacro for absolute paths

File: wilbur_description/urdf/attachments/bulkhead.urdf.xacro (robot description, xacro)
@@ -14,5 +14,5 @@
         <origin xyz="0.00705 0 0.24184" rpy="0 0 0" />
         <geometry>
-          <mesh filename="package://wilbur_description/meshes/w200/bulkhead.stl" />
+          <xacro:gen_mesh force_abs_path="${force_abs_paths}" pkg_name="wilbur_description" file_path="meshes/w200/bulkhead.stl" />
         </geometry>
         <material name="clearpath_black">
@@ -23,6 +23,5 @@
         <origin xyz="0.00705 0 0.24184" rpy="0 0 0" />
         <geometry>
-          <mesh
-            filename="package://wilbur_description/meshes/w200/bulkhead-collision.stl" />
+          <xacro:gen_mesh force_abs_path="${force_abs_paths}" pkg_name="wilbur_description" file_path="meshes/w200/bulkhead-collision.stl" />
         </geometry>
       </collision>

File: wilbur_description/urdf/diff_unit.urdf.xacro (robot description, xacro)
@@ -23,5 +23,5 @@
         <origin xyz="0 0 0" rpy="0 0 ${flip*PI/2}" />
         <geometry>
-          <mesh filename="package://wilbur_description/meshes/w200/fenders.stl" />
+          <xacro:gen_mesh force_abs_path="${force_abs_paths}" pkg_name="wilbur_description" file_path="meshes/w200/fenders.stl" />
         </geometry>
         <material name="${warthog_color}" />
@@ -30,5 +30,5 @@
         <origin xyz="0 0 0" rpy="0 0 ${flip*PI/2}" />
         <geometry>
-          <mesh filename="package://wilbur_description/meshes/w200/fenders.stl" />
+          <xacro:gen_mesh force_abs_path="${force_abs_paths}" pkg_name="wilbur_description" file_path="meshes/w200/fenders.stl" />
         </geometry>
       </collision>
@@ -36,5 +36,5 @@
         <origin xyz="0 0 0" rpy="0 0 ${flip*PI/2}" />
         <geometry>
-          <mesh filename="package://wilbur_description/meshes/w200/rocker.stl" />
+          <xacro:gen_mesh force_abs_path="${force_abs_paths}" pkg_name="wilbur_description" file_path="meshes/w200/rocker.stl" />
         </geometry>
         <material name="clearpath_black" />
@@ -54,5 +54,5 @@
         <origin xyz="0 ${flip*-0.0244} 0" rpy="0 0 0" />
         <geometry>
-          <mesh filename="package://wilbur_description/meshes/w200/light.stl" />
+          <xacro:gen_mesh force_abs_path="${force_abs_paths}" pkg_name="wilbur_description" file_path="meshes/w200/light.stl" />
         </geometry>
         <material name="clearpath_white" />
@@ -68,5 +68,5 @@
         <origin xyz="0 ${flip*-0.0244} 0" rpy="0 0 ${flip*PI}" />
         <geometry>
-          <mesh filename="package://wilbur_description/meshes/w200/light.stl" />
+          <xacro:gen_mesh force_abs_path="${force_abs_paths}" pkg_name="wilbur_description" file_path="meshes/w200/light.stl" />
         </geometry>
         <material name="clearpath_red" />

File: wilbur_description/urdf/w200/attachments/arm_plate.urdf.xacro (robot description, xacro)
@@ -11,5 +11,5 @@
         <origin xyz="0 0 0.02" rpy="0 0 0"/>
         <geometry>
-          <mesh filename="package://wilbur_description/meshes/w200/arm-mount-plate.stl" />
+          <xacro:gen_mesh force_abs_path="${force_abs_paths}" pkg_name="wilbur_description" file_path="meshes/w200/arm-mount-plate.stl" />
         </geometry>
         <material name="clearpath_light_grey"/>
@@ -18,5 +18,5 @@
         <origin xyz="0 0 0.02" rpy="0 0 0"/>
         <geometry>
-          <mesh filename="package://wilbur_description/meshes/w200/arm-mount-plate.stl" />
+          <xacro:gen_mesh force_abs_path="${force_abs_paths}" pkg_name="wilbur_description" file_path="meshes/w200/arm-mount-plate.stl" />
         </geometry>
       </collision>

File: wilbur_description/urdf/w200_macro.urdf.xacro (robot description, xacro)
@@ -67,5 +67,5 @@
         <origin xyz="0 0 0" rpy="0 0 0" />
         <geometry>
-          <mesh filename="package://wilbur_description/meshes/w200/chassis.stl" />
+          <xacro:gen_mesh force_abs_path="${force_abs_paths}" pkg_name="wilbur_description" file_path="meshes/w200/chassis.stl" />
         </geometry>
         <material name="clearpath_black">
@@ -76,5 +76,5 @@
         <origin xyz="0 0 0" rpy="0 0 0" />
         <geometry>
-          <mesh filename="package://wilbur_description/meshes/w200/e-stop.stl" />
+          <xacro:gen_mesh force_abs_path="${force_abs_paths}" pkg_name="wilbur_description" file_path="meshes/w200/e-stop.stl" />
         </geometry>
         <material name="clearpath_red">
@@ -85,6 +85,5 @@
         <origin xyz="0 0 0" rpy="0 0 0" />
         <geometry>
-          <mesh
-            filename="package://wilbur_description/meshes/w200/chassis-collision.stl" />
+          <xacro:gen_mesh force_abs_path="${force_abs_paths}" pkg_name="wilbur_description" file_path="meshes/w200/chassis-collision.stl" />
         </geometry>
       </collision>
@@ -97,5 +96,5 @@
         <origin xyz="0 0 0" rpy="0 0 0" />
         <geometry>
-          <mesh filename="package://wilbur_description/meshes/w200/diff-link.stl" />
+          <xacro:gen_mesh force_abs_path="${force_abs_paths}" pkg_name="wilbur_description" file_path="meshes/w200/diff-link.stl" />
         </geometry>
         <material name="clearpath_light_grey" />
@@ -104,5 +103,5 @@
         <origin xyz="0 0 0" rpy="0 0 0" />
         <geometry>
-          <mesh filename="package://wilbur_description/meshes/w200/susp-link.stl" />
+          <xacro:gen_mesh force_abs_path="${force_abs_paths}" pkg_name="wilbur_description" file_path="meshes/w200/susp-link.stl" />
         </geometry>
         <material name="clearpath_light_grey" />
@@ -111,5 +110,5 @@
         <origin xyz="0 0 0" rpy="0 0 0" />
         <geometry>
-          <mesh filename="package://wilbur_description/meshes/w200/susp-link.stl" />
+          <xacro:gen_mesh force_abs_path="${force_abs_paths}" pkg_name="wilbur_description" file_path="meshes/w200/susp-link.stl" />
         </geometry>
         <material name="clearpath_light_grey" />

File: wilbur_description/urdf/wheels/track.urdf.xacro (robot description, xacro)
@@ -7,5 +7,5 @@
         <origin xyz="0 0 0" rpy="0 0 0" />
         <geometry>
-          <mesh filename="package://wilbur_description/meshes/tracks.dae" />
+          <xacro:gen_mesh force_abs_path="${force_abs_paths}" pkg_name="wilbur_description" file_path="meshes/tracks.dae" />
         </geometry>
         <material name="clearpath_dark_grey" />

File: wilbur_description/urdf/wheels/wheel.urdf.xacro (robot description, xacro)
@@ -16,5 +16,5 @@
         <origin xyz="0 0 0" rpy="0 0 ${PI/2}" />
         <geometry>
-          <mesh filename="package://wilbur_description/meshes/w200/wheels/outdoor.stl" />
+          <xacro:gen_mesh force_abs_path="${force_abs_paths}" pkg_name="wilbur_description" file_path="meshes/w200/wheels/outdoor.stl" />
         </geometry>
         <material name="clearpath_dark_grey" />

File: wilbur_description/urdf/wilbur.urdf.xacro (robot description, xacro)
@@ -10,9 +10,7 @@
     <xacro:arg name="wilbur_ur10e_initial_positions" default="$(find wilbur_deploy)/config/ur_initial_positions.yaml" />
     <!-- Includes -->
-    <!-- todo - reduce the dependency on clear_path_description-->
     <xacro:include filename="$(find wilbur_description)/urdf/common.urdf.xacro" />
     <xacro:include filename="$(find wilbur_description)/urdf/w200_macro.urdf.xacro" />
-    <xacro:include
-        filename="$(find wilbur_description)/urdf/attachments/bulkhead.urdf.xacro" />
+    <xacro:include filename="$(find wilbur_description)/urdf/attachments/bulkhead.urdf.xacro" />
     <xacro:include filename="$(find wilbur_description)/urdf/links/frame.urdf.xacro" />
     <xacro:include filename="$(find wilbur_description)/urdf/links/mesh.urdf.xacro" />
@@ -49,5 +47,5 @@
       <origin xyz="0 0 0" rpy="0 0 0" />
     </joint>
-        <!-- Manipulators -->
+    <!-- Manipulators -->
     <xacro:if value="$(arg include_ur)">
       <xacro:property name="initial_positions_file"  value="$(arg wilbur_ur10e_initial_positions)"  />
