Commit message: Fixes for launching Phoebe + WilbUR together

File: wilbur_description/urdf/attachments/bulkhead.urdf.xacro (robot description, xacro)
@@ -16,5 +16,5 @@
           <xacro:gen_mesh force_abs_path="${force_abs_paths}" pkg_name="wilbur_description" file_path="meshes/w200/bulkhead.stl" />
         </geometry>
-        <material name="clearpath_black">
+        <material name="wilbur_black">
           <color rgba="0.15 0.15 0.15 1.0" />
         </material>

File: wilbur_description/urdf/common.urdf.xacro (robot description, xacro)
@@ -23,15 +23,15 @@
 -->
 <robot xmlns:xacro="http://ros.org/wiki/xacro">
-    <material name="clearpath_dark_grey"><color rgba="0.2 0.2 0.2 1.0" /></material>
-    <material name="clearpath_medium_grey"><color rgba="0.6 0.6 0.6 1.0" /></material>
-    <material name="clearpath_light_grey"><color rgba="0.8 0.8 0.8 1.0" /></material>
-    <material name="clearpath_yellow"><color rgba="0.8 0.8 0.0 1.0" /></material>
-    <material name="clearpath_black"><color rgba="0.15 0.15 0.15 1.0" /></material>
-    <material name="clearpath_white"><color rgba="1.0 1.0 1.0 1.0" /></material>
-    <material name="clearpath_red"><color rgba="1.0 0.0 0.0 1.0" /></material>
-    <material name="clearpath_aluminum">
+    <material name="wilbur_dark_grey"><color rgba="0.2 0.2 0.2 1.0" /></material>
+    <material name="wilbur_medium_grey"><color rgba="0.6 0.6 0.6 1.0" /></material>
+    <material name="wilbur_light_grey"><color rgba="0.8 0.8 0.8 1.0" /></material>
+    <material name="wilbur_yellow"><color rgba="0.8 0.8 0.0 1.0" /></material>
+    <material name="wilbur_black"><color rgba="0.15 0.15 0.15 1.0" /></material>
+    <material name="wilbur_white"><color rgba="1.0 1.0 1.0 1.0" /></material>
+    <material name="wilbur_red"><color rgba="1.0 0.0 0.0 1.0" /></material>
+    <material name="wilbur_aluminum">
       <color rgba="0.5 0.5 0.5 1"/>
     </material>
-    <material name="clearpath_plastic">
+    <material name="wilbur_plastic">
       <color rgba="0.1 0.1 0.1   1"/>
     </material>

File: wilbur_description/urdf/diff_unit.urdf.xacro (robot description, xacro)
@@ -38,5 +38,5 @@
           <xacro:gen_mesh force_abs_path="${force_abs_paths}" pkg_name="wilbur_description" file_path="meshes/w200/rocker.stl" />
         </geometry>
-        <material name="clearpath_black" />
+        <material name="wilbur_black" />
       </visual>
     </link>
@@ -56,5 +56,5 @@
           <xacro:gen_mesh force_abs_path="${force_abs_paths}" pkg_name="wilbur_description" file_path="meshes/w200/light.stl" />
         </geometry>
-        <material name="clearpath_white" />
+        <material name="wilbur_white" />
       </visual>
     </link>
@@ -70,5 +70,5 @@
           <xacro:gen_mesh force_abs_path="${force_abs_paths}" pkg_name="wilbur_description" file_path="meshes/w200/light.stl" />
         </geometry>
-        <material name="clearpath_red" />
+        <material name="wilbur_red" />
       </visual>
     </link>

File: wilbur_description/urdf/links/mesh.urdf.xacro (robot description, xacro)
@@ -7,5 +7,5 @@
           <mesh filename="${visual}"/>
         </geometry>
-        <material name="clearpath_dark_grey"/>
+        <material name="wilbur_dark_grey"/>
       </visual>
       <collision>
@@ -13,5 +13,5 @@
           <mesh filename="${visual}"/>
         </geometry>
-        <material name="clearpath_dark_grey"/>
+        <material name="wilbur_dark_grey"/>
       </collision>
     </link>

File: wilbur_description/urdf/w200/attachments/arm_plate.urdf.xacro (robot description, xacro)
@@ -13,5 +13,5 @@
           <xacro:gen_mesh force_abs_path="${force_abs_paths}" pkg_name="wilbur_description" file_path="meshes/w200/arm-mount-plate.stl" />
         </geometry>
-        <material name="clearpath_light_grey"/>
+        <material name="wilbur_light_grey"/>
       </visual>
       <collision>

File: wilbur_description/urdf/w200_macro.urdf.xacro (robot description, xacro)
@@ -69,5 +69,5 @@
             file_path="meshes/w200/chassis.stl" />
         </geometry>
-        <material name="clearpath_black">
+        <material name="wilbur_black">
           <color rgba="0.15 0.15 0.15 1.0" />
         </material>
@@ -79,5 +79,5 @@
             file_path="meshes/w200/e-stop.stl" />
         </geometry>
-        <material name="clearpath_red">
+        <material name="wilbur_red">
           <color rgba="0.9 0.0 0.0 1.0" />
         </material>
@@ -101,5 +101,5 @@
             file_path="meshes/w200/diff-link.stl" />
         </geometry>
-        <material name="clearpath_light_grey" />
+        <material name="wilbur_light_grey" />
       </visual>
       <visual>
@@ -109,5 +109,5 @@
             file_path="meshes/w200/susp-link.stl" />
         </geometry>
-        <material name="clearpath_light_grey" />
+        <material name="wilbur_light_grey" />
       </visual>
       <visual>
@@ -117,5 +117,5 @@
             file_path="meshes/w200/susp-link.stl" />
         </geometry>
-        <material name="clearpath_light_grey" />
+        <material name="wilbur_light_grey" />
       </visual>
     </link>

File: wilbur_description/urdf/wheels/track.urdf.xacro (robot description, xacro)
@@ -9,5 +9,5 @@
           <xacro:gen_mesh force_abs_path="${force_abs_paths}" pkg_name="wilbur_description" file_path="meshes/tracks.dae" />
         </geometry>
-        <material name="clearpath_dark_grey" />
+        <material name="wilbur_dark_grey" />
       </visual>
       <collision>

File: wilbur_description/urdf/wheels/wheel.urdf.xacro (robot description, xacro)
@@ -19,5 +19,5 @@
           <xacro:gen_mesh force_abs_path="${force_abs_paths}" pkg_name="wilbur_description" file_path="meshes/w200/wheels/outdoor.stl" />
         </geometry>
-        <material name="clearpath_dark_grey" />
+        <material name="wilbur_dark_grey" />
       </visual>
       <collision>

File: wilbur_description/urdf/wilbur.xacro (robot description, xacro)
@@ -10,4 +10,5 @@
             gripper_com_port:=/dev/ttyUSB0
             wilbur_ur10e_initial_positions:='$(find wilbur_deploy)/config/ur_initial_positions.yaml'
+            generate_ros2_control_tag:=true
             ">
     <!-- Includes -->
@@ -36,5 +37,5 @@
             file_path="meshes/control_frame.stl" />
         </geometry>
-        <material name="clearpath_dark_grey" />
+        <material name="wilbur_dark_grey" />
       </visual>
       <collision>
@@ -43,5 +44,5 @@
             file_path="meshes/control_frame.stl" />
         </geometry>
-        <material name="clearpath_dark_grey" />
+        <material name="wilbur_dark_grey" />
       </collision>
     </link>
@@ -75,5 +76,6 @@
         com_port="${gripper_com_port}"
         marker_opacity="0.5"
-        finger_xacro="fngr_v6">
+        finger_xacro="fngr_v6"
+        generate_ros2_control_tag="${generate_ros2_control_tag}">
         <origin xyz="0 0 0" rpy="0 0 ${radians(-90)}" />
       </xacro:dextivr_hande>

File: wilbur_mujoco_config/urdf/wilbur_mujoco_processed_inputs.xacro (robot description, xacro)
@@ -24,10 +24,10 @@
                 </xacro:if>
             </xacro:if-->
-            <modify_element type="joint" name="${tf_prefix}arm_0_shoulder_pan_joint" class="size4"/>
-            <modify_element type="joint" name="${tf_prefix}arm_0_shoulder_lift_joint" class="size4"/>
-            <modify_element type="joint" name="${tf_prefix}arm_0_elbow_joint" class="size3_limited"/>
-            <modify_element type="joint" name="${tf_prefix}arm_0_wrist_1_joint" class="size2"/>
-            <modify_element type="joint" name="${tf_prefix}arm_0_wrist_2_joint" class="size2"/>
-            <modify_element type="joint" name="${tf_prefix}arm_0_wrist_3_joint" class="size2"/>
+            <modify_element type="joint" name="${tf_prefix}arm_0_shoulder_pan_joint" class="wilbur_size4"/>
+            <modify_element type="joint" name="${tf_prefix}arm_0_shoulder_lift_joint" class="wilbur_size4"/>
+            <modify_element type="joint" name="${tf_prefix}arm_0_elbow_joint" class="wilbur_size3_limited"/>
+            <modify_element type="joint" name="${tf_prefix}arm_0_wrist_1_joint" class="wilbur_size2"/>
+            <modify_element type="joint" name="${tf_prefix}arm_0_wrist_2_joint" class="wilbur_size2"/>
+            <modify_element type="joint" name="${tf_prefix}arm_0_wrist_3_joint" class="wilbur_size2"/>
             <!--xacro:if value="$(arg hand_type) == 'hande'">
                 <modify_element type="joint" name="${tf_prefix}finger_1_joint" armature="0.5" frictionloss="5.0" />

File: wilbur_mujoco_config/urdf/wilbur_mujoco_raw_inputs.xacro (robot description, xacro)
@@ -25,29 +25,29 @@
         <default>
             <default class="wilbur">
-                <default class="visual">
+                <default class="wilbur_visual">
                     <geom group="2" type="mesh" contype="0" conaffinity="0" />
                 </default>
-                <default class="collision">
+                <default class="wilbur_collision">
                     <geom group="3" type="mesh" friction="1.0 0.005 0.0001" />
                 </default>
             </default>
-            <default class="size5">
+            <default class="wilbur_size5">
                 <joint actuatorfrclimited="true" actuatorfrcrange="-1000 1000" />
                 <position ctrlrange="0.0 0.7" kp="75000" dampratio="1.0" forcerange="-1000 1000" />
             </default>
-            <default class="size4">
+            <default class="wilbur_size4">
                 <joint damping="10" actuatorgravcomp="true" />
                 <general forcerange="-330 330" gainprm="100000" biasprm="0 -100000 -10000" />
             </default>
-            <default class="size3">
+            <default class="wilbur_size3">
                 <joint damping="5" actuatorgravcomp="true" />
                 <general forcerange="-${wheel_ctrl_rng} ${wheel_ctrl_rng}" gainprm="100000"
                     biasprm="0 -100000 -5000" />
-                <default class="size3_limited">
+                <default class="wilbur_size3_limited">
                     <joint range="-3.14${wheel_ctrl_rng} 3.14${wheel_ctrl_rng}" />
                     <general ctrlrange="-3.14${wheel_ctrl_rng} 3.14${wheel_ctrl_rng}" />
                 </default>
             </default>
-            <default class="size2">
+            <default class="wilbur_size2">
                 <joint damping="2" actuatorgravcomp="true" />
                 <general forcerange="-56 56" gainprm="10000" biasprm="0 -10000 -1000" />
@@ -78,15 +78,15 @@
         <actuator>
             <xacro:if value="${include_ur}">
-                <general class="size4" name="${tf_prefix}arm_0_shoulder_pan_joint"
+                <general class="wilbur_size4" name="${tf_prefix}arm_0_shoulder_pan_joint"
                     joint="${tf_prefix}arm_0_shoulder_pan_joint" />
-                <general class="size4" name="${tf_prefix}arm_0_shoulder_lift_joint"
+                <general class="wilbur_size4" name="${tf_prefix}arm_0_shoulder_lift_joint"
                     joint="${tf_prefix}arm_0_shoulder_lift_joint" />
-                <general class="size3_limited" name="${tf_prefix}arm_0_elbow_joint"
+                <general class="wilbur_size3_limited" name="${tf_prefix}arm_0_elbow_joint"
                     joint="${tf_prefix}arm_0_elbow_joint" />
-                <general class="size2" name="${tf_prefix}arm_0_wrist_1_joint"
+                <general class="wilbur_size2" name="${tf_prefix}arm_0_wrist_1_joint"
                     joint="${tf_prefix}arm_0_wrist_1_joint" />
-                <general class="size2" name="${tf_prefix}arm_0_wrist_2_joint"
+                <general class="wilbur_size2" name="${tf_prefix}arm_0_wrist_2_joint"
                     joint="${tf_prefix}arm_0_wrist_2_joint" />
-                <general class="size2" name="${tf_prefix}arm_0_wrist_3_joint"
+                <general class="wilbur_size2" name="${tf_prefix}arm_0_wrist_3_joint"
                     joint="${tf_prefix}arm_0_wrist_3_joint" />
             </xacro:if>

Commit message: Fix force_abs_paths property by turning it into args

File: wilbur_description/urdf/attachments/bulkhead.urdf.xacro (robot description, xacro)
@@ -7,4 +7,5 @@
     *origin
     tf_prefix
+    force_abs_paths:=false
   ">
     <xacro:include
@@ -44,5 +45,5 @@
     </joint>
     <xacro:if value="${model == 'arm_plate'}">
-      <xacro:arm_plate parent_link="${name}_mount">
+      <xacro:arm_plate parent_link="${name}_mount" force_abs_paths="${force_abs_paths}">
         <origin xyz="0.0 0.0 0.0" rpy="0.0 0.0 0.0" />
       </xacro:arm_plate>

File: wilbur_description/urdf/diff_unit.urdf.xacro (robot description, xacro)
@@ -6,5 +6,5 @@
       izz="${m*(x*x+z*z)/12}" />
   </xacro:macro>
-  <xacro:macro name="w200_diff_unit" params="side">
+  <xacro:macro name="w200_diff_unit" params="side force_abs_paths:=false">
     <xacro:if value="${side == 'left'}">
       <xacro:property name="flip" value="1" />

File: wilbur_description/urdf/w200/attachments/arm_plate.urdf.xacro (robot description, xacro)
@@ -6,5 +6,5 @@
              izz="${m*(x*x+z*z)/12}" />
   </xacro:macro>
-  <xacro:macro name="arm_plate" params="name:=arm_plate model:=default parent_link:=default_mount *origin">
+  <xacro:macro name="arm_plate" params="name:=arm_plate model:=default parent_link:=default_mount force_abs_paths:=false *origin">
     <link name="${name}_link">
       <visual>

File: wilbur_description/urdf/w200_macro.urdf.xacro (robot description, xacro)
@@ -7,4 +7,5 @@
                 color:='yellow'
                 ns
+                force_abs_paths:=false
                 ">
     <!-- Include URDF/XACRO Files -->
@@ -92,6 +93,6 @@
     </link>
     <!-- Diff. Unit -->
-    <xacro:w200_diff_unit side="left" />
-    <xacro:w200_diff_unit side="right" />
+    <xacro:w200_diff_unit side="left" force_abs_paths="${force_abs_paths}" />
+    <xacro:w200_diff_unit side="right" force_abs_paths="${force_abs_paths}" />
     <link name="${tf_prefix}diff_link">
       <visual>
@@ -127,14 +128,14 @@
     <!-- Wheels -->
     <xacro:if value="${wheel == 'default'}">
-      <xacro:w200_wheel prefix="front" side="left">
+      <xacro:w200_wheel prefix="front" side="left" force_abs_paths="${force_abs_paths}">
         <origin xyz="${axle_x_offset*1} ${axle_y_offset*1} ${axle_z_offset}" rpy="0 0 0" />
       </xacro:w200_wheel>
-      <xacro:w200_wheel prefix="front" side="right">
+      <xacro:w200_wheel prefix="front" side="right" force_abs_paths="${force_abs_paths}">
         <origin xyz="${axle_x_offset*1} ${axle_y_offset*-1} ${axle_z_offset}" rpy="0 0 0" />
       </xacro:w200_wheel>
-      <xacro:w200_wheel prefix="rear" side="left">
+      <xacro:w200_wheel prefix="rear" side="left" force_abs_paths="${force_abs_paths}">
         <origin xyz="${axle_x_offset*-1} ${axle_y_offset*1} ${axle_z_offset}" rpy="0 0 0" />
       </xacro:w200_wheel>
-      <xacro:w200_wheel prefix="rear" side="right">
+      <xacro:w200_wheel prefix="rear" side="right" force_abs_paths="${force_abs_paths}">
         <origin xyz="${axle_x_offset*-1} ${axle_y_offset*-1} ${axle_z_offset}" rpy="0 0 0" />
       </xacro:w200_wheel>
@@ -142,14 +143,14 @@
     <!-- Tracks -->
     <xacro:if value="${wheel == 'track'}">
-      <xacro:w200_track prefix="front" side="left">
+      <xacro:w200_track prefix="front" side="left" force_abs_paths="${force_abs_paths}">
         <origin xyz="${axle_x_offset*1} ${axle_y_offset*1} ${axle_z_offset}" rpy="0 0 0" />
       </xacro:w200_track>
-      <xacro:w200_track prefix="front" side="right">
+      <xacro:w200_track prefix="front" side="right" force_abs_paths="${force_abs_paths}">
         <origin xyz="${axle_x_offset*1} ${axle_y_offset*-1} ${axle_z_offset}" rpy="0 0 0" />
       </xacro:w200_track>
-      <xacro:w200_track prefix="rear" side="left">
+      <xacro:w200_track prefix="rear" side="left" force_abs_paths="${force_abs_paths}">
         <origin xyz="${axle_x_offset*-1} ${axle_y_offset*1} ${axle_z_offset}" rpy="0 0 ${PI}" />
       </xacro:w200_track>
-      <xacro:w200_track prefix="rear" side="right">
+      <xacro:w200_track prefix="rear" side="right" force_abs_paths="${force_abs_paths}">
         <origin xyz="${axle_x_offset*-1} ${axle_y_offset*-1} ${axle_z_offset}" rpy="0 0 ${PI}" />
       </xacro:w200_track>

File: wilbur_description/urdf/wheels/track.urdf.xacro (robot description, xacro)
@@ -1,5 +1,5 @@
 <?xml version="1.0"?>
 <robot xmlns:xacro="http://ros.org/wiki/xacro" name="w200_track">
-  <xacro:macro name="w200_track" params="prefix side *joint_pose">
+  <xacro:macro name="w200_track" params="prefix side force_abs_paths:=false *joint_pose">
     <xacro:property name="rotate" value="${(prefix=='rear')*math.pi}" />
     <link name="${tf_prefix}${prefix}_${side}_track_link">

File: wilbur_description/urdf/wheels/wheel.urdf.xacro (robot description, xacro)
@@ -6,5 +6,5 @@
       izz="${m*(3*r*r+h*h)/12}" />
   </xacro:macro>
-  <xacro:macro name="w200_wheel" params="prefix side *joint_pose">
+  <xacro:macro name="w200_wheel" params="prefix side force_abs_paths:=false *joint_pose">
     <link name="${tf_prefix}${prefix}_${side}_wheel_link">
       <inertial>

File: wilbur_description/urdf/wilbur.urdf.xacro (robot description, xacro)
@@ -11,6 +11,4 @@
   <xacro:arg name="wilbur_ur10e_initial_positions"
     default="$(find wilbur_deploy)/config/ur_initial_positions.yaml" />
-  <!-- Force absolute mesh paths, necessary for Gazebo. -->
-  <xacro:property name="force_abs_paths" value="$(arg abs_mesh_paths)" scope="global" />
   <xacro:include filename="$(find wilbur_description)/urdf/wilbur.xacro" />
   <xacro:wilbur
@@ -23,4 +21,5 @@
     gripper_com_port="$(arg gripper_com_port)"
     wilbur_ur10e_initial_positions="$(arg wilbur_ur10e_initial_positions)"
+    force_abs_paths="$(arg abs_mesh_paths)"
   />
 </robot>

File: wilbur_description/urdf/wilbur.xacro (robot description, xacro)
@@ -10,4 +10,5 @@
             gripper_com_port:=/dev/ttyUSB0
             wilbur_ur10e_initial_positions:='$(find wilbur_deploy)/config/ur_initial_positions.yaml'
+            force_abs_paths:=false
             generate_ros2_control_tag:=true
             ">
@@ -27,5 +28,6 @@
       model="${tf_prefix}arm_plate"
       parent_link="${tf_prefix}default_mount"
-      tf_prefix="${tf_prefix}">
+      tf_prefix="${tf_prefix}"
+      force_abs_paths="${force_abs_paths}">
       <origin xyz="0.0 0.0 0.0" rpy="0.0 0.0 0.0" />
     </xacro:bulkhead>
@@ -85,4 +87,5 @@
       tf_prefix="${tf_prefix}"
       ns="${ns}"
+      force_abs_paths="${force_abs_paths}"
     />
   </xacro:macro>

File: wilbur_description/urdf/wilbur_mock.urdf.xacro (robot description, xacro)
@@ -12,5 +12,4 @@
         default="$(find wilbur_deploy)/config/ur_initial_positions.yaml" />
     <xacro:include filename="$(find wilbur_description)/urdf/wilbur.xacro" />
-    <xacro:property name="force_abs_paths" value="$(arg abs_mesh_paths)" scope="global" />
     <!-- convert to property to use substitution in function -->
     <xacro:property name="initial_positions_file" default="$(arg wilbur_ur10e_initial_positions)"/>
@@ -24,4 +23,5 @@
         gripper_com_port="$(arg gripper_com_port)"
         wilbur_ur10e_initial_positions="$(arg wilbur_ur10e_initial_positions)"
+        force_abs_paths="$(arg abs_mesh_paths)"
     />
     <xacro:include filename="$(find wilbur_description)/urdf/wilbur_mock.ros2_control.xacro" />

File: wilbur_gz/urdf/wilbur_gz.urdf.xacro (robot description, xacro)
@@ -14,5 +14,4 @@
     <xacro:property name="initial_positions_file" value="$(arg wilbur_ur10e_initial_positions)" />
     <xacro:include filename="$(find wilbur_description)/urdf/wilbur.xacro" />
-    <xacro:property name="force_abs_paths" value="$(arg abs_mesh_paths)" scope="global" />
     <xacro:wilbur
         tf_prefix="$(arg tf_prefix)"
@@ -24,4 +23,5 @@
         gripper_com_port="$(arg gripper_com_port)"
         wilbur_ur10e_initial_positions="$(arg wilbur_ur10e_initial_positions)"
+        force_abs_paths="$(arg abs_mesh_paths)"
     />
     <xacro:include filename="$(find wilbur_gz)/urdf/wilbur_gz.ros2_control.xacro" />
