Commit message: gazebo was complaining about this material

File: wilbur_gz/urdf/w200_gz.xacro (robot description, xacro)
@@ -11,5 +11,6 @@
       <kd value="1.0" />
       <fdir1 value="1 0 0" />
-      <material>Gazebo/DarkGrey</material>
+      <!-- Gazebo was complaining about this material -->
+      <!-- <material>Gazebo/DarkGrey</material> -->
     </gazebo>
   </xacro:macro>
@@ -20,5 +21,5 @@
       <mu2>0.5</mu2>
       <fdir1 value="1 0 0" />
-      <material>Gazebo/DarkGrey</material>
+      <!-- <material>Gazebo/DarkGrey</material> -->
     </gazebo>
   </xacro:macro>
