Commit message: added w200_ros_control macro to the wilbur_gz xacro

File: wilbur_gz/urdf/wilbur_gz.xacro (robot description, xacro)
@@ -14,3 +14,113 @@
     </gazebo>
   </xacro:macro>
+  <xacro:macro name="w200_ros2_control"
+    params="
+    name
+    tf_prefix
+    include_ur:=false
+  ">
+    <ros2_control name="${name}" type="system">
+      <hardware>
+        <plugin>gz_ros2_control/GazeboSimSystem</plugin>
+      </hardware>
+      <xacro:if value="$(arg include_ur)">
+        <joint name="${tf_prefix}arm_0_shoulder_pan_joint">
+          <command_interface name="position" />
+          <command_interface name="velocity" />
+          <command_interface name="effort" />
+          <state_interface name="position" />
+          <state_interface name="velocity" />
+          <state_interface name="effort" />
+        </joint>
+        <joint name="${tf_prefix}arm_0_shoulder_lift_joint">
+          <command_interface name="position" />
+          <command_interface name="velocity" />
+          <command_interface name="effort" />
+          <state_interface name="position" />
+          <state_interface name="velocity" />
+          <state_interface name="effort" />
+        </joint>
+        <joint name="${tf_prefix}arm_0_elbow_joint">
+          <command_interface name="position" />
+          <command_interface name="velocity" />
+          <command_interface name="effort" />
+          <state_interface name="position" />
+          <state_interface name="velocity" />
+          <state_interface name="effort" />
+        </joint>
+        <joint name="${tf_prefix}arm_0_wrist_1_joint">
+          <command_interface name="position" />
+          <command_interface name="velocity" />
+          <command_interface name="effort" />
+          <state_interface name="position" />
+          <state_interface name="velocity" />
+          <state_interface name="effort" />
+        </joint>
+        <joint name="${tf_prefix}arm_0_wrist_2_joint">
+          <command_interface name="position" />
+          <command_interface name="velocity" />
+          <command_interface name="effort" />
+          <state_interface name="position" />
+          <state_interface name="velocity" />
+          <state_interface name="effort" />
+        </joint>
+        <joint name="${tf_prefix}arm_0_wrist_3_joint">
+          <command_interface name="position" />
+          <command_interface name="velocity" />
+          <command_interface name="effort" />
+          <state_interface name="position" />
+          <state_interface name="velocity" />
+          <state_interface name="effort" />
+        </joint>
+      </xacro:if>
+      <joint name="${tf_prefix}front_left_wheel_joint">
+        <command_interface name="velocity">
+          <param name="min">-25</param>
+          <param name="max">25</param>
+        </command_interface>
+        <state_interface name="position">
+          <param name="initial_value">0.0</param>
+        </state_interface>
+        <state_interface name="velocity">
+          <param name="initial_value">0.0</param>
+        </state_interface>
+      </joint>
+      <joint name="${tf_prefix}rear_left_wheel_joint">
+        <command_interface name="velocity">
+          <param name="min">-25</param>
+          <param name="max">25</param>
+        </command_interface>
+        <state_interface name="position">
+          <param name="initial_value">0.0</param>
+        </state_interface>
+        <state_interface name="velocity">
+          <param name="initial_value">0.0</param>
+        </state_interface>
+      </joint>
+      <joint name="${tf_prefix}front_right_wheel_joint">
+        <command_interface name="velocity">
+          <param name="min">-25</param>
+          <param name="max">25</param>
+        </command_interface>
+        <state_interface name="position">
+          <param name="initial_value">0.0</param>
+        </state_interface>
+        <state_interface name="velocity">
+          <param name="initial_value">0.0</param>
+        </state_interface>
+      </joint>
+      <joint name="${tf_prefix}rear_right_wheel_joint">
+        <command_interface name="velocity">
+          <param name="min">-25</param>
+          <param name="max">25</param>
+        </command_interface>
+        <state_interface name="position">
+          <param name="initial_value">0.0</param>
+        </state_interface>
+        <state_interface name="velocity">
+          <param name="initial_value">0.0</param>
+        </state_interface>
+      </joint>
+    </ros2_control>
+  </xacro:macro>
 </robot>
