Commit message: passing initial position gz ros2 control

File: wilbur_gz/urdf/wilbur_gz.urdf.xacro (robot description, xacro)
@@ -12,4 +12,5 @@
     <xacro:arg name="wilbur_ur10e_initial_positions"
         default="$(find wilbur_deploy)/config/ur_initial_positions.yaml" />
+    <xacro:property name="initial_positions_file" value="$(arg wilbur_ur10e_initial_positions)" />
     <xacro:include filename="$(find wilbur_description)/urdf/wilbur.xacro" />
     <xacro:property name="force_abs_paths" value="$(arg abs_mesh_paths)" scope="global" />
@@ -34,4 +35,6 @@
         name="wilbur"
         tf_prefix="$(arg tf_prefix)"
-        include_ur="$(arg include_ur)" />
+        include_ur="$(arg include_ur)"
+        wilbur_ur10e_initial_positions="${xacro.load_yaml(initial_positions_file)}"
+    />
 </robot>
