Commit message: added imu_broadcaster

File: wilbur_mujoco_config/urdf/wilbur_mujoco_processed_inputs.xacro (robot description, xacro)
@@ -1 +1,38 @@
-!co
+<?xml version="1.0"?>
+<robot xmlns:xacro="http://wiki.ros.org/xacro">
+  <xacro:macro name="wilbur_mujoco_processed_inputs" params="
+    tf_prefix:=''
+    hand_type:='hande'
+    hande_finger_type:='fngr_v6'
+    include_ur:='true'
+  ">
+        <!-- Process arguments for the URDF -->
+        <xacro:if value="$(arg include_ur)">
+            <!-- Decompose the finger meshes based on the finger types available. hw2-->
+            <!--xacro:if value="$(arg hand_type) == 'hande'">
+                <xacro:if value="$(arg hande_finger_type) == 'fngr_original' or right_hande_finger_type == 'fngr_original'}">
+                <decompose_mesh mesh_name="finger_1" threshold="0.05"/>
+                </xacro:if>
+                <xacro:if value="$(arg hande_finger_type) == 'fngr_nail_v2'}">
+                <decompose_mesh mesh_name="hande_fngr_nail_v2" threshold="0.05"/>
+                </xacro:if>
+                <xacro:if value="$(arg hande_finger_type) == 'fngr_v2_m'}">
+                <decompose_mesh mesh_name="imetro_finger_v2_m_vis" threshold="0.05"/>
+                </xacro:if>
+                <xacro:if value="$(arg hande_finger_type) == 'fngr_v6'}">
+                <decompose_mesh mesh_name="finger_v6" threshold="0.05"/>
+                </xacro:if>
+            </xacro:if-->
+            <modify_element type="joint" name="${tf_prefix}arm_0_shoulder_pan_joint" class="size4"/>
+            <modify_element type="joint" name="${tf_prefix}arm_0_shoulder_lift_joint" class="size4"/>
+            <modify_element type="joint" name="${tf_prefix}arm_0_elbow_joint" class="size3_limited"/>
+            <modify_element type="joint" name="${tf_prefix}arm_0_wrist_1_joint" class="size2"/>
+            <modify_element type="joint" name="${tf_prefix}arm_0_wrist_2_joint" class="size2"/>
+            <modify_element type="joint" name="${tf_prefix}arm_0_wrist_3_joint" class="size2"/>
+            <!--xacro:if value="$(arg hand_type) == 'hande'">
+                <modify_element type="joint" name="${tf_prefix}finger_1_joint" armature="0.5" frictionloss="5.0" />
+                <modify_element type="joint" name="${tf_prefix}finger_2_joint" armature="0.5" frictionloss="5.0" />
+            </xacro:if-->
+        </xacro:if>
+    </xacro:macro>
+</robot>

File: wilbur_mujoco_config/urdf/wilbur_mujoco_raw_inputs.xacro (robot description, xacro)
@@ -1,5 +1,6 @@
 <?xml version="1.0"?>
 <robot xmlns:xacro="http://wiki.ros.org/xacro">
-    <xacro:macro name="wilbur_mujoco_raw_inputs" params="
+    <xacro:macro name="wilbur_mujoco_raw_inputs"
+        params="
         tf_prefix:=''
         hand_type:='hande'
@@ -11,9 +12,9 @@
         <xacro:property name="wheel_ctrl_rng" value="5" />
         <option
-           solver="Newton"
-           cone="elliptic"
-           noslip_iterations="3"
+            solver="Newton"
+            cone="elliptic"
+            noslip_iterations="3"
             tolerance="1e-10">
-           <flag multiccd="enable" />
+            <flag multiccd="enable" />
         </option>
         <default>
@@ -32,56 +33,65 @@
                         condim="6"
                         friction="1.0 0.005 0.0001"
-                        priority="1"/>
+                        priority="1" />
                 </default>
             </default>
             <default class="size5">
-                <joint actuatorfrclimited="true" actuatorfrcrange="-1000 1000"/>
-                <position ctrlrange="0.0 0.7" kp="75000" dampratio="1.0" forcerange="-1000 1000"/>
+                <joint actuatorfrclimited="true" actuatorfrcrange="-1000 1000" />
+                <position ctrlrange="0.0 0.7" kp="75000" dampratio="1.0" forcerange="-1000 1000" />
             </default>
             <default class="size4">
-                <joint damping="10" actuatorgravcomp="true"/>
-                <general forcerange="-330 330" gainprm="100000" biasprm="0 -100000 -10000"/>
+                <joint damping="10" actuatorgravcomp="true" />
+                <general forcerange="-330 330" gainprm="100000" biasprm="0 -100000 -10000" />
             </default>
             <default class="size3">
-                <joint damping="5" actuatorgravcomp="true"/>
-                <general forcerange="-${wheel_ctrl_rng}0 ${wheel_ctrl_rng}0" gainprm="100000" biasprm="0 -100000 -5000"/>
+                <joint damping="5" actuatorgravcomp="true" />
+                <general forcerange="-${wheel_ctrl_rng}0 ${wheel_ctrl_rng}0" gainprm="100000"
+                    biasprm="0 -100000 -5000" />
                 <default class="size3_limited">
-                    <joint range="-3.14${wheel_ctrl_rng} 3.14${wheel_ctrl_rng}"/>
-                    <general ctrlrange="-3.14${wheel_ctrl_rng} 3.14${wheel_ctrl_rng}"/>
+                    <joint range="-3.14${wheel_ctrl_rng} 3.14${wheel_ctrl_rng}" />
+                    <general ctrlrange="-3.14${wheel_ctrl_rng} 3.14${wheel_ctrl_rng}" />
                 </default>
             </default>
             <default class="size2">
                 <joint damping="2" actuatorgravcomp="true" />
-                <general forcerange="-56 56" gainprm="10000" biasprm="0 -10000 -1000"/>
+                <general forcerange="-56 56" gainprm="10000" biasprm="0 -10000 -1000" />
             </default>
         </default>
-        <!--extension>
-        <plugin plugin="mujoco.plugin.lidar">
-            <instance name="lidar3d_0">
-                <config key="resolution" value="120 1"/>
-                <config key="azimuth_range" value="-1.55 1.55"/>
-                <config key="elevation_range" value="0.0, 0.3"/>
-                <config key="max_range" value="${wheel_ctrl_rng}.0"/>
-                <config key="min_range" value="0.05"/>
-                <config key="update_rate" value="4.0"/>
-            </instance>
-        </plugin>
-    </extension-->
-        <!--sensor>
-        <plugin name="lidar3d_0" instance="lidar3d_0" objtype="site" objname="lidar3d_0_laser"/>
-    </sensor-->
-        <!--sensor>
-        <framequat name="imu_sensor_quat" objtype="site" objname="imu_0_link" />
-        <gyro name="imu_sensor_gyro" site="imu_0_link" />
-        <accelerometer name="imu_sensor_accel" site="imu_0_link" />
-    </sensor-->
+        <!--
+        <extension>
+            <plugin plugin="mujoco.plugin.lidar">
+                <instance name="lidar3d_0">
+                    <config key="resolution" value="120 1"/>
+                    <config key="azimuth_range" value="-1.55 1.55"/>
+                    <config key="elevation_range" value="0.0, 0.3"/>
+                    <config key="max_range" value="${wheel_ctrl_rng}.0"/>
+                    <config key="min_range" value="0.05"/>
+                    <config key="update_rate" value="4.0"/>
+                </instance>
+            </plugin>
+        </extension>
+        <sensor>
+            <plugin name="lidar3d_0" instance="lidar3d_0" objtype="site" objname="lidar3d_0_laser"/>
+        </sensor>
+    -->
+        <sensor>
+            <framequat name="imu_sensor_quat" objtype="site" objname="imu_0_link" />
+            <gyro name="imu_sensor_gyro" site="imu_0_link" />
+            <accelerometer name="imu_sensor_accel" site="imu_0_link" />
+        </sensor>
         <actuator>
             <xacro:if value="${include_ur}">
-                <general class="size4" name="${tf_prefix}arm_0_shoulder_pan_joint" joint="${tf_prefix}arm_0_shoulder_pan_joint"/>
-                <general class="size4" name="${tf_prefix}arm_0_shoulder_lift_joint" joint="${tf_prefix}arm_0_shoulder_lift_joint"/>
-                <general class="size3_limited" name="${tf_prefix}arm_0_elbow_joint" joint="${tf_prefix}arm_0_elbow_joint"/>
-                <general class="size2" name="${tf_prefix}arm_0_wrist_1_joint" joint="${tf_prefix}arm_0_wrist_1_joint"/>
-                <general class="size2" name="${tf_prefix}arm_0_wrist_2_joint" joint="${tf_prefix}arm_0_wrist_2_joint"/>
-                <general class="size2" name="${tf_prefix}arm_0_wrist_3_joint" joint="${tf_prefix}arm_0_wrist_3_joint"/>
+                <general class="size4" name="${tf_prefix}arm_0_shoulder_pan_joint"
+                    joint="${tf_prefix}arm_0_shoulder_pan_joint" />
+                <general class="size4" name="${tf_prefix}arm_0_shoulder_lift_joint"
+                    joint="${tf_prefix}arm_0_shoulder_lift_joint" />
+                <general class="size3_limited" name="${tf_prefix}arm_0_elbow_joint"
+                    joint="${tf_prefix}arm_0_elbow_joint" />
+                <general class="size2" name="${tf_prefix}arm_0_wrist_1_joint"
+                    joint="${tf_prefix}arm_0_wrist_1_joint" />
+                <general class="size2" name="${tf_prefix}arm_0_wrist_2_joint"
+                    joint="${tf_prefix}arm_0_wrist_2_joint" />
+                <general class="size2" name="${tf_prefix}arm_0_wrist_3_joint"
+                    joint="${tf_prefix}arm_0_wrist_3_joint" />
             </xacro:if>
             <velocity name="rear_right_wheel_joint" joint="rear_right_wheel_joint"

File: wilbur_mujoco_config/urdf/wilbur_mujoco_ros2_control.xacro (robot description, xacro)
@@ -118,4 +118,18 @@
                 <state_interface name="effort" />
             </joint>
+            <sensor name="imu_sensor">
+                <param name="mujoco_type">imu</param>
+                <param name="mujoco_sensor_name">imu_sensor</param>
+                <state_interface name="orientation.x" />
+                <state_interface name="orientation.y" />
+                <state_interface name="orientation.z" />
+                <state_interface name="orientation.w" />
+                <state_interface name="angular_velocity.x" />
+                <state_interface name="angular_velocity.y" />
+                <state_interface name="angular_velocity.z" />
+                <state_interface name="linear_acceleration.x" />
+                <state_interface name="linear_acceleration.y" />
+                <state_interface name="linear_acceleration.z" />
+            </sensor>
         </ros2_control>
     </xacro:macro>
