Commit message: Working with wheel friction to get turning behavior

File: wilbur_mujoco_config/urdf/wilbur_mujoco_raw_inputs.xacro (robot description, xacro)
@@ -1,21 +1,31 @@
 <?xml version="1.0"?>
 <robot xmlns:xacro="http://wiki.ros.org/xacro">
-  <xacro:macro name="wilbur_mujoco_raw_inputs">
-    <xacro:property name="wheel_joint_force_limit" value="10000" />
-    <xacro:property name="steering_joint_force_limit" value="10000" />
-    <option integrator="implicitfast" impratio="20" cone="elliptic" noslip_iterations="5">
-    <flag multiccd="enable"/>
-    </option>
-    <default>
-        <default class="wilbur">
-            <default class="visual">
-                <geom group="2" type="mesh" contype="0" conaffinity="0"/>
-            </default>
-            <default class="collision">
-                <geom group="3" type="mesh"/>
+    <xacro:macro name="wilbur_mujoco_raw_inputs">
+        <xacro:property name="wheel_joint_force_limit" value="100000" />
+        <xacro:property name="wheel_kv" value="125" />
+        <!--option
+            integrator="implicitfast" impratio="20" cone="elliptic" noslip_iterations="5">
+            <flag multiccd="enable" />
+        </option-->
+        <default>
+            <default class="wilbur">
+                <default class="visual">
+                    <geom group="2" type="mesh" contype="0" conaffinity="0" />
+                </default>
+                <default class="collision">
+                    <geom group="3" type="mesh" friction="1.0 0.005 0.0001" />
+                </default>
+                <default class="wheel">
+                    <!--geom
+                    group="3" type="mesh" friction="1.0 0.005 0.0001" solref="0.015 1"
+                        solimp="0.9 0.95 0.001 0.5 2" /-->
+                    <geom group="3" type="cylinder" size="0.3 0.125"
+                        friction="0.9 0.1 0.1"
+                        solref="0.02 1.0"
+                        solimp="0.01 0.95 0.001 0.5 2" />
+                </default>
             </default>
         </default>
-    </default>
-    <!--extension>
+        <!--extension>
         <plugin plugin="mujoco.plugin.lidar">
             <instance name="lidar3d_0">
@@ -29,24 +39,37 @@
         </plugin>
     </extension-->
-    <!--sensor>
+        <!--sensor>
         <plugin name="lidar3d_0" instance="lidar3d_0" objtype="site" objname="lidar3d_0_laser"/>
     </sensor-->
-    <!--sensor>
+        <!--sensor>
         <framequat name="imu_sensor_quat" objtype="site" objname="imu_0_link" />
         <gyro name="imu_sensor_gyro" site="imu_0_link" />
         <accelerometer name="imu_sensor_accel" site="imu_0_link" />
     </sensor-->
-    <actuator>
-        <velocity name="rear_right_wheel_joint" joint="rear_right_wheel_joint" ctrlrange="-15 15" kv="500000" forcerange="${-1 * wheel_joint_force_limit}  ${wheel_joint_force_limit}"/>
-        <velocity name="rear_left_wheel_joint" joint="rear_left_wheel_joint" ctrlrange="-15 15" kv="500000" forcerange="${-1 * wheel_joint_force_limit}  ${wheel_joint_force_limit}"/>
-        <velocity name="front_right_wheel_joint" joint="rear_right_wheel_joint" ctrlrange="-15 15" kv="500000" forcerange="${-1 * wheel_joint_force_limit}  ${wheel_joint_force_limit}"/>
-        <velocity name="front_left_wheel_joint" joint="rear_left_wheel_joint" ctrlrange="-15 15" kv="500000" forcerange="${-1 * wheel_joint_force_limit}  ${wheel_joint_force_limit}"/>
-    </actuator>
-    <contact>
-        <exclude body1="base_link" body2="front_left_wheel_link"/>
-        <exclude body1="base_link" body2="front_right_wheel_link"/>
-        <exclude body1="base_link" body2="rear_left_wheel_link"/>
-        <exclude body1="base_link" body2="rear_right_wheel_link"/>
-    </contact>
-  </xacro:macro>
+        <actuator>
+            <velocity name="rear_right_wheel_joint" joint="rear_right_wheel_joint"
+                ctrlrange="-15 15" kv="${wheel_kv}"
+                forcerange="${-1 * wheel_joint_force_limit}  ${wheel_joint_force_limit}" />
+            <velocity name="rear_left_wheel_joint" joint="rear_left_wheel_joint"
+                ctrlrange="-15 15" kv="${wheel_kv}"
+                forcerange="${-1 * wheel_joint_force_limit}  ${wheel_joint_force_limit}" />
+            <velocity name="front_right_wheel_joint" joint="front_right_wheel_joint"
+                ctrlrange="-15 15" kv="${wheel_kv}"
+                forcerange="${-1 * wheel_joint_force_limit}  ${wheel_joint_force_limit}" />
+            <velocity name="front_left_wheel_joint" joint="front_left_wheel_joint"
+                ctrlrange="-15 15" kv="${wheel_kv}"
+                forcerange="${-1 * wheel_joint_force_limit}  ${wheel_joint_force_limit}" />
+        </actuator>
+        <contact>
+            <exclude body1="base_link" body2="front_left_wheel_link" />
+            <exclude body1="base_link" body2="front_right_wheel_link" />
+            <exclude body1="base_link" body2="rear_left_wheel_link" />
+            <exclude body1="base_link" body2="rear_right_wheel_link" />
+        </contact>
+        <!-- Welds a free-floating body to a fixed/mocap frame in mid-air -->
+        <!-- puts the robot "on blocks"-->
+        <!--equality>
+            <weld body1="base_link" body2="world" />
+        </equality-->
+    </xacro:macro>
 </robot>

Commit message: Adjusted wheel velocity options

File: wilbur_mujoco_config/urdf/wilbur_mujoco_raw_inputs.xacro (robot description, xacro)
@@ -1,9 +1,22 @@
 <?xml version="1.0"?>
 <robot xmlns:xacro="http://wiki.ros.org/xacro">
-    <xacro:macro name="wilbur_mujoco_raw_inputs">
+    <xacro:macro name="wilbur_mujoco_raw_inputs" params="
+        tf_prefix:=''
+        hand_type:='hande'
+        hande_finger_type:='fngr_v6'
+        include_ur:='true'
+    ">
         <xacro:property name="wheel_joint_force_limit" value="100000" />
-        <xacro:property name="wheel_kv" value="125" />
+        <xacro:property name="wheel_kv" value="400" />
+        <xacro:property name="wheel_ctrl_rng" value="5" />
+        <option
+           solver="Newton"
+           cone="elliptic"
+           noslip_iterations="3"
+            tolerance="1e-10">
+           <flag multiccd="enable" />
+        </option>
         <!--option
-            integrator="implicitfast" impratio="20" cone="elliptic" noslip_iterations="5">
+            integrator="implicitfast" impratio="20" cone="elliptic" noslip_iterations="5" >
             <flag multiccd="enable" />
         </option-->
@@ -18,11 +31,41 @@
                 <default class="wheel">
                     <!--geom
-                    group="3" type="mesh" friction="1.0 0.005 0.0001" solref="0.015 1"
+                    group="3" type="mesh" friction="1.0 0.005 0.0001" solref="0.0${wheel_ctrl_rng} 1"
                         solimp="0.9 0.95 0.001 0.5 2" /-->
-                    <geom group="3" type="cylinder" size="0.3 0.125"
-                        friction="0.9 0.1 0.1"
-                        solref="0.02 1.0"
-                        solimp="0.01 0.95 0.001 0.5 2" />
+                    <!--geom type="capsule" size="0.3 0.0125" euler="90 0 0" condim="4"
+                          friction="1.0 0.005 0.01" solref="0.004 1" solimp="0.95 0.99 0.001" group="3"/-->
+                    <!--
+              condim="6" enables 2D sliding, 1D torsional (spinning), and 2D rolling friction.
+              friction order: [sliding_x, sliding_y, torsional, rolling_x, rolling_y]
+              solimp/solref: tuned for Newton solver stability to prevent numerical jitter.
+            -->
+                    <geom type="mesh"
+                        mass="15.0"
+                        zaxis="0 1 0"
+                        material="rubber"
+                        condim="6"
+                        friction="1.0 0.005 0.0001"
+                        priority="1"/>
                 </default>
+            </default>
+            <default class="size5">
+                <joint actuatorfrclimited="true" actuatorfrcrange="-1000 1000"/>
+                <position ctrlrange="0.0 0.7" kp="75000" dampratio="1.0" forcerange="-1000 1000"/>
+            </default>
+            <default class="size4">
+                <joint damping="10" actuatorgravcomp="true"/>
+                <general forcerange="-330 330" gainprm="100000" biasprm="0 -100000 -10000"/>
+            </default>
+            <default class="size3">
+                <joint damping="5" actuatorgravcomp="true"/>
+                <general forcerange="-${wheel_ctrl_rng}0 ${wheel_ctrl_rng}0" gainprm="100000" biasprm="0 -100000 -5000"/>
+                <default class="size3_limited">
+                    <joint range="-3.14${wheel_ctrl_rng} 3.14${wheel_ctrl_rng}"/>
+                    <general ctrlrange="-3.14${wheel_ctrl_rng} 3.14${wheel_ctrl_rng}"/>
+                </default>
+            </default>
+            <default class="size2">
+                <joint damping="2" actuatorgravcomp="true" />
+                <general forcerange="-56 56" gainprm="10000" biasprm="0 -10000 -1000"/>
             </default>
         </default>
@@ -33,5 +76,5 @@
                 <config key="azimuth_range" value="-1.55 1.55"/>
                 <config key="elevation_range" value="0.0, 0.3"/>
-                <config key="max_range" value="15.0"/>
+                <config key="max_range" value="${wheel_ctrl_rng}.0"/>
                 <config key="min_range" value="0.05"/>
                 <config key="update_rate" value="4.0"/>
@@ -48,15 +91,23 @@
     </sensor-->
         <actuator>
+            <xacro:if value="${include_ur}">
+                <general class="size4" name="${tf_prefix}arm_0_shoulder_pan_joint" joint="${tf_prefix}arm_0_shoulder_pan_joint"/>
+                <general class="size4" name="${tf_prefix}arm_0_shoulder_lift_joint" joint="${tf_prefix}arm_0_shoulder_lift_joint"/>
+                <general class="size3_limited" name="${tf_prefix}arm_0_elbow_joint" joint="${tf_prefix}arm_0_elbow_joint"/>
+                <general class="size2" name="${tf_prefix}arm_0_wrist_1_joint" joint="${tf_prefix}arm_0_wrist_1_joint"/>
+                <general class="size2" name="${tf_prefix}arm_0_wrist_2_joint" joint="${tf_prefix}arm_0_wrist_2_joint"/>
+                <general class="size2" name="${tf_prefix}arm_0_wrist_3_joint" joint="${tf_prefix}arm_0_wrist_3_joint"/>
+            </xacro:if>
             <velocity name="rear_right_wheel_joint" joint="rear_right_wheel_joint"
-                ctrlrange="-15 15" kv="${wheel_kv}"
+                ctrlrange="${-1 * wheel_ctrl_rng} ${wheel_ctrl_rng}" kv="${wheel_kv}"
                 forcerange="${-1 * wheel_joint_force_limit}  ${wheel_joint_force_limit}" />
             <velocity name="rear_left_wheel_joint" joint="rear_left_wheel_joint"
-                ctrlrange="-15 15" kv="${wheel_kv}"
+                ctrlrange="${-1 * wheel_ctrl_rng} ${wheel_ctrl_rng}" kv="${wheel_kv}"
                 forcerange="${-1 * wheel_joint_force_limit}  ${wheel_joint_force_limit}" />
             <velocity name="front_right_wheel_joint" joint="front_right_wheel_joint"
-                ctrlrange="-15 15" kv="${wheel_kv}"
+                ctrlrange="${-1 * wheel_ctrl_rng} ${wheel_ctrl_rng}" kv="${wheel_kv}"
                 forcerange="${-1 * wheel_joint_force_limit}  ${wheel_joint_force_limit}" />
             <velocity name="front_left_wheel_joint" joint="front_left_wheel_joint"
-                ctrlrange="-15 15" kv="${wheel_kv}"
+                ctrlrange="${-1 * wheel_ctrl_rng} ${wheel_ctrl_rng}" kv="${wheel_kv}"
                 forcerange="${-1 * wheel_joint_force_limit}  ${wheel_joint_force_limit}" />
         </actuator>

Commit message: Matched the ros control rate to the mujoco step size

File: wilbur_mujoco_config/urdf/wilbur_mujoco_raw_inputs.xacro (robot description, xacro)
@@ -7,13 +7,18 @@
         hande_finger_type:='fngr_v6'
         include_ur:='true'
+        on_blocks:='false'
     ">
         <xacro:property name="wheel_joint_force_limit" value="100000" />
-        <xacro:property name="wheel_kv" value="400" />
-        <xacro:property name="wheel_ctrl_rng" value="5" />
+        <xacro:property name="wheel_kv" value="50" />
+        <xacro:property name="wheel_ctrl_rng" value="30" />
+        <xacro:property name="wheel_gear" value="1" />
+        <xacro:property name="wheel_mass" value="23.0" />
         <option
             solver="Newton"
             cone="elliptic"
             noslip_iterations="3"
-            tolerance="1e-10">
+            integrator="implicitfast"
+            timestep="0.002"
+            tolerance="1e-6">
             <flag multiccd="enable" />
         </option>
@@ -26,15 +31,17 @@
                     <geom group="3" type="mesh" friction="1.0 0.005 0.0001" />
                 </default>
+                <!-- this is not used in the code - would like to be able to change the collision properties on the wheel
                 <default class="wheel">
                     <geom type="mesh"
-                        mass="15.0"
+                        mass="${wheel_mass}"
                         zaxis="0 1 0"
                         material="rubber"
                         condim="6"
-                        friction="2.0 0.005 0.0001"
+                        friction="3.0 0.005 0.0001"
                         solimp="0.015 1.0 0.9 0.95 2"
                         solref="0.02 1.0"
                         priority="1" />
                 </default>
+            -->
             </default>
             <default class="size5">
@@ -48,5 +55,5 @@
             <default class="size3">
                 <joint damping="5" actuatorgravcomp="true" />
-                <general forcerange="-${wheel_ctrl_rng}0 ${wheel_ctrl_rng}0" gainprm="100000"
+                <general forcerange="-${wheel_ctrl_rng} ${wheel_ctrl_rng}" gainprm="100000"
                     biasprm="0 -100000 -5000" />
                 <default class="size3_limited">
@@ -58,4 +65,7 @@
                 <joint damping="2" actuatorgravcomp="true" />
                 <general forcerange="-56 56" gainprm="10000" biasprm="0 -10000 -1000" />
+            </default>
+            <default class="wheel_joint">
+                <joint damping="0.001" armature="0.01"/>
             </default>
         </default>
@@ -99,14 +109,18 @@
             <velocity name="rear_right_wheel_joint" joint="rear_right_wheel_joint"
                 ctrlrange="${-1 * wheel_ctrl_rng} ${wheel_ctrl_rng}" kv="${wheel_kv}"
-                forcerange="${-1 * wheel_joint_force_limit}  ${wheel_joint_force_limit}" />
+                forcerange="${-1 * wheel_joint_force_limit}  ${wheel_joint_force_limit}"
+                gear="${wheel_gear}"/>
             <velocity name="rear_left_wheel_joint" joint="rear_left_wheel_joint"
                 ctrlrange="${-1 * wheel_ctrl_rng} ${wheel_ctrl_rng}" kv="${wheel_kv}"
-                forcerange="${-1 * wheel_joint_force_limit}  ${wheel_joint_force_limit}" />
+                forcerange="${-1 * wheel_joint_force_limit}  ${wheel_joint_force_limit}"
+                gear="${wheel_gear}"/>
             <velocity name="front_right_wheel_joint" joint="front_right_wheel_joint"
                 ctrlrange="${-1 * wheel_ctrl_rng} ${wheel_ctrl_rng}" kv="${wheel_kv}"
-                forcerange="${-1 * wheel_joint_force_limit}  ${wheel_joint_force_limit}" />
+                forcerange="${-1 * wheel_joint_force_limit}  ${wheel_joint_force_limit}"
+                gear="${wheel_gear}"/>
             <velocity name="front_left_wheel_joint" joint="front_left_wheel_joint"
                 ctrlrange="${-1 * wheel_ctrl_rng} ${wheel_ctrl_rng}" kv="${wheel_kv}"
-                forcerange="${-1 * wheel_joint_force_limit}  ${wheel_joint_force_limit}" />
+                forcerange="${-1 * wheel_joint_force_limit}  ${wheel_joint_force_limit}"
+                gear="${wheel_gear}"/>
         </actuator>
         <contact>
@@ -118,7 +132,9 @@
         <!-- Welds a free-floating body to a fixed/mocap frame in mid-air -->
         <!-- puts the robot "on blocks"-->
-        <!--equality>
-            <weld body1="base_link" body2="world" />
-        </equality-->
+        <xacro:if value="${on_blocks}">
+            <equality>
+                <weld body1="base_link" body2="world" />
+            </equality>
+        </xacro:if>
     </xacro:macro>
 </robot>

Commit message: Updated kv

File: wilbur_mujoco_config/urdf/wilbur_mujoco_raw_inputs.xacro (robot description, xacro)
@@ -10,5 +10,5 @@
     ">
         <xacro:property name="wheel_joint_force_limit" value="100000" />
-        <xacro:property name="wheel_kv" value="50" />
+        <xacro:property name="wheel_kv" value="350" />
         <xacro:property name="wheel_ctrl_rng" value="30" />
         <xacro:property name="wheel_gear" value="1" />

Commit message: made the send_cmd node time based

File: wilbur_mujoco_config/urdf/wilbur_mujoco_raw_inputs.xacro (robot description, xacro)
@@ -9,16 +9,16 @@
         on_blocks:='false'
     ">
-        <xacro:property name="wheel_joint_force_limit" value="100000" />
-        <xacro:property name="wheel_kv" value="350" />
+        <xacro:property name="wheel_joint_force_limit" value="10000000" />
+        <xacro:property name="wheel_kv" value="60000" />
         <xacro:property name="wheel_ctrl_rng" value="30" />
         <xacro:property name="wheel_gear" value="1" />
-        <xacro:property name="wheel_mass" value="23.0" />
         <option
             solver="Newton"
             cone="elliptic"
-            noslip_iterations="3"
+            noslip_iterations="5"
             integrator="implicitfast"
             timestep="0.002"
-            tolerance="1e-6">
+            impratio="15.0"
+            tolerance="1e-10">
             <flag multiccd="enable" />
         </option>
@@ -31,17 +31,13 @@
                     <geom group="3" type="mesh" friction="1.0 0.005 0.0001" />
                 </default>
-                <!-- this is not used in the code - would like to be able to change the collision properties on the wheel
-                <default class="wheel">
+                <!-- this is not used in the code - would like to be able to change the collision properties on the wheel -->
+                <!--default class="wheel">
                     <geom type="mesh"
-                        mass="${wheel_mass}"
-                        zaxis="0 1 0"
-                        material="rubber"
                         condim="6"
-                        friction="3.0 0.005 0.0001"
-                        solimp="0.015 1.0 0.9 0.95 2"
+                        friction="1.0 0.005 0.00001"
+                        solimp=".5 1.0 0.9 0.95 2"
                         solref="0.02 1.0"
                         priority="1" />
-                </default>
-            -->
+                </default-->
             </default>
             <default class="size5">
@@ -67,5 +63,5 @@
             </default>
             <default class="wheel_joint">
-                <joint damping="0.001" armature="0.01"/>
+                <joint frictionloss="0.05" armature="0.5" damping="0.8"/>
             </default>
         </default>

Commit message: change options and set forcelimited to "true" for wheel joints

File: wilbur_mujoco_config/urdf/wilbur_mujoco_raw_inputs.xacro (robot description, xacro)
@@ -16,8 +16,8 @@
             solver="Newton"
             cone="elliptic"
-            noslip_iterations="5"
+            noslip_iterations="2"
             integrator="implicitfast"
             timestep="0.002"
-            impratio="15.0"
+            impratio="100"
             tolerance="1e-10">
             <flag multiccd="enable" />
@@ -63,5 +63,6 @@
             </default>
             <default class="wheel_joint">
-                <joint frictionloss="0.05" armature="0.5" damping="0.8"/>
+                <!--joint armature="0.5" damping="10" /-->
+                <!--joint frictionloss="0.05" armature="0.5" damping="10" /-->
             </default>
         </default>
@@ -105,16 +106,20 @@
             <velocity name="rear_right_wheel_joint" joint="rear_right_wheel_joint"
                 ctrlrange="${-1 * wheel_ctrl_rng} ${wheel_ctrl_rng}" kv="${wheel_kv}"
+                forcelimited="true"
                 forcerange="${-1 * wheel_joint_force_limit}  ${wheel_joint_force_limit}"
                 gear="${wheel_gear}"/>
             <velocity name="rear_left_wheel_joint" joint="rear_left_wheel_joint"
                 ctrlrange="${-1 * wheel_ctrl_rng} ${wheel_ctrl_rng}" kv="${wheel_kv}"
+                forcelimited="true"
                 forcerange="${-1 * wheel_joint_force_limit}  ${wheel_joint_force_limit}"
                 gear="${wheel_gear}"/>
             <velocity name="front_right_wheel_joint" joint="front_right_wheel_joint"
                 ctrlrange="${-1 * wheel_ctrl_rng} ${wheel_ctrl_rng}" kv="${wheel_kv}"
+                forcelimited="true"
                 forcerange="${-1 * wheel_joint_force_limit}  ${wheel_joint_force_limit}"
                 gear="${wheel_gear}"/>
             <velocity name="front_left_wheel_joint" joint="front_left_wheel_joint"
                 ctrlrange="${-1 * wheel_ctrl_rng} ${wheel_ctrl_rng}" kv="${wheel_kv}"
+                forcelimited="true"
                 forcerange="${-1 * wheel_joint_force_limit}  ${wheel_joint_force_limit}"
                 gear="${wheel_gear}"/>
